File: I2C1_SPI3.kicad_sch (KiCad schematic)
At the start: 6 parts, among them U18 ZX-SH1.0-4PWT, U19 ZX-SH1.0-6PWT

Commit message: Remove unused file
Parts:
- removed R30, R31: 4.7K, Resistor_SMD:R_0402_1005Metric, symbol Device:R_Small
- removed U18: ZX-SH1.0-4PWT, EasyEDA:CONN-SMD_4P-P1.00_MEGASTAR_ZX-SH1.0-4PWT, symbol EasyEDA:ZX-SH1.0-4PWT
