File: LEVIA_H7.kicad_sch (KiCad schematic)
At the start: 8 parts, among them U1 USBLC6-2P6

Commit message: Remove unused file
Connections:
- net USB_OTG_P.DN renamed USB_OTG_P.DM
Other:
- sheet ANALOG VTX renamed UART_I2C
- removed sheet DIGITAL VTX
- removed sheet I2C1|SPI3
- removed sheet MOTORS[5-8]
- removed sheet RC INPUT
- sheet MCU ports: added none; removed ADC_CURR2, I2C1{I2C}, MOTOR[5..8], SPI3{SPI}
- sheet SENSORS ports: added I2C1{I2C}; removed none
- sheet UART_I2C: file ANALOG_VTX.kicad_sch -> UART_I2C.kicad_sch
- sheet UART_I2C ports: added UART2{UART}, UART3{UART}, UART4{UART}, UART6{UART}, UART7{UART}; removed SPI2{SPI}
