File: RC_INPUT.kicad_sch (KiCad schematic)
At the start: 1 part, among them U8 ZX-SH1.0-4PWT

Commit message: Remove unused file
Parts:
- removed U8: ZX-SH1.0-4PWT, EasyEDA:CONN-SMD_4P-P1.00_MEGASTAR_ZX-SH1.0-4PWT, symbol EasyEDA:ZX-SH1.0-4PWT
Other:
- note removed: "RX_PPM"
