File: untitled.kicad_sch (KiCad schematic)
At the start: 10 parts, among them J11 Conn_01x04

Commit message: upsadte SPI4 set to Baro
Other:
- title: (none) -> H743_ARDUPILOT
Changed lines of the file:
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@@
 	(generator "eeschema")
 	(generator_version "10.0")
-	(paper "A4")
+	(paper "A3")
 	(title_block
+		(title "H743_ARDUPILOT")
 		(date "2026-09-24")
 	)
