File: CAN.kicad_sch (KiCad schematic)
At the start: 7 parts, among them U12 SIT1051TK/3, U13 ZX-SH1.0-4PWT

Commit message: Remove unused file
Parts:
- removed JP1: SolderJumper_2_Open, _pico:SolderJumper_Mini, symbol Jumper:SolderJumper_2_Open
- removed R24: 120R, Resistor_SMD:R_0402_1005Metric, symbol Device:R_Small
Changed lines of the file:
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@@
-	)
-	(junction
-		(at 120.65 72.39)
-		(diameter 0)
-		(color 0 0 0 0)
 	)
 	(junction
@@
 		(color 0 0 0 0)
 	)
-	(junction
-		(at 120.65 59.69)
-		(diameter 0)
-		(color 0 0 0 0)
-	)
 	(bus_entry
 		(at 31.75 34.29)
@@
 	(wire
 		(pts
-			(xy 120.65 59.69) (xy 133.35 59.69)
+			(xy 114.3 59.69) (xy 133.35 59.69)
 		)
 		(stroke
@@
 	(wire
 		(pts
-			(xy 114.3 59.69) (xy 120.65 59.69)
-		)
-		(stroke
-			(width 0)
-			(type default)
-		)
-	)
-	(wire
-		(pts
 			(xy 148.59 60.96) (xy 149.86 60.96)
 		)
@@
 	(wire
 		(pts
-			(xy 120.65 72.39) (xy 128.27 72.39)
+			(xy 114.3 72.39) (xy 128.27 72.39)
 		)
 		(stroke
@@
 		(pts
 			(xy 76.2 69.85) (xy 88.9 69.85)
-		)
-		(stroke
-			(width 0)
-			(type default)
-		)
-	)
-	(wire
-		(pts
-			(xy 114.3 72.39) (xy 120.65 72.39)
 		)
 		(stroke
@@
 				(path "/6b768b36-fce6-4be0-9021-6d41bddc3a70/339be1e4-df07-445e-a0aa-e25cab3c571c"
 					(reference "C40")
-					(unit 1)
-				)
-			)
-		)
-	)
-	(symbol
-		(lib_id "Jumper:SolderJumper_2_Open")
-		(at 120.65 68.58 90)
-		(unit 1)
-		(body_style 1)
-		(exclude_from_sim no)
-		(in_bom no)
-		(on_board yes)
-		(in_pos_files no)
-		(dnp no)
-		(property "Reference" "JP1"
-			(at 124.46 68.58 90)
-			(show_name no)
-			(do_not_autoplace no)
-			(effects
-				(font
-					(size 1.016 1.016)
-				)
-			)
-		)
-		(property "Value" "SolderJumper_2_Open"
-			(at 116.84 68.58 0)
-			(hide yes)
-			(show_name no)
-			(do_not_autoplace no)
-			(effects
-				(font
-					(size 1.27 1.27)
-				)
-			)
-		)
-		(property "Footprint" "_pico:SolderJumper_Mini"
-			(at 120.65 68.58 0)
-			(hide yes)
-			(show_name no)
-			(do_not_autoplace no)
-			(effects
-				(font
-					(size 1.27 1.27)
-				)
-			)
-		)
-		(property "Datasheet" "~"
-			(at 120.65 68.58 0)
-			(hide yes)
-			(show_name no)
-			(do_not_autoplace no)
-			(effects
-				(font
-					(size 1.27 1.27)
-				)
-			)
-		)
-		(property "Description" "Solder Jumper, 2-pole, open"
-			(at 120.65 68.58 0)
-			(hide yes)
-			(show_name no)
-			(do_not_autoplace no)
-			(effects
-				(font
-					(size 1.27 1.27)
-				)
-			)
-		)
-		(pin "2"
-		)
-		(pin "1"
-		)
-		(instances
-			(project "LEVIA_H7"
-				(path "/6b768b36-fce6-4be0-9021-6d41bddc3a70/339be1e4-df07-445e-a0aa-e25cab3c571c"
-					(reference "JP1")
 					(unit 1)
 				)
@@
 					(unit 1)
 				)
-			)
-		)
-	)
-	(symbol
-		(lib_id "Device:R_Small")
-		(at 120.65 62.23 0)
-		(unit 1)
-		(body_style 1)
-		(exclude_from_sim no)
-		(in_bom yes)
-		(on_board yes)
-		(in_pos_files yes)
-		(dnp no)
-		(fields_autoplaced yes)
-		(property "Reference" "R24"
-			(at 123.19 60.9599 0)
-			(show_name no)
-			(do_not_autoplace no)
-			(effects
-				(font
-					(size 1.016 1.016)
-				)
-				(justify left)
-			)
-		)
-		(property "Value" "120R"
-			(at 123.19 63.4999 0)
-			(show_name no)
-			(do_not_autoplace no)
-			(effects
-				(font
-					(size 1.016 1.016)
-				)
-				(justify left)
-			)
-		)
-		(property "Footprint" "Resistor_SMD:R_0402_1005Metric"
-			(at 120.65 62.23 0)
-			(hide yes)
-			(show_name no)
-			(do_not_autoplace no)
-			(effects
-				(font
-					(size 1.27 1.27)
-				)
-			)
-		)
-		(property "Datasheet" ""
-			(at 120.65 62.23 0)
-			(hide yes)
-			(show_name no)
-			(do_not_autoplace no)
-			(effects
-				(font
-					(size 1.27 1.27)
-				)
-			)
-		)
-		(property "Description" "Resistor, small symbol"
-			(at 120.65 62.23 0)
-			(hide yes)
-			(show_name no)
-			(do_not_autoplace no)
-			(effects
-				(font
-					(size 1.27 1.27)
-				)
-			)
-		)
-		(property "LCSC Part" "C25079"
-			(at 120.65 62.23 0)
-			(hide yes)
-			(show_name no)
-			(do_not_autoplace no)
-			(effects
-				(font
-					(size 1.27 1.27)
-				)
-			)
-		)
-		(property "LCSC" "C25079"
-			(at 120.65 62.23 0)
-			(hide yes)
-			(show_name no)
-			(do_not_autoplace no)
-			(effects
-				(font
-					(size 1.27 1.27)
-				)
-			)
-		)
-		(property "MPN" "0402WGF1200TCE"
-			(at 120.65 62.23 0)
-			(hide yes)
-			(show_name no)
-			(do_not_autoplace no)
-			(effects
-				(font
-					(size 1.27 1.27)
-				)
-			)
-		)
-		(property "Manufacturer" "UNI-ROYAL(Uniroyal Elec)"
-			(at 120.65 62.23 0)
-			(hide yes)
-			(show_name no)
-			(do_not_autoplace no)
-			(effects
-				(font
-					(size 1.27 1.27)
-				)
-			)
-		)
-		(pin "2"
-		)
-		(pin "1"
-		)
-		(instances
-			(project "LEVIA_H7"
-				(path "/6b768b36-fce6-4be0-9021-6d41bddc3a70/339be1e4-df07-445e-a0aa-e25cab3c571c"
-					(reference "R24")
-					(unit 1)
-				)

Commit message: update name
Other:
- note removed: "CAN"
- company: Pierluigi Colangeli, PhD -> (none)
- title: LEVIA H7 -> (none)

Commit message: upsadte SPI4 set to Baro
Other:
- title: (none) -> H743_ARDUPILOT
Changed lines of the file:
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@@
 	(generator "eeschema")
 	(generator_version "10.0")
-	(paper "A5")
+	(paper "A3")
 	(title_block
+		(title "H743_ARDUPILOT")
 		(date "2026-09-24")
 	)

Commit message: re annotate componant globaly
Parts:
- renumbered C39 to C25, C40 to C26, D6 to D2, U12 to U3, U13 to U4
Changed lines of the file:
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@@
 		(in_pos_files yes)
 		(dnp no)
-		(property "Reference" "C40"
+		(property "Reference" "C26"
 			(at 71.12 63.5 0)
 			(show_name no)
@@
 			(project "H743_Ardupilot"
 				(path "/6b768b36-fce6-4be0-9021-6d41bddc3a70/339be1e4-df07-445e-a0aa-e25cab3c571c"
-					(reference "C40")
+					(reference "C26")
 					(unit 1)
 				)
@@
 		(dnp no)
 		(fields_autoplaced yes)
-		(property "Reference" "#PWR084"
+		(property "Reference" "#PWR053"
 			(at 69.85 59.69 0)
 			(hide yes)
@@
 			(project "H743_Ardupilot"
 				(path "/6b768b36-fce6-4be0-9021-6d41bddc3a70/339be1e4-df07-445e-a0aa-e25cab3c571c"
-					(reference "#PWR084")
+					(reference "#PWR053")
 					(unit 1)
 				)
@@
 		(dnp no)
 		(fields_autoplaced yes)
-		(property "Reference" "#PWR087"
+		(property "Reference" "#PWR057"
 			(at 148.59 60.96 0)
 			(hide yes)
@@
 			(project "H743_Ardupilot"
 				(path "/6b768b36-fce6-4be0-9021-6d41bddc3a70/339be1e4-df07-445e-a0aa-e25cab3c571c"
-					(reference "#PWR087")
+					(reference "#PWR057")
 					(unit 1)
 				)
@@
 		(dnp no)
 		(fields_autoplaced yes)
-		(property "Reference" "#PWR086"
+		(property "Reference" "#PWR055"
 			(at 100.33 87.63 0)
 			(hide yes)
@@
 			(project "H743_Ardupilot"
 				(path "/6b768b36-fce6-4be0-9021-6d41bddc3a70/339be1e4-df07-445e-a0aa-e25cab3c571c"
-					(reference "#PWR086")
+					(reference "#PWR055")
 					(unit 1)
 				)
@@
 		(dnp no)
 		(fields_autoplaced yes)
-		(property "Reference" "#PWR083"
+		(property "Reference" "#PWR052"
 			(at 64.77 76.2 0)
 			(hide yes)
@@
 			(project "H743_Ardupilot"
 				(path "/6b768b36-fce6-4be0-9021-6d41bddc3a70/339be1e4-df07-445e-a0aa-e25cab3c571c"
-					(reference "#PWR083")
+					(reference "#PWR052")
 					(unit 1)
 				)
@@
 		(in_pos_files yes)
 		(dnp no)
-		(property "Reference" "C39"
+		(property "Reference" "C25"
 			(at 66.04 63.5 0)
 			(show_name no)
@@
 			(project "H743_Ardupilot"
 				(path "/6b768b36-fce6-4be0-9021-6d41bddc3a70/339be1e4-df07-445e-a0aa-e25cab3c571c"
-					(reference "C39")
+					(reference "C25")
 					(unit 1)
 				)
@@
 		(dnp no)
 		(fields_autoplaced yes)
-		(property "Reference" "#PWR082"
+		(property "Reference" "#PWR051"
 			(at 64.77 64.77 0)
 			(hide yes)
@@
 			(project "H743_Ardupilot"
 				(path "/6b768b36-fce6-4be0-9021-6d41bddc3a70/339be1e4-df07-445e-a0aa-e25cab3c571c"
-					(reference "#PWR082")
+					(reference "#PWR051")
 					(unit 1)
 				)
@@
 		(dnp no)
 		(fields_autoplaced yes)
-		(property "Reference" "#PWR0124"
+		(property "Reference" "#PWR056"
 			(at 130.81 100.33 0)
 			(hide yes)
@@
 			(project "H743_Ardupilot"
 				(path "/6b768b36-fce6-4be0-9021-6d41bddc3a70/339be1e4-df07-445e-a0aa-e25cab3c571c"
-					(reference "#PWR0124")
+					(reference "#PWR056")
 					(unit 1)
 				)
@@
 		(dnp no)
 		(fields_autoplaced yes)
-		(property "Reference" "U12"
+		(property "Reference" "U3"
 			(at 101.6 49.53 0)
 			(show_name no)
@@
 			(project "H743_Ardupilot"
 				(path "/6b768b36-fce6-4be0-9021-6d41bddc3a70/339be1e4-df07-445e-a0aa-e25cab3c571c"
-					(reference "U12")
+					(reference "U3")
 					(unit 1)
 				)
@@
 		(dnp no)
 		(fields_autoplaced yes)
-		(property "Reference" "D6"
+		(property "Reference" "D2"
 			(at 137.16 84.3914 90)
 			(show_name no)
@@
 			(project "H743_Ardupilot"
 				(path "/6b768b36-fce6-4be0-9021-6d41bddc3a70/339be1e4-df07-445e-a0aa-e25cab3c571c"
-					(reference "D6")
+					(reference "D2")
 					(unit 1)
 				)
@@
 		(in_pos_files yes)
 		(dnp no)
-		(property "Reference" "U13"
+		(property "Reference" "U4"
 			(at 151.13 55.88 0)
 			(show_name no)
@@
 			(project "H743_Ardupilot"
 				(path "/6b768b36-fce6-4be0-9021-6d41bddc3a70/339be1e4-df07-445e-a0aa-e25cab3c571c"
-					(reference "U13")
+					(reference "U4")
 					(unit 1)
 				)
@@
 		(dnp no)
 		(fields_autoplaced yes)
-		(property "Reference" "#PWR088"
+		(property "Reference" "#PWR058"
 			(at 148.59 82.55 0)
 			(hide yes)
@@
 			(project "H743_Ardupilot"
 				(path "/6b768b36-fce6-4be0-9021-6d41bddc3a70/339be1e4-df07-445e-a0aa-e25cab3c571c"
-					(reference "#PWR088")
+					(reference "#PWR058")
 					(unit 1)
 				)
@@
 		(dnp no)
 		(fields_autoplaced yes)
-		(property "Reference" "#PWR085"
+		(property "Reference" "#PWR054"
 			(at 69.85 76.2 0)
 			(hide yes)
@@
 			(project "H743_Ardupilot"
 				(path "/6b768b36-fce6-4be0-9021-6d41bddc3a70/339be1e4-df07-445e-a0aa-e25cab3c571c"
-					(reference "#PWR085")
+					(reference "#PWR054")
 					(unit 1)
 				)

Commit message: audit DigiKey metadata: CAN.kicad_sch
Parts:
- C25, C26: DigiKey Part Number (none) -> 1276-1001-1-ND; DigiKey Price Qty (none) -> 1 CT; DigiKey Specs (none) -> 100 nF ±10%, 16 V, X7R, 0402; DigiKey Status (none) -> Active; DigiKey URL (none) -> https://www.digikey.fr/fr/products/detail/samsung-electro-m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; DigiKey Unit Price EUR (none) -> 0.09; Footprint Audit (none) -> OK; LCSC C1525 -> (none); LCSC Part C1525 -> (none); Library Audit (none) -> KiCad standard; MPN GRM022R60J104KE15D -> CL05B104KO5NNNC; Manufacturer Murata Electronics -> Samsung Electro-Mechanics; Package (none) -> 0402 (1005); Price Checked (none) -> 2026-09-25
- D2: DigiKey Part Number (none) -> 1727-PESD2CANFD24V-CT-ND; DigiKey Price Qty (none) -> 1 CT; DigiKey Specs (none) -> Dual CAN TVS, 24 V standoff, 42 V clamp, 5.2 pF, SOT-23; DigiKey Status (none) -> Active; DigiKey URL (none) -> https://www.digikey.fr/en/products/detail/nexperia-usa-inc/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; DigiKey Unit Price EUR (none) -> 0.40; Footprint Audit (none) -> OK; Library Audit (none) -> Custom symbol + KiCad footprint; Package (none) -> SOT-23 / TO-236AB; Price Checked (none) -> 2026-09-25
- U3: value SIT1051TK/3 -> TJA1051TK/3,118; DigiKey Part Number (none) -> 568-8686-1-ND; DigiKey Price Qty (none) -> 1 CT; DigiKey Specs (none) -> CAN 5 Mbps, 4.5–5.5 V, 8-HVSON 3x3; DigiKey Status (none) -> Last Time Buy; DigiKey last availability 2026-12-26; DigiKey URL (none) -> https://www.digikey.fr/fr/products/detail/nxp-usa-inc/TJA10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; DigiKey Unit Price EUR (none) -> 1.65; Footprint Audit (none) -> OK; Library Audit (none) -> EasyEDA; Manufacturer NXP(恩智浦) -> NXP USA Inc.; Package (none) -> 8-HVSON 3x3 EP; Price Checked (none) -> 2026-09-25
- U4: DigiKey Specs (none) -> SH 1.0 mm, 4P right-angle SMD, 1 A, 50 V; DigiKey Status (none) -> No exact DigiKey listing; supplier part retained; Footprint Audit (none) -> OK against Megastar drawing; Library Audit (none) -> EasyEDA; Manufacturer Megastar(兆星) -> Megastar; Package (none) -> SH1.0 4P right-angle SMD; Price Checked (none) -> 2026-09-25
