File: CAN.kicad_sch (KiCad schematic)
At the start: 5 parts, among them U3 TJA1051TK/3,118, U4 ZX-SH1.0-4PWT

Commit message: update
Parts:
- renumbered C25 to C42, C26 to C43, D2 to D5, U3 to U7, U4 to U8
Changed lines of the file:
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@@
 		(in_pos_files yes)
 		(dnp no)
-		(property "Reference" "C26"
+		(property "Reference" "C43"
 			(at 71.12 63.5 0)
 			(show_name no)
@@
 			(project "H743_Ardupilot"
 				(path "/6b768b36-fce6-4be0-9021-6d41bddc3a70/339be1e4-df07-445e-a0aa-e25cab3c571c"
-					(reference "C26")
+					(reference "C43")
 					(unit 1)
 				)
@@
 		(dnp no)
 		(fields_autoplaced yes)
-		(property "Reference" "#PWR053"
+		(property "Reference" "#PWR082"
 			(at 69.85 59.69 0)
 			(hide yes)
@@
 			(project "H743_Ardupilot"
 				(path "/6b768b36-fce6-4be0-9021-6d41bddc3a70/339be1e4-df07-445e-a0aa-e25cab3c571c"
-					(reference "#PWR053")
+					(reference "#PWR082")
 					(unit 1)
 				)
@@
 		(dnp no)
 		(fields_autoplaced yes)
-		(property "Reference" "#PWR057"
+		(property "Reference" "#PWR086"
 			(at 148.59 60.96 0)
 			(hide yes)
@@
 			(project "H743_Ardupilot"
 				(path "/6b768b36-fce6-4be0-9021-6d41bddc3a70/339be1e4-df07-445e-a0aa-e25cab3c571c"
-					(reference "#PWR057")
+					(reference "#PWR086")
 					(unit 1)
 				)
@@
 		(dnp no)
 		(fields_autoplaced yes)
-		(property "Reference" "#PWR055"
+		(property "Reference" "#PWR084"
 			(at 100.33 87.63 0)
 			(hide yes)
@@
 			(project "H743_Ardupilot"
 				(path "/6b768b36-fce6-4be0-9021-6d41bddc3a70/339be1e4-df07-445e-a0aa-e25cab3c571c"
-					(reference "#PWR055")
+					(reference "#PWR084")
 					(unit 1)
 				)
@@
 		(dnp no)
 		(fields_autoplaced yes)
-		(property "Reference" "#PWR052"
+		(property "Reference" "#PWR081"
 			(at 64.77 76.2 0)
 			(hide yes)
@@
 			(project "H743_Ardupilot"
 				(path "/6b768b36-fce6-4be0-9021-6d41bddc3a70/339be1e4-df07-445e-a0aa-e25cab3c571c"
-					(reference "#PWR052")
+					(reference "#PWR081")
 					(unit 1)
 				)
@@
 		(in_pos_files yes)
 		(dnp no)
-		(property "Reference" "C25"
+		(property "Reference" "C42"
 			(at 66.04 63.5 0)
 			(show_name no)
@@
 			(project "H743_Ardupilot"
 				(path "/6b768b36-fce6-4be0-9021-6d41bddc3a70/339be1e4-df07-445e-a0aa-e25cab3c571c"
-					(reference "C25")
+					(reference "C42")
 					(unit 1)
 				)
@@
 		(dnp no)
 		(fields_autoplaced yes)
-		(property "Reference" "#PWR051"
+		(property "Reference" "#PWR080"
 			(at 64.77 64.77 0)
 			(hide yes)
@@
 			(project "H743_Ardupilot"
 				(path "/6b768b36-fce6-4be0-9021-6d41bddc3a70/339be1e4-df07-445e-a0aa-e25cab3c571c"
-					(reference "#PWR051")
+					(reference "#PWR080")
 					(unit 1)
 				)
@@
 		(dnp no)
 		(fields_autoplaced yes)
-		(property "Reference" "#PWR056"
+		(property "Reference" "#PWR085"
 			(at 130.81 100.33 0)
 			(hide yes)
@@
 			(project "H743_Ardupilot"
 				(path "/6b768b36-fce6-4be0-9021-6d41bddc3a70/339be1e4-df07-445e-a0aa-e25cab3c571c"
-					(reference "#PWR056")
+					(reference "#PWR085")
 					(unit 1)
 				)
@@
 		(dnp no)
 		(fields_autoplaced yes)
-		(property "Reference" "U3"
+		(property "Reference" "U7"
 			(at 101.6 49.53 0)
 			(show_name no)
@@
 			(project "H743_Ardupilot"
 				(path "/6b768b36-fce6-4be0-9021-6d41bddc3a70/339be1e4-df07-445e-a0aa-e25cab3c571c"
-					(reference "U3")
+					(reference "U7")
 					(unit 1)
 				)
@@
 		(dnp no)
 		(fields_autoplaced yes)
-		(property "Reference" "D2"
+		(property "Reference" "D5"
 			(at 137.16 84.3914 90)
 			(show_name no)
@@
 			(project "H743_Ardupilot"
 				(path "/6b768b36-fce6-4be0-9021-6d41bddc3a70/339be1e4-df07-445e-a0aa-e25cab3c571c"
-					(reference "D2")
+					(reference "D5")
 					(unit 1)
 				)
@@
 		(in_pos_files yes)
 		(dnp no)
-		(property "Reference" "U4"
+		(property "Reference" "U8"
 			(at 151.13 55.88 0)
 			(show_name no)
@@
 			(project "H743_Ardupilot"
 				(path "/6b768b36-fce6-4be0-9021-6d41bddc3a70/339be1e4-df07-445e-a0aa-e25cab3c571c"
-					(reference "U4")
+					(reference "U8")
 					(unit 1)
 				)
@@
 		(dnp no)
 		(fields_autoplaced yes)
-		(property "Reference" "#PWR058"
+		(property "Reference" "#PWR087"
 			(at 148.59 82.55 0)
 			(hide yes)
@@
 			(project "H743_Ardupilot"
 				(path "/6b768b36-fce6-4be0-9021-6d41bddc3a70/339be1e4-df07-445e-a0aa-e25cab3c571c"
-					(reference "#PWR058")
+					(reference "#PWR087")
 					(unit 1)
 				)
@@
 		(dnp no)
 		(fields_autoplaced yes)
-		(property "Reference" "#PWR054"
+		(property "Reference" "#PWR083"
 			(at 69.85 76.2 0)
 			(hide yes)
@@
 			(project "H743_Ardupilot"
 				(path "/6b768b36-fce6-4be0-9021-6d41bddc3a70/339be1e4-df07-445e-a0aa-e25cab3c571c"
-					(reference "#PWR054")
+					(reference "#PWR083")
 					(unit 1)
 				)

Commit message: update pcb
Parts:
- U8: footprint EasyEDA:CONN-SMD_4P-P1.00_MEGASTAR_ZX-SH1.0-4PWT -> Connector_JST:JST_GH_SM05B-GHS-TB_1x05-1MP_P1.25mm_Horizontal
Changed lines of the file:
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@@
 			)
 		)
-		(property "Footprint" "EasyEDA:CONN-SMD_4P-P1.00_MEGASTAR_ZX-SH1.0-4PWT"
+		(property "Footprint" "Connector_JST:JST_GH_SM05B-GHS-TB_1x05-1MP_P1.25mm_Horizontal"
 			(at 154.94 81.28 0)
 			(hide yes)

Commit message: Migrate SM04B-GHS-TB(LF)(SN) to verified JST symbol and footprint
Parts:
- U7: Library Audit EasyEDA -> Project-local symbol + verified JST footprint
- U8: value ZX-SH1.0-4PWT -> SM04B-GHS-TB(LF)(SN); footprint Connector_JST:JST_GH_SM05B-GHS-TB_1x05-1MP_P1.25mm_Horizontal -> H743_Custom:JST_GH_SM04B-GHS-TB_1x04_P1.25mm_Horizontal_GNDtabs; symbol EasyEDA:ZX-SH1.0-4PWT -> H743_Ardupilot:JST_GH_SM04B_GHS_TB_4P; Footprint Audit OK against Megastar drawing -> OK against JST drawing; Library Audit EasyEDA -> Project-local symbol + verified JST footprint; MPN ZX-SH1.0-4PWT -> SM04B-GHS-TB(LF)(SN); Manufacturer Megastar -> JST
Changed lines of the file:
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@@
 			)
 		)
-		(property "Library Audit" "EasyEDA"
+		(property "Library Audit" "Project-local symbol + verified JST footprint"
 			(at 101.6 49.53 0)
 			(hide yes)
@@
 	)
 	(symbol
-		(lib_id "EasyEDA:ZX-SH1.0-4PWT")
+		(lib_id "H743_Ardupilot:JST_GH_SM04B_GHS_TB_4P")
 		(at 154.94 64.77 0)
 		(unit 1)
@@
 			)
 		)
-		(property "Value" "ZX-SH1.0-4PWT"
+		(property "Value" "SM04B-GHS-TB(LF)(SN)"
 			(at 161.29 66.0399 0)
 			(hide yes)
@@
 			)
 		)
-		(property "Footprint" "Connector_JST:JST_GH_SM05B-GHS-TB_1x05-1MP_P1.25mm_Horizontal"
+		(property "Footprint" "H743_Custom:JST_GH_SM04B-GHS-TB_1x04_P1.25mm_Horizontal_GNDtabs"
 			(at 154.94 81.28 0)
 			(hide yes)
@@
 			)
 		)
-		(property "Datasheet" "https://xonstorage.z8.web.core.windows.net/pdf/megastar_zxsh104pwt_apr22_xonlink.pdf"
+		(property "Datasheet" "https://www.jst-mfg.com/product/pdf/eng/eGH.pdf"
 			(at 154.94 83.82 0)
 			(hide yes)
@@
 			)
 		)
-		(property "Manufacturer" "Megastar"
+		(property "Manufacturer" "JST"
 			(at 154.94 86.36 0)
 			(hide yes)
@@
 			)
 		)
-		(property "MPN" "ZX-SH1.0-4PWT"
+		(property "MPN" "SM04B-GHS-TB(LF)(SN)"
 			(at 154.94 88.9 0)
 			(hide yes)
@@
 			)
 		)
-		(property "Footprint Audit" "OK against Megastar drawing"
-			(at 151.13 55.88 0)
-			(hide yes)
-			(show_name no)
-			(do_not_autoplace no)
-			(effects
-				(font
-					(size 1.27 1.27)
-				)
-			)
-		)
-		(property "Library Audit" "EasyEDA"
-			(at 151.13 55.88 0)
-			(hide yes)
+		(property "Footprint Audit" "OK against JST drawing"
+			(at 151.13 55.88 0)
+			(hide yes)
+			(show_name no)
+			(do_not_autoplace no)
+			(effects
+				(font
+					(size 1.27 1.27)
+				)
+			)
+		)
+		(property "Library Audit" "Project-local symbol + verified JST footprint"
+			(at 151.13 55.88 0)
+			(hide yes)

Commit message: Verify CAN transceiver and TVS symbol-footprint mappings
Parts:
- C42, C43: Footprint Audit OK -> VERIFIED: NXP HVSON8 SOT782-1, 3x3 mm, P0.65, EP 1.6x2.4; s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
- D5: footprint PCM_Package_TO_SOT_SMD_AKL:SOT-23 -> Package_TO_SOT_SMD:SOT-23; Footprint Audit OK -> VERIFIED: NXP HVSON8 SOT782-1, 3x3 mm, P0.65, EP 1.6x2.4; s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; Library Audit Custom symbol + KiCad footprint -> Custom verified symbol + KiCad standard SOT-23 footprint; Mouser URL (none) -> https://www.mouser.fr/fr/ProductDetail/Nexperia/PESD2CANFD2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; Supplier Specs (none) -> Automotive CAN TVS, VRWM 24 V, VCL 42 V, SOT-23/TO-236AB, A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
- U7: footprint EasyEDA:HVSON-8_L3.0-W3.0-P0.65-BL-EP -> Package_SON:HVSON-8-1EP_3x3mm_P0.65mm_EP1.6x2.4mm; symbol EasyEDA:TJA1051TK_3,118 -> Interface_CAN_LIN:TJA1051TK-3; Farnell URL (none) -> https://fr.farnell.com/nxp/tja1051tk-3-118/can-fd-transceiv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; Footprint Audit OK -> VERIFIED: NXP HVSON8 SOT782-1, 3x3 mm, P0.65, EP 1.6x2.4; s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; Mouser URL (none) -> https://eu.mouser.com/en/ProductDetail/NXP-Semiconductors/T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; RS URL (none) -> https://ch.rs-online.com/web/p/can-schnittstellen-ics/21946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; Supplier Specs (none) -> CAN FD transceiver, 5 Mbps, 4.5-5.5 V, HVSON-8 3x3 mm, -40.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
Changed lines of the file:
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@@
 			)
 		)
-		(property "Footprint Audit" "OK"
+		(property "Footprint Audit" "VERIFIED: NXP HVSON8 SOT782-1, 3x3 mm, P0.65, EP 1.6x2.4; symbol pin 9 EP/GND matches exposed pad"
 			(at 71.12 63.5 0)
 			(hide yes)
@@
 			)
 		)
-		(property "Footprint Audit" "OK"
+		(property "Footprint Audit" "VERIFIED: NXP HVSON8 SOT782-1, 3x3 mm, P0.65, EP 1.6x2.4; symbol pin 9 EP/GND matches exposed pad"
 			(at 66.04 63.5 0)
 			(hide yes)
@@
 	)
 	(symbol
-		(lib_id "EasyEDA:TJA1051TK_3,118")
+		(lib_id "Interface_CAN_LIN:TJA1051TK-3")
 		(at 101.6 66.04 0)
 		(unit 1)
@@
 			)
 		)
-		(property "Footprint" "EasyEDA:HVSON-8_L3.0-W3.0-P0.65-BL-EP"
+		(property "Footprint" "Package_SON:HVSON-8-1EP_3x3mm_P0.65mm_EP1.6x2.4mm"
 			(at 101.6 83.82 0)
 			(hide yes)
@@
 			)
 		)
+		(property "Supplier Specs" "CAN FD transceiver, 5 Mbps, 4.5-5.5 V, HVSON-8 3x3 mm, -40..150 C"
+			(at 101.6 91.44 0)
+			(hide yes)
+			(show_name no)
+			(do_not_autoplace no)
+			(effects (font (size 1.27 1.27)))
+		)
+		(property "RS URL" "https://ch.rs-online.com/web/p/can-schnittstellen-ics/2194675"
+			(at 101.6 91.44 0)
+			(hide yes)
+			(show_name no)
+			(do_not_autoplace no)
+			(effects (font (size 1.27 1.27)))
+		)
+		(property "Farnell URL" "https://fr.farnell.com/nxp/tja1051tk-3-118/can-fd-transceiver-5mbps-hvson/dp/2776121"
+			(at 101.6 91.44 0)
+			(hide yes)
+			(show_name no)
+			(do_not_autoplace no)
+			(effects (font (size 1.27 1.27)))
+		)
+		(property "Mouser URL" "https://eu.mouser.com/en/ProductDetail/NXP-Semiconductors/TJA1051TK-3118"
+			(at 101.6 91.44 0)
+			(hide yes)
+			(show_name no)
+			(do_not_autoplace no)
+			(effects (font (size 1.27 1.27)))
+		)
 		(property "LCSC Part" "C124020"
 			(at 101.6 93.98 0)
@@
 			)
 		)
-		(property "Footprint Audit" "OK"
+		(property "Footprint Audit" "VERIFIED: NXP HVSON8 SOT782-1, 3x3 mm, P0.65, EP 1.6x2.4; symbol pin 9 EP/GND matches exposed pad"
 			(at 101.6 49.53 0)
 			(hide yes)
@@
 			)
 		)
-		(property "Footprint" "PCM_Package_TO_SOT_SMD_AKL:SOT-23"
+		(property "Footprint" "Package_TO_SOT_SMD:SOT-23"
 			(at 121.92 85.09 0)
 			(hide yes)
@@
 			)
 		)
-		(property "Datasheet" "https://www.tme.eu/Document/ad02fbf39ace74a5161accc984238198/PESD2CAN.pdf"
+		(property "Datasheet" "https://assets.nexperia.com/documents/data-sheet/PESD2CANFD24V.pdf"
 			(at 121.92 85.09 0)
 			(hide yes)
@@
 			)
 		)
+		(property "Supplier Specs" "Automotive CAN TVS, VRWM 24 V, VCL 42 V, SOT-23/TO-236AB, AEC-Q101"
+			(at 130.81 85.09 90)
+			(hide yes)
+			(show_name no)
+			(do_not_autoplace no)
+			(effects (font (size 1.27 1.27)))
+		)
+		(property "Mouser URL" "https://www.mouser.fr/fr/ProductDetail/Nexperia/PESD2CANFD24V-TR"
+			(at 130.81 85.09 90)
+			(hide yes)
+			(show_name no)
+			(do_not_autoplace no)
+			(effects (font (size 1.27 1.27)))
+		)
 		(property "Manufacturer" "Nexperia"
 			(at 130.81 85.09 90)
@@
 			)
 		)
-		(property "Footprint Audit" "OK"
+		(property "Footprint Audit" "VERIFIED: NXP HVSON8 SOT782-1, 3x3 mm, P0.65, EP 1.6x2.4; symbol pin 9 EP/GND matches exposed pad"
 			(at 137.16 84.3914 90)
 			(hide yes)
@@
 			)
 		)
-		(property "Library Audit" "Custom symbol + KiCad footprint"
+		(property "Library Audit" "Custom verified symbol + KiCad standard SOT-23 footprint"
 			(at 137.16 84.3914 90)
 			(hide yes)

Commit message: update pcb
Parts:
- added J13: Can1_2, H743_Custom:SolderPadArray_1x04_P2.54mm_1x1mm, symbol Connector_Generic:Conn_01x04
- added J14: Can1_1, H743_Custom:SolderPadArray_1x04_P2.54mm_1x1mm, symbol Connector_Generic:Conn_01x04
Connections:
- net +5V_SYS: now also J13.1 (Pin_1), J14.1 (Pin_1)
- net CAN1_H: now also J13.2 (Pin_2), J14.2 (Pin_2)
- net CAN1_L: now also J13.3 (Pin_3), J14.3 (Pin_3)
- net GND: now also J13.4 (Pin_4), J14.4 (Pin_4)

Commit message: Review component footprints, restore local libraries and reconcile PCB pads
Parts:
- C42, C43: symbol Device:C_Small -> FC01_Project:CAN__C_Small; Footprint Audit VERIFIED: NXP HVSON8 SOT782-1, 3x3 mm, P0.65, EP 1.6x2.4; s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 -> See verification/COMPONENTS.csv and verification/REPORT.md; Library Audit KiCad standard -> See verification/COMPONENTS.csv and verification/REPORT.md
- D5: symbol PCM_Diode_TVS_AKL:PESD2CAN -> FC01_Project:CAN__PESD2CAN; Footprint Audit VERIFIED: NXP HVSON8 SOT782-1, 3x3 mm, P0.65, EP 1.6x2.4; s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 -> See verification/COMPONENTS.csv and verification/REPORT.md; Library Audit Custom verified symbol + KiCad standard SOT-23 footprint -> See verification/COMPONENTS.csv and verification/REPORT.md
- J13, J14: symbol Connector_Generic:Conn_01x04 -> FC01_Project:CAN__Conn_01x04; Footprint Audit OK: 4 square SMD pads 1.00x1.00 mm, P2.54 mm, no holes, no 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 -> See verification/COMPONENTS.csv and verification/REPORT.md; Library Audit Project-local H743_Custom footprint -> See verification/COMPONENTS.csv and verification/REPORT.md
- U7: symbol Interface_CAN_LIN:TJA1051TK-3 -> FC01_Project:CAN__TJA1051TK-3; Footprint Audit VERIFIED: NXP HVSON8 SOT782-1, 3x3 mm, P0.65, EP 1.6x2.4; s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 -> See verification/COMPONENTS.csv and verification/REPORT.md; Library Audit Project-local symbol + verified JST footprint -> See verification/COMPONENTS.csv and verification/REPORT.md
- U8: symbol H743_Ardupilot:JST_GH_SM04B_GHS_TB_4P -> FC01_Project:CAN__JST_GH_SM04B_GHS_TB_4P; Footprint Audit OK against JST drawing -> See verification/COMPONENTS.csv and verification/REPORT.md; Library Audit Project-local symbol + verified JST footprint -> See verification/COMPONENTS.csv and verification/REPORT.md; Package SH1.0 4P right-angle SMD -> JST GH 4 contacts, P1.25 mm, side entry; mounting tabs pads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
Changed lines of the file:
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@@
 	)
 	(symbol
-		(lib_id "Connector_Generic:Conn_01x04")
+		(lib_id "FC01_Project:CAN__Conn_01x04")
 		(at 162.56 106.68 0)
 		(unit 1)
@@
 			)
 		)
-		(property "Footprint Audit" "OK: 4 square SMD pads 1.00x1.00 mm, P2.54 mm, no holes, no paste"
+		(property "Footprint Audit" "See verification/COMPONENTS.csv and verification/REPORT.md"
 			(at 165.1 106.6799 0)
 			(hide yes)
@@
 			)
 		)
-		(property "Library Audit" "Project-local H743_Custom footprint"
+		(property "Library Audit" "See verification/COMPONENTS.csv and verification/REPORT.md"
 			(at 165.1 106.6799 0)
 			(hide yes)
@@
 	)
 	(symbol
-		(lib_id "Device:C_Small")
+		(lib_id "FC01_Project:CAN__C_Small")
 		(at 69.85 66.04 0)
 		(unit 1)
@@
 			)
 		)
-		(property "Footprint Audit" "VERIFIED: NXP HVSON8 SOT782-1, 3x3 mm, P0.65, EP 1.6x2.4; symbol pin 9 EP/GND matches exposed pad"
+		(property "Footprint Audit" "See verification/COMPONENTS.csv and verification/REPORT.md"
 			(at 71.12 63.5 0)
 			(hide yes)
@@
 			)
 		)
-		(property "Library Audit" "KiCad standard"
+		(property "Library Audit" "See verification/COMPONENTS.csv and verification/REPORT.md"
 			(at 71.12 63.5 0)
 			(hide yes)
@@
 	)
 	(symbol
-		(lib_id "power:+5V")
+		(lib_id "FC01_Project:CAN__+5V")
 		(at 69.85 55.88 0)
 		(unit 1)
@@
 	)
 	(symbol
-		(lib_id "power:+5V")
+		(lib_id "FC01_Project:CAN__+5V")
 		(at 148.59 57.15 0)
 		(unit 1)
@@
 	)
 	(symbol
-		(lib_id "power:GND")
+		(lib_id "FC01_Project:CAN__GND")
 		(at 100.33 81.28 0)
 		(unit 1)
@@
 	)
 	(symbol
-		(lib_id "power:GND")
+		(lib_id "FC01_Project:CAN__GND")
 		(at 64.77 69.85 0)
 		(unit 1)
@@
 	)
 	(symbol
-		(lib_id "Device:C_Small")
+		(lib_id "FC01_Project:CAN__C_Small")
 		(at 64.77 66.04 0)
 		(unit 1)
@@
 			)
 		)
-		(property "Footprint Audit" "VERIFIED: NXP HVSON8 SOT782-1, 3x3 mm, P0.65, EP 1.6x2.4; symbol pin 9 EP/GND matches exposed pad"
+		(property "Footprint Audit" "See verification/COMPONENTS.csv and verification/REPORT.md"
 			(at 66.04 63.5 0)
 			(hide yes)
@@
 			)
 		)
-		(property "Library Audit" "KiCad standard"
+		(property "Library Audit" "See verification/COMPONENTS.csv and verification/REPORT.md"
 			(at 66.04 63.5 0)
 			(hide yes)
@@
 	)
 	(symbol
-		(lib_id "power:+3V3")
+		(lib_id "FC01_Project:CAN__+3V3")
 		(at 64.77 60.96 0)
 		(unit 1)
@@
 	)
 	(symbol
-		(lib_id "power:GND")
+		(lib_id "FC01_Project:CAN__GND")
 		(at 130.81 93.98 0)
 		(unit 1)
@@
 	)
 	(symbol
-		(lib_id "power:GND")
+		(lib_id "FC01_Project:CAN__GND")
 		(at 154.94 115.57 0)
 		(unit 1)
@@
 	)
 	(symbol
-		(lib_id "Interface_CAN_LIN:TJA1051TK-3")
+		(lib_id "FC01_Project:CAN__TJA1051TK-3")
 		(at 101.6 66.04 0)
 		(unit 1)
@@
 			)
 		)
-		(property "Footprint Audit" "VERIFIED: NXP HVSON8 SOT782-1, 3x3 mm, P0.65, EP 1.6x2.4; symbol pin 9 EP/GND matches exposed pad"
+		(property "Footprint Audit" "See verification/COMPONENTS.csv and verification/REPORT.md"
 			(at 101.6 49.53 0)
 			(hide yes)
@@
 			)
 		)
-		(property "Library Audit" "Project-local symbol + verified JST footprint"
+		(property "Library Audit" "See verification/COMPONENTS.csv and verification/REPORT.md"
 			(at 101.6 49.53 0)
 			(hide yes)
@@
 	)
 	(symbol
-		(lib_id "power:+5V")
+		(lib_id "FC01_Project:CAN__+5V")
 		(at 152.4 88.9 0)
 		(unit 1)
@@
 	)
 	(symbol
-		(lib_id "PCM_Diode_TVS_AKL:PESD2CAN")
+		(lib_id "FC01_Project:CAN__PESD2CAN")
 		(at 130.81 85.09 90)
 		(unit 1)
@@
 			)
 		)
-		(property "Datasheet" "https://assets.nexperia.com/documents/data-sheet/PESD2CANFD24V.pdf"
+		(property "Datasheet" "https://assets.nexperia.com/documents/data-sheet/PESD2CANFD24V-T.pdf"
 			(at 121.92 85.09 0)
 			(hide yes)
@@
 			)
 		)
-		(property "Footprint Audit" "VERIFIED: NXP HVSON8 SOT782-1, 3x3 mm, P0.65, EP 1.6x2.4; symbol pin 9 EP/GND matches exposed pad"
+		(property "Footprint Audit" "See verification/COMPONENTS.csv and verification/REPORT.md"
 			(at 137.16 84.3914 90)
 			(hide yes)
@@
 			)
 		)
-		(property "Library Audit" "Custom verified symbol + KiCad standard SOT-23 footprint"
+		(property "Library Audit" "See verification/COMPONENTS.csv and verification/REPORT.md"
 			(at 137.16 84.3914 90)
 			(hide yes)
@@
 	)
 	(symbol
-		(lib_id "H743_Ardupilot:JST_GH_SM04B_GHS_TB_4P")
+		(lib_id "FC01_Project:CAN__JST_GH_SM04B_GHS_TB_4P")
 		(at 154.94 64.77 0)
 		(unit 1)
@@
 			)
 		)
-		(property "Package" "SH1.0 4P right-angle SMD"
+		(property "Package" "JST GH 4 contacts, P1.25 mm, side entry; mounting tabs pads 5/6"
 			(at 151.13 55.88 0)
 			(hide yes)
@@
 			)
 		)
-		(property "Footprint Audit" "OK against JST drawing"
+		(property "Footprint Audit" "See verification/COMPONENTS.csv and verification/REPORT.md"
 			(at 151.13 55.88 0)
 			(hide yes)
@@
 			)
 		)
-		(property "Library Audit" "Project-local symbol + verified JST footprint"
+		(property "Library Audit" "See verification/COMPONENTS.csv and verification/REPORT.md"
 			(at 151.13 55.88 0)
 			(hide yes)
@@
 	)
 	(symbol
-		(lib_id "power:GND")
+		(lib_id "FC01_Project:CAN__GND")
 		(at 148.59 76.2 0)
 		(unit 1)
@@
 	)
 	(symbol
-		(lib_id "Connector_Generic:Conn_01x04")
+		(lib_id "FC01_Project:CAN__Conn_01x04")
 		(at 162.56 95.25 0)
 		(unit 1)
@@
 			)
 		)
-		(property "Footprint Audit" "OK: 4 square SMD pads 1.00x1.00 mm, P2.54 mm, no holes, no paste"
+		(property "Footprint Audit" "See verification/COMPONENTS.csv and verification/REPORT.md"
 			(at 165.1 95.2499 0)
 			(hide yes)
@@
 			)
 		)
-		(property "Library Audit" "Project-local H743_Custom footprint"
+		(property "Library Audit" "See verification/COMPONENTS.csv and verification/REPORT.md"
 			(at 165.1 95.2499 0)
 			(hide yes)
@@
 	)
 	(symbol
-		(lib_id "power:GND")
+		(lib_id "FC01_Project:CAN__GND")
 		(at 69.85 69.85 0)
 		(unit 1)
