File: CAN.kicad_sch (KiCad schematic)
At the start: 7 parts, among them J13 Can1_2, J14 Can1_1, U7 TJA1051TK/3,118, U8 SM04B-GHS-TB(LF)(SN)

Commit message: Replace EOL CAN transceiver with TJA1057GTK/3Z
Parts:
- U7: value TJA1051TK/3,118 -> TJA1057GTK/3Z; symbol FC01_Project:CAN__TJA1051TK-3 -> FC01_Project:CAN__TJA1057GTK-3; Datasheet_URL https://www.nxp.com/docs/en/data-sheet/TJA1051.pdf -> https://www.nxp.com/docs/en/data-sheet/TJA1057.pdf; Footprint Audit NXP TJA1051 Rev9 pp.4,16: TK=SOT782 HVSON8+EP; variante /3 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 -> NXP TJA1057: GTK/3Z, SOT782 HVSON8+EP; pinout compatible /3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; LCSC C124020 -> (none); LCSC Part C124020 -> (none); MPN TJA1051TK/3,118 -> TJA1057GTK/3Z; Manufacturer NXP USA Inc. -> NXP Semiconductors; Symbol_ID FC01_Project:CAN__TJA1051TK-3 -> FC01_Project:CAN__TJA1057GTK-3
Changed lines of the file:
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@@
 		(date "2026-09-24")
 	)
-	(text_box "CAN-FD ALTERNATIVES\n\n! TO BE VALIDATED !\n\nTJA1051TK/3,118:	C124020\nSIT1051TK/3:		C1121846\n"
+	(text_box "CAN-FD ALTERNATIVES\n\n! TO BE VALIDATED !\n\nTJA1057GTK/3Z:	\nSIT1051TK/3:		C1121846\n"
 		(exclude_from_sim no)
 		(at 83.82 88.9 0)
@@
 	)
 	(symbol
-		(lib_id "FC01_Project:CAN__TJA1051TK-3")
+		(lib_id "FC01_Project:CAN__TJA1057GTK-3")
 		(at 101.6 66.04 0)
 		(unit 1)
@@
 			)
 		)
-		(property "Value" "TJA1051TK/3,118"
+		(property "Value" "TJA1057GTK/3Z"
 			(at 101.6 52.07 0)
 			(show_name no)
@@
 			)
 		)
-		(property "Manufacturer" "NXP USA Inc."
+		(property "Manufacturer" "NXP Semiconductors"
 			(at 101.6 88.9 0)
 			(hide yes)
@@
 			)
 		)
-		(property "MPN" "TJA1051TK/3,118"
+		(property "MPN" "TJA1057GTK/3Z"
 			(at 101.6 91.44 0)
 			(hide yes)
@@
 			)
 		)
-		(property "LCSC Part" "C124020"
+		(property "LCSC Part" ""
 			(at 101.6 93.98 0)
 			(hide yes)
@@
 			)
 		)
-		(property "LCSC" "C124020"
+		(property "LCSC" ""
 			(at 101.6 66.04 0)
 			(hide yes)
@@
 			)
 		)
-		(property "Footprint Audit" "NXP TJA1051 Rev9 pp.4,16: TK=SOT782 HVSON8+EP; variante /3 pin5 VIO. 1TXD 2GND 3VCC 4RXD 5VIO 6CANL 7CANH 8S; EP9 GND. Corps 3 x 3, pas 0.65 mm."
+		(property "Footprint Audit" "NXP TJA1057: GTK/3Z, SOT782 HVSON8+EP; pinout compatible /3: 1 TXD, 2 GND, 3 VCC, 4 RXD, 5 VIO, 6 CANL, 7 CANH, 8 S; EP GND. Successor selected for EOL TJA1051TK/3."
 			(at 101.6 49.53 0)
 			(hide yes)
@@
 			)
 		)
-		(property "Datasheet_URL" "https://www.nxp.com/docs/en/data-sheet/TJA1051.pdf"
+		(property "Datasheet_URL" "https://www.nxp.com/docs/en/data-sheet/TJA1057.pdf"
 			(at 0 0 0)
 			(hide yes)
@@
 			)
 		)
-		(property "Symbol_ID" "FC01_Project:CAN__TJA1051TK-3"
+		(property "Symbol_ID" "FC01_Project:CAN__TJA1057GTK-3"
 			(at 0 0 0)
 			(hide yes)

Commit message: Audit FC_01 libraries nets supplier specs and placement
Parts:
- U7: Component_PDF ${KIPRJMOD}/composants/controle/TJA1051TK_3_118.pdf -> ${KIPRJMOD}/composants/pdf/U7_datasheet.pdf; DigiKey Part Number 568-8686-1-ND -> (none); DigiKey Price Qty 1 -> (none); DigiKey Status Stock positif au releve -> Offre DigiKey France non retenue ou non confirmee; DigiKey URL https://www.digikey.fr/fr/products/detail/nxp-usa-inc/TJA10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 -> (none); DigiKey Unit Price EUR 1.65 -> (none); DigiKey_Part_Number 568-8686-1-ND -> (none); DigiKey_URL https://www.digikey.fr/fr/products/detail/nxp-usa-inc/TJA10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 -> (none); Footprint Audit NXP TJA1057: GTK/3Z, SOT782 HVSON8+EP; pinout compatible /3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 -> NXP TJA1057 Rev 8.1, 2 mars 2026: GTK/3Z = HVSON8 SOT782-1,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; Price Checked 2026-09-27 -> (none); Price_Basis EUR HT par piece, hors port -> (none); Price_Checked 2026-09-27 -> (none); Price_Qty 1 -> (none); Stock_Checked 2026-09-27 -> (none); Stock_Units 20970 -> (none); Supplier DigiKey France -> Non confirme; Supplier Specs Relevé web; stock et prix variables. Derniere date d achat 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 -> Ne pas reutiliser les prix et stocks du TJA1051; reference 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; Supplier_Notes Relevé web; stock et prix variables. Derniere date d achat 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 -> Ne pas reutiliser les prix et stocks du TJA1051; reference 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; Supplier_Order_Code 568-8686-1-ND -> (none); Supplier_Status Stock positif au releve -> Offre France non confirmee; Supplier_URL https://www.digikey.fr/fr/products/detail/nxp-usa-inc/TJA10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 -> (none); Unit_Price_EUR 1.65 -> (none)
Changed lines of the file:
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@@
 			)
 		)
-		(property "Supplier Specs" "Relevé web; stock et prix variables. Derniere date d achat annoncee: 26/12/2026; verifier cycle de vie."
+		(property "Supplier Specs" "Ne pas reutiliser les prix et stocks du TJA1051; reference TJA1057GTK/3Z a confirmer avant achat."
 			(at 101.6 91.44 0)
 			(hide yes)
@@
 			)
 		)
-		(property "DigiKey Part Number" "568-8686-1-ND"
-			(at 101.6 49.53 0)
-			(hide yes)
-			(show_name no)
-			(do_not_autoplace no)
-			(effects
-				(font
-					(size 1.27 1.27)
-				)
-			)
-		)
-		(property "DigiKey URL" "https://www.digikey.fr/fr/products/detail/nxp-usa-inc/TJA1051TK-3-118/2803572"
+		(property "DigiKey Part Number" ""
+			(at 101.6 49.53 0)
+			(hide yes)
+			(show_name no)
+			(do_not_autoplace no)
+			(effects
+				(font
+					(size 1.27 1.27)
+				)
+			)
+		)
+		(property "DigiKey URL" ""
 			(at 101.6 49.53 0)
 			(hide yes)
@@
 			)
 		)
-		(property "DigiKey Unit Price EUR" "1.65"
-			(at 101.6 49.53 0)
-			(hide yes)
-			(show_name no)
-			(do_not_autoplace no)
-			(effects
-				(font
-					(size 1.27 1.27)
-				)
-			)
-		)
-		(property "DigiKey Price Qty" "1"
-			(at 101.6 49.53 0)
-			(hide yes)
-			(show_name no)
-			(do_not_autoplace no)
-			(effects
-				(font
-					(size 1.27 1.27)
-				)
-			)
-		)
-		(property "Price Checked" "2026-09-27"
-			(at 101.6 49.53 0)
-			(hide yes)
-			(show_name no)
-			(do_not_autoplace no)
-			(effects
-				(font
-					(size 1.27 1.27)
-				)
-			)
-		)
-		(property "DigiKey Status" "Stock positif au releve"
+		(property "DigiKey Unit Price EUR" ""
+			(at 101.6 49.53 0)
+			(hide yes)
+			(show_name no)
+			(do_not_autoplace no)
+			(effects
+				(font
+					(size 1.27 1.27)
+				)
+			)
+		)
+		(property "DigiKey Price Qty" ""
+			(at 101.6 49.53 0)
+			(hide yes)
+			(show_name no)
+			(do_not_autoplace no)
+			(effects
+				(font
+					(size 1.27 1.27)
+				)
+			)
+		)
+		(property "Price Checked" ""
+			(at 101.6 49.53 0)
+			(hide yes)
+			(show_name no)
+			(do_not_autoplace no)
+			(effects
+				(font
+					(size 1.27 1.27)
+				)
+			)
+		)
+		(property "DigiKey Status" "Offre DigiKey France non retenue ou non confirmee"
 			(at 101.6 49.53 0)
 			(hide yes)
@@
 			)
 		)
-		(property "Footprint Audit" "NXP TJA1057: GTK/3Z, SOT782 HVSON8+EP; pinout compatible /3: 1 TXD, 2 GND, 3 VCC, 4 RXD, 5 VIO, 6 CANL, 7 CANH, 8 S; EP GND. Successor selected for EOL TJA1051TK/3."
+		(property "Footprint Audit" "NXP TJA1057 Rev 8.1, 2 mars 2026: GTK/3Z = HVSON8 SOT782-1, 3 x 3 x 0.85 mm, pin 5 VIO; 1 TXD, 2 GND, 3 VCC, 4 RXD, 5 VIO, 6 CANL, 7 CANH, 8 S. Pad central relie GND. Implantation HVSON8 existante a confirmer avec tolerances de soudure."
 			(at 101.6 49.53 0)
 			(hide yes)
@@
 			)
 		)
-		(property "DigiKey_Part_Number" "568-8686-1-ND"
-			(at 0 0 0)
-			(hide yes)
-			(show_name no)
-			(do_not_autoplace no)
-			(effects
-				(font
-					(size 1.27 1.27)
-				)
-			)
-		)
-		(property "DigiKey_URL" "https://www.digikey.fr/fr/products/detail/nxp-usa-inc/TJA1051TK-3-118/2803572"
-			(at 0 0 0)
-			(hide yes)
-			(show_name no)
-			(do_not_autoplace no)
-			(effects
-				(font
-					(size 1.27 1.27)
-				)
-			)
-		)
-		(property "Price_Checked" "2026-09-27"
-			(at 0 0 0)
-			(hide yes)
-			(show_name no)
-			(do_not_autoplace no)
-			(effects
-				(font
-					(size 1.27 1.27)
-				)
-			)
-		)
-		(property "Price_Qty" "1"
-			(at 0 0 0)
-			(hide yes)
-			(show_name no)
-			(do_not_autoplace no)
-			(effects
-				(font
-					(size 1.27 1.27)
-				)
-			)
-		)
-		(property "Stock_Units" "20970"
-			(at 0 0 0)
-			(hide yes)
-			(show_name no)
-			(do_not_autoplace no)
-			(effects
-				(font
-					(size 1.27 1.27)
-				)
-			)
-		)
-		(property "Supplier" "DigiKey France"
-			(at 0 0 0)
-			(hide yes)
-			(show_name no)
-			(do_not_autoplace no)
-			(effects
-				(font
-					(size 1.27 1.27)
-				)
-			)
-		)
-		(property "Supplier_Order_Code" "568-8686-1-ND"
-			(at 0 0 0)
-			(hide yes)
-			(show_name no)
-			(do_not_autoplace no)
-			(effects
-				(font
-					(size 1.27 1.27)
-				)
-			)
-		)
-		(property "Supplier_URL" "https://www.digikey.fr/fr/products/detail/nxp-usa-inc/TJA1051TK-3-118/2803572"
-			(at 0 0 0)
-			(hide yes)
-			(show_name no)
-			(do_not_autoplace no)
-			(effects
-				(font
-					(size 1.27 1.27)
-				)
-			)
-		)
-		(property "Unit_Price_EUR" "1.65"
+		(property "DigiKey_Part_Number" ""
+			(at 0 0 0)
+			(hide yes)
+			(show_name no)
+			(do_not_autoplace no)
+			(effects
+				(font
+					(size 1.27 1.27)
+				)
+			)
+		)
+		(property "DigiKey_URL" ""
+			(at 0 0 0)
+			(hide yes)
+			(show_name no)
+			(do_not_autoplace no)
+			(effects
+				(font
+					(size 1.27 1.27)
+				)
+			)
+		)
+		(property "Price_Checked" ""
+			(at 0 0 0)
+			(hide yes)
+			(show_name no)
+			(do_not_autoplace no)
+			(effects
+				(font
+					(size 1.27 1.27)
+				)
+			)
+		)
+		(property "Price_Qty" ""
+			(at 0 0 0)
+			(hide yes)
+			(show_name no)
+			(do_not_autoplace no)
+			(effects
+				(font
+					(size 1.27 1.27)
+				)
+			)
+		)
+		(property "Stock_Units" ""
+			(at 0 0 0)
+			(hide yes)
+			(show_name no)
+			(do_not_autoplace no)
+			(effects
+				(font
+					(size 1.27 1.27)
+				)
+			)
+		)
+		(property "Supplier" "Non confirme"
+			(at 0 0 0)
+			(hide yes)
+			(show_name no)
+			(do_not_autoplace no)
+			(effects
+				(font
+					(size 1.27 1.27)
+				)
+			)
+		)
+		(property "Supplier_Order_Code" ""
+			(at 0 0 0)
+			(hide yes)
+			(show_name no)
+			(do_not_autoplace no)
+			(effects
+				(font
+					(size 1.27 1.27)
+				)
+			)
+		)
+		(property "Supplier_URL" ""
+			(at 0 0 0)
+			(hide yes)
+			(show_name no)
+			(do_not_autoplace no)
+			(effects
+				(font
+					(size 1.27 1.27)
+				)
+			)
+		)
+		(property "Unit_Price_EUR" ""
 			(at 0 0 0)
 			(hide yes)
@@
 			)
 		)
-		(property "Component_PDF" "${KIPRJMOD}/composants/controle/TJA1051TK_3_118.pdf"
+		(property "Component_PDF" "${KIPRJMOD}/composants/pdf/U7_datasheet.pdf"
 			(at 0 0 0)
 			(hide yes)
@@
 			)
 		)
-		(property "Price_Basis" "EUR HT par piece, hors port"
-			(at 0 0 0)
-			(hide yes)
-			(show_name no)
-			(do_not_autoplace no)
-			(effects
-				(font
-					(size 1.27 1.27)
-				)
-			)
-		)
-		(property "Stock_Checked" "2026-09-27"
-			(at 0 0 0)
-			(hide yes)
-			(show_name no)
-			(do_not_autoplace no)
-			(effects
-				(font
-					(size 1.27 1.27)
-				)
-			)
-		)
-		(property "Supplier_Notes" "Relevé web; stock et prix variables. Derniere date d achat annoncee: 26/12/2026; verifier cycle de vie."
-			(at 0 0 0)
-			(hide yes)
-			(show_name no)
-			(do_not_autoplace no)
-			(effects
-				(font
-					(size 1.27 1.27)
-				)
-			)
-		)
-		(property "Supplier_Status" "Stock positif au releve"
-			(at 0 0 0)
-			(hide yes)
+		(property "Price_Basis" ""
+			(at 0 0 0)
+			(hide yes)
+			(show_name no)
+			(do_not_autoplace no)
+			(effects
+				(font
+					(size 1.27 1.27)
+				)
+			)
+		)
+		(property "Stock_Checked" ""
+			(at 0 0 0)
+			(hide yes)
+			(show_name no)
+			(do_not_autoplace no)
+			(effects
+				(font
+					(size 1.27 1.27)
+				)
+			)
+		)
+		(property "Supplier_Notes" "Ne pas reutiliser les prix et stocks du TJA1051; reference TJA1057GTK/3Z a confirmer avant achat."
+			(at 0 0 0)
+			(hide yes)
+			(show_name no)
+			(do_not_autoplace no)
+			(effects
+				(font
+					(size 1.27 1.27)
+				)
+			)
+		)
+		(property "Supplier_Status" "Offre France non confirmee"
+			(at 0 0 0)
+			(hide yes)
