File: POWER.kicad_sch (KiCad schematic)
At the start: 32 parts, among them U12 LMR43620R5RPER, U13 LMR604303SRAKRQ1, U14 AP7361C-33FGE-7, U15 AP7361C-33FGE-7

Commit message: fill verified DigiKey pricing for 50V power capacitors
Parts:
- C44, C45, C47, C48, C52, C54: DigiKey Price Qty (none) -> 1 CT; DigiKey Unit Price EUR (none) -> 0.09
Changed lines of the file:
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@@
 			(effects (font (size 1.27 1.27)))
 		)
-		(property "DigiKey Unit Price EUR" ""
+		(property "DigiKey Unit Price EUR" "0.09"
 			(at 160.02 119.38 0)
 			(hide yes)
@@
 			(effects (font (size 1.27 1.27)))
 		)
-		(property "DigiKey Price Qty" ""
+		(property "DigiKey Price Qty" "1 CT"
 			(at 160.02 119.38 0)
 			(hide yes)
@@
 			(effects (font (size 1.27 1.27)))
 		)
-		(property "DigiKey Unit Price EUR" ""
+		(property "DigiKey Unit Price EUR" "0.09"
 			(at 48.26 119.38 0)
 			(hide yes)
@@
 			(effects (font (size 1.27 1.27)))
 		)
-		(property "DigiKey Price Qty" ""
+		(property "DigiKey Price Qty" "1 CT"
 			(at 48.26 119.38 0)
 			(hide yes)
@@
 			(effects (font (size 1.27 1.27)))
 		)
-		(property "DigiKey Unit Price EUR" ""
+		(property "DigiKey Unit Price EUR" "0.09"
 			(at 115.57 59.69 90)
 			(hide yes)
@@
 			(effects (font (size 1.27 1.27)))
 		)
-		(property "DigiKey Price Qty" ""
+		(property "DigiKey Price Qty" "1 CT"
 			(at 115.57 59.69 90)
 			(hide yes)
@@
 			(effects (font (size 1.27 1.27)))
 		)
-		(property "DigiKey Unit Price EUR" ""
+		(property "DigiKey Unit Price EUR" "0.09"
 			(at 152.4 63.5 0)
 			(hide yes)
@@
 			(effects (font (size 1.27 1.27)))
 		)
-		(property "DigiKey Price Qty" ""
+		(property "DigiKey Price Qty" "1 CT"
 			(at 152.4 63.5 0)
 			(hide yes)
@@
 			(effects (font (size 1.27 1.27)))
 		)
-		(property "DigiKey Unit Price EUR" ""
+		(property "DigiKey Unit Price EUR" "0.09"
 			(at 118.11 115.57 90)
 			(hide yes)
@@
 			(effects (font (size 1.27 1.27)))
 		)
-		(property "DigiKey Price Qty" ""
+		(property "DigiKey Price Qty" "1 CT"
 			(at 118.11 115.57 90)
 			(hide yes)
@@
 			(effects (font (size 1.27 1.27)))
 		)
-		(property "DigiKey Unit Price EUR" ""
+		(property "DigiKey Unit Price EUR" "0.09"
 			(at 48.26 63.5 0)
 			(hide yes)
@@
 			(effects (font (size 1.27 1.27)))
 		)
-		(property "DigiKey Price Qty" ""
+		(property "DigiKey Price Qty" "1 CT"
 			(at 48.26 63.5 0)
 			(hide yes)

Commit message: review power line
Other:
- note added: "+3V3 MCU"
- note added: "+9V - DJI VIDEO TX"
- note added: "+Ext 5v power supply"
- note added: "3V3 Sens"
- note removed: "Ajouter 100 kΩ entre DJI_EN et +3V3_MCU est la bonne conception."
- note removed: "PIN-TO-PIN COMPATIBLE WITH 4A/6A VERSIONS LIKE LMR60440-Q1"
- moved on the sheet: C43, C45, C48, C51, C53, C54, L2, R45, R46, R47, R48, U13
