File: POWER.kicad_sch (KiCad schematic)
At the start: 32 parts, among them U12 LMR43620R5RPER, U13 LMR604303SRAKRQ1, U14 AP7361C-33FGE-7, U15 AP7361C-33FGE-7

Commit message: use official KiCad CFP3 footprint for D4
Parts:
- D4: footprint Diode_SMD:D_SOD-123W -> Diode_SMD:Nexperia_CFP3_SOD-123W; Footprint Audit OK: KiCad SOD-123W matches Nexperia CFP3/SOD123W package cl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 -> OK: official KiCad Nexperia_CFP3_SOD-123W footprint matches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
Changed lines of the file:
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@@
 			)
 		)
-		(property "Footprint" "Diode_SMD:D_SOD-123W"
+		(property "Footprint" "Diode_SMD:Nexperia_CFP3_SOD-123W"
 			(at 170.18 56.515 0)
 			(hide yes)
@@
 			)
 		)
-		(property "Footprint Audit" "OK: KiCad SOD-123W matches Nexperia CFP3/SOD123W package class"
+		(property "Footprint Audit" "OK: official KiCad Nexperia_CFP3_SOD-123W footprint matches Nexperia CFP3/SOD123W"
 			(at 166.37 59.69 0)
 			(hide yes)

Commit message: normalize 3V3 rail labels
Other:
- note added: "+3V3_MCU"
- note added: "+3V3_SENS"
- note removed: "+3V3 MCU"
- note removed: "3V3 Sens"
Changed lines of the file:
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@@
 		)
 	)
-	(text "3V3 Sens"
+	(text "+3V3_SENS"
 		(exclude_from_sim no)
 		(at 255.016 105.156 0)
@@
 		)
 	)
-	(text "+3V3 MCU"
+	(text "+3V3_MCU"
 		(exclude_from_sim no)
 		(at 251.206 49.784 0)

Commit message: upgrade L1 L2 to XGL4030 3.3uH
Parts:
- L1, L2: value 2.2u -> 3.3u; footprint H743_Custom:L_Coilcraft_XGL4020 -> H743_Custom:L_Coilcraft_XGL4030; DigiKey Specs 2.2 µH, ±20%, Irms 8.9 A, Isat 6.2 A typ listing, DCR 21.5 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 -> 3.3 µH, ±20%, Irms 7.5 A, Isat 5.3 A (30% L drop), DCR 21.9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; DigiKey URL https://www.digikey.fr/en/products/result?keywords=XGL4020-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 -> https://www.digikey.fr/en/products/result?keywords=XGL4030-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; Footprint Audit OK: exact Coilcraft XGL4020 recommended land pattern; pads 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 -> OK: Coilcraft XGL4030 recommended land pattern; pads 0.98x3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; MPN XGL4020-222MEC -> XGL4030-332MEC; Package XGL4020, 4.0x4.0x2.1 mm -> XGL4030, 4.0x4.0x3.1 mm
Changed lines of the file:
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@@
 			)
 		)
-		(property "Value" "2.2u"
+		(property "Value" "3.3u"
 			(at 140.97 118.11 90)
 			(show_name no)
@@
 			)
 		)
-		(property "Footprint" "H743_Custom:L_Coilcraft_XGL4020"
+		(property "Footprint" "H743_Custom:L_Coilcraft_XGL4030"
 			(at 140.97 120.65 0)
 			(hide yes)
@@
 			)
 		)
-		(property "Datasheet" "https://www.coilcraft.com/en-us/products/power/shielded-inductors/molded-inductor/xgl/xgl4020/xgl4020-222/"
+		(property "Datasheet" "https://www.coilcraft.com/en-us/products/power/shielded-inductors/molded-inductor/xgl/xgl4030/xgl4030-332/"
 			(at 140.97 120.65 0)
 			(hide yes)
@@
 			)
 		)
-		(property "MPN" "XGL4020-222MEC"
+		(property "MPN" "XGL4030-332MEC"
 			(at 140.97 120.65 90)
 			(hide yes)
@@
 			)
 		)
-		(property "DigiKey URL" "https://www.digikey.fr/en/products/result?keywords=XGL4020-222MEC"
+		(property "DigiKey URL" "https://www.digikey.fr/en/products/result?keywords=XGL4030-332MEC"
 			(at 140.97 115.57 90)
 			(hide yes)
@@
 			)
 		)
-		(property "DigiKey Specs" "2.2 µH, ±20%, Irms 8.9 A, Isat 6.2 A typ listing, DCR 21.5 mΩ max, 4.0x4.0x2.1 mm"
+		(property "DigiKey Specs" "3.3 µH, ±20%, Irms 7.5 A, Isat 5.3 A (30% L drop), DCR 21.9 mΩ max, 4.0x4.0x3.1 mm"
 			(at 140.97 115.57 90)
 			(hide yes)
@@
 			)
 		)
-		(property "Package" "XGL4020, 4.0x4.0x2.1 mm"
+		(property "Package" "XGL4030, 4.0x4.0x3.1 mm"
 			(at 140.97 115.57 90)
 			(hide yes)
@@
 			)
 		)
-		(property "Footprint Audit" "OK: exact Coilcraft XGL4020 recommended land pattern; pads 0.98x3.40 mm at ±1.185 mm"
+		(property "Footprint Audit" "OK: Coilcraft XGL4030 recommended land pattern; pads 0.98x3.40 mm at ±1.185 mm"
 			(at 140.97 115.57 90)
 			(hide yes)
@@
 			)
 		)
-		(property "Value" "2.2u"
+		(property "Value" "3.3u"
 			(at 129.54 58.42 90)
 			(show_name no)
@@
 			)
 		)
-		(property "Footprint" "H743_Custom:L_Coilcraft_XGL4020"
+		(property "Footprint" "H743_Custom:L_Coilcraft_XGL4030"
 			(at 129.54 60.96 0)
 			(hide yes)
@@
 			)
 		)
-		(property "Datasheet" "https://www.coilcraft.com/en-us/products/power/shielded-inductors/molded-inductor/xgl/xgl4020/xgl4020-222/"
+		(property "Datasheet" "https://www.coilcraft.com/en-us/products/power/shielded-inductors/molded-inductor/xgl/xgl4030/xgl4030-332/"
 			(at 129.54 60.96 0)
 			(hide yes)
@@
 			)
 		)
-		(property "MPN" "XGL4020-222MEC"
+		(property "MPN" "XGL4030-332MEC"
 			(at 129.54 60.96 90)
 			(hide yes)
@@
 			)
 		)
-		(property "DigiKey URL" "https://www.digikey.fr/en/products/result?keywords=XGL4020-222MEC"
+		(property "DigiKey URL" "https://www.digikey.fr/en/products/result?keywords=XGL4030-332MEC"
 			(at 129.54 55.88 90)
 			(hide yes)
@@
 			)
 		)
-		(property "DigiKey Specs" "2.2 µH, ±20%, Irms 8.9 A, Isat 6.2 A typ listing, DCR 21.5 mΩ max, 4.0x4.0x2.1 mm"
+		(property "DigiKey Specs" "3.3 µH, ±20%, Irms 7.5 A, Isat 5.3 A (30% L drop), DCR 21.9 mΩ max, 4.0x4.0x3.1 mm"
 			(at 129.54 55.88 90)
 			(hide yes)
@@
 			)
 		)
-		(property "Package" "XGL4020, 4.0x4.0x2.1 mm"
+		(property "Package" "XGL4030, 4.0x4.0x3.1 mm"
 			(at 129.54 55.88 90)
 			(hide yes)
@@
 			)
 		)
-		(property "Footprint Audit" "OK: exact Coilcraft XGL4020 recommended land pattern; pads 0.98x3.40 mm at ±1.185 mm"
+		(property "Footprint Audit" "OK: Coilcraft XGL4030 recommended land pattern; pads 0.98x3.40 mm at ±1.185 mm"
 			(at 129.54 55.88 90)
 			(hide yes)

Commit message: finalize XGL4030 sourcing metadata
Parts:
- L1, L2: DigiKey URL https://www.digikey.fr/en/products/result?keywords=XGL4030-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 -> https://www.digikey.com/en/products/detail/coilcraft/XGL403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
Changed lines of the file:
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@@
 			)
 		)
-		(property "DigiKey URL" "https://www.digikey.fr/en/products/result?keywords=XGL4030-332MEC"
+		(property "DigiKey URL" "https://www.digikey.com/en/products/detail/coilcraft/XGL4030-332MEC/12714440"
 			(at 140.97 115.57 90)
 			(hide yes)
@@
 			)
 		)
-		(property "DigiKey URL" "https://www.digikey.fr/en/products/result?keywords=XGL4030-332MEC"
+		(property "DigiKey URL" "https://www.digikey.com/en/products/detail/coilcraft/XGL4030-332MEC/12714440"
 			(at 129.54 55.88 90)
 			(hide yes)

Commit message: update
Parts:
- renumbered C42 to C16, C44 to C17, C43 to C18, C45 to C19, C46 to C20, C47 to C21, C48 to C22, C49 to C23, C50 to C24, C52 to C25, C51 to C26, C53 to C27, C54 to C28, C55 to C29, C56 to C30, C57 to C31, C58 to C32, D3 to D2, D4 to D3, D5 to D4, R47 to R10, R48 to R11, R49 to R12, R50 to R13, R45 to R8, R46 to R9, U12 to U3, U13 to U4, U14 to U5, U15 to U6

Commit message: Use verified LMR43620 footprint and add sourcing metadata
Parts:
- U3: footprint EasyEDA:VQFN-9_L2.1-W2.1-P0.50-TL -> H743_Custom:TI_RPE0009B_VQFN-HR-9_2x2mm; DigiKey EDA Model URL (none) -> https://www.digikey.com/en/models/20414090; Footprint Audit CHECK: current EasyEDA footprint named 2.1x2.1; compare to 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 -> OK: project-local native KiCad footprint derived from suppl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; Footprint Source (none) -> Ultra Librarian archive supplied for LMR43620R5RPER; normal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; LCSC URL (none) -> https://www.lcsc.com/product-detail/C32712896.html; Mouser URL (none) -> https://www.mouser.com/ProductDetail/Texas-Instruments/LMR4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; TI Datasheet PDF (none) -> https://www.ti.com/lit/ds/symlink/lmr43620.pdf; TI Product URL (none) -> https://www.ti.com/product/LMR43620/part-details/LMR43620R5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
- U6: Library Audit EasyEDA external -> Project-local H743_Custom footprint; no EasyEDA footprint d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
Changed lines of the file:
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@@
 			)
 		)
-		(property "Library Audit" "EasyEDA external"
+		(property "Library Audit" "Project-local H743_Custom footprint; no EasyEDA footprint dependency"
 			(at 237.49 109.22 0)
 			(hide yes)
@@
 			)
 		)
-		(property "Footprint" "EasyEDA:VQFN-9_L2.1-W2.1-P0.50-TL"
+		(property "Footprint" "H743_Custom:TI_RPE0009B_VQFN-HR-9_2x2mm"
 			(at 96.52 82.55 0)
 			(hide yes)
@@
 			)
 		)
-		(property "Footprint Audit" "CHECK: current EasyEDA footprint named 2.1x2.1; compare to TI RPE land pattern"
+		(property "TI Product URL" "https://www.ti.com/product/LMR43620/part-details/LMR43620R5RPER"
 			(at 96.52 52.07 0)
 			(hide yes)
+			(show_name no)
+			(do_not_autoplace no)
+			(effects
+				(font
+					(size 1.27 1.27)
+				)
+			)
+		)
+		(property "TI Datasheet PDF" "https://www.ti.com/lit/ds/symlink/lmr43620.pdf"
+			(at 96.52 52.07 0)
+			(hide yes)
+			(show_name no)
+			(do_not_autoplace no)
+			(effects
+				(font
+					(size 1.27 1.27)
+				)
+			)
+		)
+		(property "Mouser URL" "https://www.mouser.com/ProductDetail/Texas-Instruments/LMR43620R5RPER"
+			(at 96.52 52.07 0)
+			(hide yes)
+			(show_name no)
+			(do_not_autoplace no)
+			(effects
+				(font
+					(size 1.27 1.27)
+				)
+			)
+		)
+		(property "LCSC URL" "https://www.lcsc.com/product-detail/C32712896.html"
+			(at 96.52 52.07 0)
+			(hide yes)
+			(show_name no)
+			(do_not_autoplace no)
+			(effects
+				(font
+					(size 1.27 1.27)
+				)
+			)
+		)
+		(property "DigiKey EDA Model URL" "https://www.digikey.com/en/models/20414090"
+			(at 96.52 52.07 0)
+			(hide yes)
+			(show_name no)
+			(do_not_autoplace no)
+			(effects
+				(font
+					(size 1.27 1.27)
+				)
+			)
+		)
+		(property "Footprint Source" "Ultra Librarian archive supplied for LMR43620R5RPER; normalized to native KiCad custom pads"
+			(at 96.52 52.07 0)
+			(hide yes)
+			(show_name no)
+			(do_not_autoplace no)
+			(effects
+				(font
+					(size 1.27 1.27)
+				)
+			)
+		)
+		(property "Footprint Audit" "OK: project-local native KiCad footprint derived from supplied Ultra Librarian RPE0009A-MFG data and checked against TI RPE VQFN-HR 9-pin geometry"
+			(at 96.52 52.07 0)
+			(hide yes)

Commit message: ok
Parts:
- U5, U6: footprint EasyEDA:DFN-8_L3.0-W3.0-P0.65-BL-EP -> Package_DFN_QFN:DFN-8-1EP_3x3mm_P0.65mm_EP1.5x2.25mm
Changed lines of the file:
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@@
 			)
 		)
-		(property "Footprint" "EasyEDA:DFN-8_L3.0-W3.0-P0.65-BL-EP"
+		(property "Footprint" "Package_DFN_QFN:DFN-8-1EP_3x3mm_P0.65mm_EP1.5x2.25mm"
 			(at 237.49 134.62 0)
 			(hide yes)
@@
 			)
 		)
-		(property "Footprint" "EasyEDA:DFN-8_L3.0-W3.0-P0.65-BL-EP"
+		(property "Footprint" "Package_DFN_QFN:DFN-8-1EP_3x3mm_P0.65mm_EP1.5x2.25mm"
 			(at 237.49 78.74 0)
 			(hide yes)

Commit message: ok
Parts:
- U4: footprint EasyEDA:WQFN-9_L2.5-W2.0_RAK0009A -> H743_Custom:TI_RAK0009A_WQFN-HR-9_2.5x2.0mm
Changed lines of the file:
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@@
 			)
 		)
-		(property "Footprint" "EasyEDA:WQFN-9_L2.5-W2.0_RAK0009A"
+		(property "Footprint" "H743_Custom:TI_RAK0009A_WQFN-HR-9_2.5x2.0mm"
 			(at 104.14 138.43 0)
 			(hide yes)
