File: POWER.kicad_sch (KiCad schematic)
At the start: 32 parts, among them U3 LMR43620R5RPER, U4 LMR604303SRAKRQ1, U5 AP7361C-33FGE-7, U6 AP7361C-33FGE-7

Commit message: Use local RAK0009A footprint and add LMR604303 sourcing metadata
Parts:
- U4: footprint EasyEDA:WQFN-9_L2.5-W2.0_RAK0009A -> H743_Custom:TI_RAK0009A_WQFN-HR-9_2.5x2.0mm; Footprint Audit OK by package name/dimensions; final overlay recommended -> OK: project-local native KiCad footprint for TI RAK0009A WQ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; Footprint Source (none) -> Public KiCad RAK0009A implementation normalized into projec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; Footprint Source URL (none) -> https://github.com/beaked99/air-scales/blob/ab5531a3598be3d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; LCSC URL (none) -> https://www.lcsc.com/product-detail/C49292342.html; Mouser URL (none) -> https://www.mouser.com/ProductDetail/Texas-Instruments/LMR6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; TI Datasheet PDF (none) -> https://www.ti.com/lit/ds/symlink/lmr60430-q1.pdf; TI Product URL (none) -> https://www.ti.com/product/LMR60430-Q1/part-details/LMR6043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
- U5: Library Audit EasyEDA external -> Project-local H743_Custom footprint; no EasyEDA footprint d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
Changed lines of the file:
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@@
 			)
 		)
-		(property "Library Audit" "EasyEDA external"
+		(property "Library Audit" "Project-local H743_Custom footprint; no EasyEDA footprint dependency"
 			(at 237.49 53.34 0)
 			(hide yes)
@@
 			)
 		)
-		(property "Footprint" "EasyEDA:WQFN-9_L2.5-W2.0_RAK0009A"
+		(property "Footprint" "H743_Custom:TI_RAK0009A_WQFN-HR-9_2.5x2.0mm"
 			(at 104.14 138.43 0)
 			(hide yes)
@@
 			)
 		)
-		(property "Footprint Audit" "OK by package name/dimensions; final overlay recommended"
+		(property "TI Product URL" "https://www.ti.com/product/LMR60430-Q1/part-details/LMR604303SRAKRQ1"
+			(at 104.14 113.03 0)
+			(hide yes)
+			(show_name no)
+			(do_not_autoplace no)
+			(effects
+				(font
+					(size 1.27 1.27)
+				)
+			)
+		)
+		(property "TI Datasheet PDF" "https://www.ti.com/lit/ds/symlink/lmr60430-q1.pdf"
+			(at 104.14 113.03 0)
+			(hide yes)
+			(show_name no)
+			(do_not_autoplace no)
+			(effects
+				(font
+					(size 1.27 1.27)
+				)
+			)
+		)
+		(property "Mouser URL" "https://www.mouser.com/ProductDetail/Texas-Instruments/LMR604303SRAKRQ1"
+			(at 104.14 113.03 0)
+			(hide yes)
+			(show_name no)
+			(do_not_autoplace no)
+			(effects
+				(font
+					(size 1.27 1.27)
+				)
+			)
+		)
+		(property "LCSC URL" "https://www.lcsc.com/product-detail/C49292342.html"
+			(at 104.14 113.03 0)
+			(hide yes)
+			(show_name no)
+			(do_not_autoplace no)
+			(effects
+				(font
+					(size 1.27 1.27)
+				)
+			)
+		)
+		(property "Footprint Source URL" "https://github.com/beaked99/air-scales/blob/ab5531a3598be3d716514b864d2fc2af20bb4d99/hardware/LMR604xx/footprints.pretty/RAK0009A-MFG.kicad_mod"
+			(at 104.14 113.03 0)
+			(hide yes)
+			(show_name no)
+			(do_not_autoplace no)
+			(effects
+				(font
+					(size 1.27 1.27)
+				)
+			)
+		)
+		(property "Footprint Source" "Public KiCad RAK0009A implementation normalized into project-local H743_Custom library"
+			(at 104.14 113.03 0)
+			(hide yes)
+			(show_name no)
+			(do_not_autoplace no)
+			(effects
+				(font
+					(size 1.27 1.27)
+				)
+			)
+		)
+		(property "Footprint Audit" "OK: project-local native KiCad footprint for TI RAK0009A WQFN-HR-9 2.5x2.0 mm, sourced from a public KiCad implementation and checked against TI package geometry"
 			(at 104.14 113.03 0)
 			(hide yes)

Commit message: Localize power IC symbols and verify AP7361C package
Parts:
- U3: symbol EasyEDA:LMR43620R5RPER -> H743_Ardupilot:LMR43620R5RPER; Library Audit EasyEDA external -> Project-local verified symbol + KiCad standard footprint
- U4: symbol EasyEDA:LMR604303SRAKRQ1 -> H743_Ardupilot:LMR604303SRAKRQ1; Library Audit EasyEDA external -> Project-local verified symbol + KiCad standard footprint
- U5, U6: symbol EasyEDA:AP7361C-33FGE-7 -> H743_Ardupilot:AP7361C-33FGE-7; Farnell URL (none) -> https://de.farnell.com/diodes-inc/ap7361c-33fge-7/ldo-fests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; Mouser URL (none) -> https://www.mouser.com/en/ProductDetail/Diodes-Incorporated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; Supplier Specs (none) -> Fixed 3.3 V LDO, 1 A, Vin 2.2-6 V, U-DFN3030-8 Type E
Changed lines of the file:
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@@
 	)
 	(symbol
-		(lib_id "EasyEDA:AP7361C-33FGE-7")
+		(lib_id "H743_Ardupilot:AP7361C-33FGE-7")
 		(at 237.49 121.92 0)
 		(unit 1)
@@
 			)
 		)
+		(property "Supplier Specs" "Fixed 3.3 V LDO, 1 A, Vin 2.2-6 V, U-DFN3030-8 Type E"
+			(at 237.49 142.24 0)
+			(hide yes)
+			(show_name no)
+			(do_not_autoplace no)
+			(effects (font (size 1.27 1.27)))
+		)
+		(property "Farnell URL" "https://de.farnell.com/diodes-inc/ap7361c-33fge-7/ldo-festsp-regl-3-3v-1a-40-bis/dp/3482979"
+			(at 237.49 142.24 0)
+			(hide yes)
+			(show_name no)
+			(do_not_autoplace no)
+			(effects (font (size 1.27 1.27)))
+		)
+		(property "Mouser URL" "https://www.mouser.com/en/ProductDetail/Diodes-Incorporated/AP7361C-33FGE-7"
+			(at 237.49 142.24 0)
+			(hide yes)
+			(show_name no)
+			(do_not_autoplace no)
+			(effects (font (size 1.27 1.27)))
+		)
 		(property "LCSC Part" "C151007"
 			(at 237.49 144.78 0)
@@
 	)
 	(symbol
-		(lib_id "EasyEDA:AP7361C-33FGE-7")
+		(lib_id "H743_Ardupilot:AP7361C-33FGE-7")
 		(at 237.49 66.04 0)
 		(unit 1)
@@
 			)
 		)
+		(property "Supplier Specs" "Fixed 3.3 V LDO, 1 A, Vin 2.2-6 V, U-DFN3030-8 Type E"
+			(at 237.49 86.36 0)
+			(hide yes)
+			(show_name no)
+			(do_not_autoplace no)
+			(effects (font (size 1.27 1.27)))
+		)
+		(property "Farnell URL" "https://de.farnell.com/diodes-inc/ap7361c-33fge-7/ldo-festsp-regl-3-3v-1a-40-bis/dp/3482979"
+			(at 237.49 86.36 0)
+			(hide yes)
+			(show_name no)
+			(do_not_autoplace no)
+			(effects (font (size 1.27 1.27)))
+		)
+		(property "Mouser URL" "https://www.mouser.com/en/ProductDetail/Diodes-Incorporated/AP7361C-33FGE-7"
+			(at 237.49 86.36 0)
+			(hide yes)
+			(show_name no)
+			(do_not_autoplace no)
+			(effects (font (size 1.27 1.27)))
+		)
 		(property "LCSC Part" "C151007"
 			(at 237.49 88.9 0)
@@
 	)
 	(symbol
-		(lib_id "EasyEDA:LMR43620R5RPER")
+		(lib_id "H743_Ardupilot:LMR43620R5RPER")
 		(at 96.52 67.31 0)
 		(unit 1)
@@
 			)
 		)
-		(property "Library Audit" "EasyEDA external"
+		(property "Library Audit" "Project-local verified symbol + KiCad standard footprint"
 			(at 96.52 52.07 0)
 			(hide yes)
@@
 	)
 	(symbol
-		(lib_id "EasyEDA:LMR604303SRAKRQ1")
+		(lib_id "H743_Ardupilot:LMR604303SRAKRQ1")
 		(at 104.14 125.73 0)
 		(unit 1)
@@
 			)
 		)
-		(property "Library Audit" "EasyEDA external"
+		(property "Library Audit" "Project-local verified symbol + KiCad standard footprint"
 			(at 104.14 113.03 0)
 			(hide yes)

Commit message: Fix CAN schematic symbol and update SMAJ30CA footprint
Parts:
- D2: footprint Diode_SMD:D_SMA -> H743_Custom:SMAJ30CA_SMA_LTF; Footprint Audit OK -> VERIFIED: supplied SMAJ30CA.zip nominal SMASeries_LTF land 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; Library Audit KiCad standard -> Project-local H743_Custom footprint
Changed lines of the file:
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@@
 			)
 		)
-		(property "Footprint" "Diode_SMD:D_SMA"
+		(property "Footprint" "H743_Custom:SMAJ30CA_SMA_LTF"
 			(at 35.56 66.04 0)
 			(hide yes)
@@
 			)
 		)
-		(property "Footprint Audit" "OK"
+		(property "Footprint Audit" "VERIFIED: supplied SMAJ30CA.zip nominal SMASeries_LTF land pattern; pads 1.651 x 2.1844 mm at +/-1.7018 mm"
 			(at 33.02 63.5 90)
 			(hide yes)
@@
 			)
 		)
-		(property "Library Audit" "KiCad standard"
+		(property "Library Audit" "Project-local H743_Custom footprint"
 			(at 33.02 63.5 90)
 			(hide yes)

Commit message: Use dedicated SMAJ30CA footprint library for D2
Parts:
- D2: footprint H743_Custom:SMAJ30CA_SMA_LTF -> SMAJ30CA:SMASeries_LTF
Changed lines of the file:
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@@
 			)
 		)
-		(property "Footprint" "H743_Custom:SMAJ30CA_SMA_LTF"
+		(property "Footprint" "SMAJ30CA:SMASeries_LTF"
 			(at 35.56 66.04 0)
 			(hide yes)
