File: ANALOG_SENS.kicad_sch (KiCad schematic)
At the start: 10 parts, among them J11 Conn_01x04

Commit message: add ANALOG_SENS sheet
Parts:
- renumbered C17 to C1, C33 to C10, C19 to C7, J11 to J2, R13 to R10, R14 to R11, R21 to R12, R22 to R13, R10 to R8, R11 to R9
Connections:
- net ADC_VBAT1: now also C10.1, R12.2, R13.1
- net ADC_VBAT2: no longer C10.1, R12.2, R13.1
Other:
- title: H743_ARDUPILOT -> (none)
- moved on the sheet: C1, C10, C7, J2, R10, R11, R12, R13, R8, R9

Commit message: delete unused sheet
Parts:
- renumbered C1 to C17, C7 to C19, C10 to C33, J2 to J11, R8 to R10, R9 to R11, R10 to R13, R11 to R14, R12 to R21, R13 to R22
Changed lines of the file:
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@@
 		(dnp no)
 		(fields_autoplaced yes)
-		(property "Reference" "R11"
+		(property "Reference" "R14"
 			(at 102.87 74.9299 0)
 			(show_name no)
@@
 				(path "/6b768b36-fce6-4be0-9021-6d41bddc3a70/05a39706-93dd-4215-aab0-0781f7da02e1"
 					(reference "R14")
-					(unit 1)
-				)
-				(path "/6b768b36-fce6-4be0-9021-6d41bddc3a70/35dc580c-330e-4c18-9b1d-970b7f83579d"
-					(reference "R11")
 					(unit 1)
 				)
@@
 					(unit 1)
 				)
-				(path "/6b768b36-fce6-4be0-9021-6d41bddc3a70/35dc580c-330e-4c18-9b1d-970b7f83579d"
-					(reference "#PWR066")
-					(unit 1)
-				)
 			)
 		)
@@
 		(dnp no)
 		(fields_autoplaced yes)
-		(property "Reference" "R8"
+		(property "Reference" "R10"
 			(at 71.12 67.3099 0)
 			(show_name no)
@@
 				(path "/6b768b36-fce6-4be0-9021-6d41bddc3a70/05a39706-93dd-4215-aab0-0781f7da02e1"
 					(reference "R10")
-					(unit 1)
-				)
-				(path "/6b768b36-fce6-4be0-9021-6d41bddc3a70/35dc580c-330e-4c18-9b1d-970b7f83579d"
-					(reference "R8")
 					(unit 1)
 				)
@@
 		(in_pos_files yes)
 		(dnp no)
-		(property "Reference" "C10"
+		(property "Reference" "C33"
 			(at 125.73 74.9362 0)
 			(show_name no)
@@
 				(path "/6b768b36-fce6-4be0-9021-6d41bddc3a70/05a39706-93dd-4215-aab0-0781f7da02e1"
 					(reference "C33")
-					(unit 1)
-				)
-				(path "/6b768b36-fce6-4be0-9021-6d41bddc3a70/35dc580c-330e-4c18-9b1d-970b7f83579d"
-					(reference "C10")
 					(unit 1)
 				)
@@
 					(unit 1)
 				)
-				(path "/6b768b36-fce6-4be0-9021-6d41bddc3a70/35dc580c-330e-4c18-9b1d-970b7f83579d"
-					(reference "#PWR073")
-					(unit 1)
-				)
 			)
 		)
@@
 		(dnp no)
 		(fields_autoplaced yes)
-		(property "Reference" "R10"
+		(property "Reference" "R13"
 			(at 102.87 67.3099 0)
 			(show_name no)
@@
 				(path "/6b768b36-fce6-4be0-9021-6d41bddc3a70/05a39706-93dd-4215-aab0-0781f7da02e1"
 					(reference "R13")
-					(unit 1)
-				)
-				(path "/6b768b36-fce6-4be0-9021-6d41bddc3a70/35dc580c-330e-4c18-9b1d-970b7f83579d"
-					(reference "R10")
 					(unit 1)
 				)
@@
 		(in_pos_files yes)
 		(dnp no)
-		(property "Reference" "C7"
+		(property "Reference" "C19"
 			(at 93.98 74.9362 0)
 			(show_name no)
@@
 				(path "/6b768b36-fce6-4be0-9021-6d41bddc3a70/05a39706-93dd-4215-aab0-0781f7da02e1"
 					(reference "C19")
-					(unit 1)
-				)
-				(path "/6b768b36-fce6-4be0-9021-6d41bddc3a70/35dc580c-330e-4c18-9b1d-970b7f83579d"
-					(reference "C7")
 					(unit 1)
 				)
@@
 		(in_pos_files yes)
 		(dnp no)
-		(property "Reference" "C1"
+		(property "Reference" "C17"
 			(at 62.23 74.9362 0)
 			(show_name no)
@@
 				(path "/6b768b36-fce6-4be0-9021-6d41bddc3a70/05a39706-93dd-4215-aab0-0781f7da02e1"
 					(reference "C17")
-					(unit 1)
-				)
-				(path "/6b768b36-fce6-4be0-9021-6d41bddc3a70/35dc580c-330e-4c18-9b1d-970b7f83579d"
-					(reference "C1")
 					(unit 1)
 				)
@@
 			(project "H743_Ardupilot"
 				(path "/6b768b36-fce6-4be0-9021-6d41bddc3a70/05a39706-93dd-4215-aab0-0781f7da02e1"
-					(reference "#PWR036")
-					(unit 1)
-				)
-				(path "/6b768b36-fce6-4be0-9021-6d41bddc3a70/35dc580c-330e-4c18-9b1d-970b7f83579d"
 					(reference "#PWR036")
 					(unit 1)
@@
 					(unit 1)
 				)
-				(path "/6b768b36-fce6-4be0-9021-6d41bddc3a70/35dc580c-330e-4c18-9b1d-970b7f83579d"
-					(reference "#PWR072")
-					(unit 1)
-				)
 			)
 		)
@@
 					(unit 1)
 				)
-				(path "/6b768b36-fce6-4be0-9021-6d41bddc3a70/35dc580c-330e-4c18-9b1d-970b7f83579d"
-					(reference "#PWR040")
-					(unit 1)
-				)
 			)
 		)
@@
 		(dnp no)
 		(fields_autoplaced yes)
-		(property "Reference" "R9"
+		(property "Reference" "R11"
 			(at 71.12 74.9299 0)
 			(show_name no)
@@
 				(path "/6b768b36-fce6-4be0-9021-6d41bddc3a70/05a39706-93dd-4215-aab0-0781f7da02e1"
 					(reference "R11")
-					(unit 1)
-				)
-				(path "/6b768b36-fce6-4be0-9021-6d41bddc3a70/35dc580c-330e-4c18-9b1d-970b7f83579d"
-					(reference "R9")
 					(unit 1)
 				)
@@
 		(dnp no)
 		(fields_autoplaced yes)
-		(property "Reference" "R13"
+		(property "Reference" "R22"
 			(at 134.62 74.9299 0)
 			(show_name no)
@@
 				(path "/6b768b36-fce6-4be0-9021-6d41bddc3a70/05a39706-93dd-4215-aab0-0781f7da02e1"
 					(reference "R22")
-					(unit 1)
-				)
-				(path "/6b768b36-fce6-4be0-9021-6d41bddc3a70/35dc580c-330e-4c18-9b1d-970b7f83579d"
-					(reference "R13")
 					(unit 1)
 				)
@@
 					(unit 1)
 				)
-				(path "/6b768b36-fce6-4be0-9021-6d41bddc3a70/35dc580c-330e-4c18-9b1d-970b7f83579d"
-					(reference "#PWR043")
-					(unit 1)
-				)
 			)
 		)
@@
 					(unit 1)
 				)
-				(path "/6b768b36-fce6-4be0-9021-6d41bddc3a70/35dc580c-330e-4c18-9b1d-970b7f83579d"
-					(reference "#PWR037")
-					(unit 1)
-				)
 			)
 		)
@@
 					(unit 1)
 				)
-				(path "/6b768b36-fce6-4be0-9021-6d41bddc3a70/35dc580c-330e-4c18-9b1d-970b7f83579d"
-					(reference "#PWR033")
-					(unit 1)
-				)
 			)
 		)
@@
 		(dnp no)
 		(fields_autoplaced yes)
-		(property "Reference" "R12"
+		(property "Reference" "R21"
 			(at 134.62 67.3099 0)
 			(show_name no)
@@
 				(path "/6b768b36-fce6-4be0-9021-6d41bddc3a70/05a39706-93dd-4215-aab0-0781f7da02e1"
 					(reference "R21")
-					(unit 1)
-				)
-				(path "/6b768b36-fce6-4be0-9021-6d41bddc3a70/35dc580c-330e-4c18-9b1d-970b7f83579d"
-					(reference "R12")
 					(unit 1)
 				)
@@
 					(unit 1)
 				)
-				(path "/6b768b36-fce6-4be0-9021-6d41bddc3a70/35dc580c-330e-4c18-9b1d-970b7f83579d"
-					(reference "#PWR074")
-					(unit 1)
-				)
 			)
 		)
@@
 		(dnp no)
 		(fields_autoplaced yes)
-		(property "Reference" "J2"
+		(property "Reference" "J11"
 			(at 109.22 39.37 90)
 			(show_name no)
@@
 					(unit 1)
 				)
-				(path "/6b768b36-fce6-4be0-9021-6d41bddc3a70/35dc580c-330e-4c18-9b1d-970b7f83579d"
-					(reference "J2")
-					(unit 1)
-				)

Commit message: re annotate componant globaly
Parts:
- renumbered C17 to C16, C19 to C17, C33 to C18, J11 to J1, R13 to R10, R14 to R11, R21 to R12, R22 to R13, R10 to R8, R11 to R9
Other:
- title: (none) -> H743_ARDUPILOT
Changed lines of the file:
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@@
 	(paper "A5")
 	(title_block
+		(title "H743_ARDUPILOT")
 		(date "2026-09-24")
 	)
@@
 		(dnp no)
 		(fields_autoplaced yes)
-		(property "Reference" "R14"
+		(property "Reference" "R11"
 			(at 102.87 74.9299 0)
 			(show_name no)
@@
 			(project "H743_Ardupilot"
 				(path "/6b768b36-fce6-4be0-9021-6d41bddc3a70/05a39706-93dd-4215-aab0-0781f7da02e1"
-					(reference "R14")
+					(reference "R11")
 					(unit 1)
 				)
@@
 		(dnp no)
 		(fields_autoplaced yes)
-		(property "Reference" "#PWR066"
+		(property "Reference" "#PWR031"
 			(at 123.19 87.63 0)
 			(hide yes)
@@
 			(project "H743_Ardupilot"
 				(path "/6b768b36-fce6-4be0-9021-6d41bddc3a70/05a39706-93dd-4215-aab0-0781f7da02e1"
-					(reference "#PWR066")
+					(reference "#PWR031")
 					(unit 1)
 				)
@@
 		(dnp no)
 		(fields_autoplaced yes)
-		(property "Reference" "R10"
+		(property "Reference" "R8"
 			(at 71.12 67.3099 0)
 			(show_name no)
@@
 			(project "H743_Ardupilot"
 				(path "/6b768b36-fce6-4be0-9021-6d41bddc3a70/05a39706-93dd-4215-aab0-0781f7da02e1"
-					(reference "R10")
+					(reference "R8")
 					(unit 1)
 				)
@@
 		(in_pos_files yes)
 		(dnp no)
-		(property "Reference" "C33"
+		(property "Reference" "C18"
 			(at 125.73 74.9362 0)
 			(show_name no)
@@
 			(project "H743_Ardupilot"
 				(path "/6b768b36-fce6-4be0-9021-6d41bddc3a70/05a39706-93dd-4215-aab0-0781f7da02e1"
-					(reference "C33")
+					(reference "C18")
 					(unit 1)
 				)
@@
 		(in_pos_files yes)
 		(dnp no)
-		(property "Reference" "#PWR073"
+		(property "Reference" "#PWR029"
 			(at 107.95 57.15 0)
 			(hide yes)
@@
 			(project "H743_Ardupilot"
 				(path "/6b768b36-fce6-4be0-9021-6d41bddc3a70/05a39706-93dd-4215-aab0-0781f7da02e1"
-					(reference "#PWR073")
+					(reference "#PWR029")
 					(unit 1)
 				)
@@
 		(dnp no)
 		(fields_autoplaced yes)
-		(property "Reference" "R13"
+		(property "Reference" "R10"
 			(at 102.87 67.3099 0)
 			(show_name no)
@@
 			(project "H743_Ardupilot"
 				(path "/6b768b36-fce6-4be0-9021-6d41bddc3a70/05a39706-93dd-4215-aab0-0781f7da02e1"
-					(reference "R13")
+					(reference "R10")
 					(unit 1)
 				)
@@
 		(in_pos_files yes)
 		(dnp no)
-		(property "Reference" "C19"
+		(property "Reference" "C17"
 			(at 93.98 74.9362 0)
 			(show_name no)
@@
 			(project "H743_Ardupilot"
 				(path "/6b768b36-fce6-4be0-9021-6d41bddc3a70/05a39706-93dd-4215-aab0-0781f7da02e1"
-					(reference "C19")
+					(reference "C17")
 					(unit 1)
 				)
@@
 		(in_pos_files yes)
 		(dnp no)
-		(property "Reference" "C17"
+		(property "Reference" "C16"
 			(at 62.23 74.9362 0)
 			(show_name no)
@@
 			(project "H743_Ardupilot"
 				(path "/6b768b36-fce6-4be0-9021-6d41bddc3a70/05a39706-93dd-4215-aab0-0781f7da02e1"
-					(reference "C17")
+					(reference "C16")
 					(unit 1)
 				)
@@
 		(in_pos_files yes)
 		(dnp no)
-		(property "Reference" "#PWR036"
+		(property "Reference" "#PWR025"
 			(at 68.58 67.31 0)
 			(hide yes)
@@
 			(project "H743_Ardupilot"
 				(path "/6b768b36-fce6-4be0-9021-6d41bddc3a70/05a39706-93dd-4215-aab0-0781f7da02e1"
-					(reference "#PWR036")
+					(reference "#PWR025")
 					(unit 1)
 				)
@@
 		(dnp no)
 		(fields_autoplaced yes)
-		(property "Reference" "#PWR072"
+		(property "Reference" "#PWR032"
 			(at 132.08 87.63 0)
 			(hide yes)
@@
 			(project "H743_Ardupilot"
 				(path "/6b768b36-fce6-4be0-9021-6d41bddc3a70/05a39706-93dd-4215-aab0-0781f7da02e1"
-					(reference "#PWR072")
+					(reference "#PWR032")
 					(unit 1)
 				)
@@
 		(dnp no)
 		(fields_autoplaced yes)
-		(property "Reference" "#PWR040"
+		(property "Reference" "#PWR027"
 			(at 91.44 87.63 0)
 			(hide yes)
@@
 			(project "H743_Ardupilot"
 				(path "/6b768b36-fce6-4be0-9021-6d41bddc3a70/05a39706-93dd-4215-aab0-0781f7da02e1"
-					(reference "#PWR040")
+					(reference "#PWR027")
 					(unit 1)
 				)
@@
 		(dnp no)
 		(fields_autoplaced yes)
-		(property "Reference" "R11"
+		(property "Reference" "R9"
 			(at 71.12 74.9299 0)
 			(show_name no)
@@
 			(project "H743_Ardupilot"
 				(path "/6b768b36-fce6-4be0-9021-6d41bddc3a70/05a39706-93dd-4215-aab0-0781f7da02e1"
-					(reference "R11")
+					(reference "R9")
 					(unit 1)
 				)
@@
 		(dnp no)
 		(fields_autoplaced yes)
-		(property "Reference" "R22"
+		(property "Reference" "R13"
 			(at 134.62 74.9299 0)
 			(show_name no)
@@
 			(project "H743_Ardupilot"
 				(path "/6b768b36-fce6-4be0-9021-6d41bddc3a70/05a39706-93dd-4215-aab0-0781f7da02e1"
-					(reference "R22")
+					(reference "R13")
 					(unit 1)
 				)
@@
 		(dnp no)
 		(fields_autoplaced yes)
-		(property "Reference" "#PWR043"
+		(property "Reference" "#PWR028"
 			(at 100.33 87.63 0)
 			(hide yes)
@@
 			(project "H743_Ardupilot"
 				(path "/6b768b36-fce6-4be0-9021-6d41bddc3a70/05a39706-93dd-4215-aab0-0781f7da02e1"
-					(reference "#PWR043")
+					(reference "#PWR028")
 					(unit 1)
 				)
@@
 		(dnp no)
 		(fields_autoplaced yes)
-		(property "Reference" "#PWR037"
+		(property "Reference" "#PWR026"
 			(at 68.58 87.63 0)
 			(hide yes)
@@
 			(project "H743_Ardupilot"
 				(path "/6b768b36-fce6-4be0-9021-6d41bddc3a70/05a39706-93dd-4215-aab0-0781f7da02e1"
-					(reference "#PWR037")
+					(reference "#PWR026")
 					(unit 1)
 				)
@@
 		(dnp no)
 		(fields_autoplaced yes)
-		(property "Reference" "#PWR033"
+		(property "Reference" "#PWR024"
 			(at 59.69 87.63 0)
 			(hide yes)
@@
 			(project "H743_Ardupilot"
 				(path "/6b768b36-fce6-4be0-9021-6d41bddc3a70/05a39706-93dd-4215-aab0-0781f7da02e1"
-					(reference "#PWR033")
+					(reference "#PWR024")
 					(unit 1)
 				)
@@
 		(dnp no)
 		(fields_autoplaced yes)
-		(property "Reference" "R21"
+		(property "Reference" "R12"
 			(at 134.62 67.3099 0)
 			(show_name no)
@@
 			(project "H743_Ardupilot"
 				(path "/6b768b36-fce6-4be0-9021-6d41bddc3a70/05a39706-93dd-4215-aab0-0781f7da02e1"
-					(reference "R21")
+					(reference "R12")
 					(unit 1)
 				)
@@
 		(in_pos_files yes)
 		(dnp no)
-		(property "Reference" "#PWR074"
+		(property "Reference" "#PWR030"
 			(at 110.49 57.15 0)
 			(hide yes)
@@
 			(project "H743_Ardupilot"
 				(path "/6b768b36-fce6-4be0-9021-6d41bddc3a70/05a39706-93dd-4215-aab0-0781f7da02e1"
-					(reference "#PWR074")
+					(reference "#PWR030")
 					(unit 1)
 				)
@@
 		(dnp no)
 		(fields_autoplaced yes)
-		(property "Reference" "J11"
+		(property "Reference" "J1"
 			(at 109.22 39.37 90)
 			(show_name no)
@@
 			(project "H743_Ardupilot"
 				(path "/6b768b36-fce6-4be0-9021-6d41bddc3a70/05a39706-93dd-4215-aab0-0781f7da02e1"
-					(reference "J11")
+					(reference "J1")
 					(unit 1)
 				)

Commit message: audit DigiKey metadata: ANALOG_SENS.kicad_sch
Parts:
- C16, C17, C18: DigiKey Part Number (none) -> 1276-1001-1-ND; DigiKey Price Qty (none) -> 1 CT; DigiKey Specs (none) -> 100 nF ±10%, 16 V, X7R, 0402; DigiKey Status (none) -> Active; DigiKey URL (none) -> https://www.digikey.fr/fr/products/detail/samsung-electro-m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; DigiKey Unit Price EUR (none) -> 0.09; Footprint Audit (none) -> OK; LCSC C1525 -> (none); LCSC Part C1525 -> (none); Library Audit (none) -> KiCad standard; MPN GRM022R60J104KE15D -> CL05B104KO5NNNC; Manufacturer Murata Electronics -> Samsung Electro-Mechanics; Package (none) -> 0402 (1005); Price Checked (none) -> 2026-09-25
- J1: DigiKey Status (none) -> TBD: connector not physically selected; Footprint Audit (none) -> BLOCKING: no footprint assigned; Library Audit (none) -> Generic KiCad connector; Package (none) -> TBD; Price Checked (none) -> 2026-09-25
- R10, R8: DigiKey Price Qty (none) -> 1 CT; DigiKey Specs (none) -> 10 kΩ ±1%, 0402; DigiKey Status (none) -> Active / family verified; DigiKey URL (none) -> https://www.digikey.fr/en/products/result?keywords=RC0402FR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; DigiKey Unit Price EUR (none) -> 0.09; Footprint Audit (none) -> OK; LCSC C25744 -> (none); LCSC Part C25744 -> (none); Library Audit (none) -> KiCad standard; MPN 0402WGF1002TCE -> RC0402FR-0710KL; Manufacturer UNI-ROYAL(Uniroyal Elec) -> YAGEO; Package (none) -> 0402 (1005); Price Checked (none) -> 2026-09-25
- R11: DigiKey Price Qty (none) -> 1 CT; DigiKey Specs (none) -> 10 kΩ ±1%, 0402; DigiKey Status (none) -> Active / family verified; DigiKey URL (none) -> https://www.digikey.fr/en/products/result?keywords=RC0402FR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; DigiKey Unit Price EUR (none) -> 0.09; Footprint Audit (none) -> OK; LCSC C11702 -> (none); LCSC Part C11702 -> (none); Library Audit (none) -> KiCad standard; MPN 0402WGF1001TCE -> RC0402FR-0710KL; Manufacturer UNI-ROYAL(Uniroyal Elec) -> YAGEO; Package (none) -> 0402 (1005); Price Checked (none) -> 2026-09-25
- R12: DigiKey Price Qty (none) -> 1 CT; DigiKey Specs (none) -> 20 kΩ ±1%, 0402; DigiKey Status (none) -> Active / family verified; DigiKey URL (none) -> https://www.digikey.fr/en/products/result?keywords=RC0402FR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; DigiKey Unit Price EUR (none) -> 0.09; Footprint Audit (none) -> OK; LCSC C25744 -> (none); LCSC Part C25744 -> (none); Library Audit (none) -> KiCad standard; MPN 0402WGF1002TCE -> RC0402FR-0720KL; Manufacturer UNI-ROYAL(Uniroyal Elec) -> YAGEO; Package (none) -> 0402 (1005); Price Checked (none) -> 2026-09-25
- R13, R9: DigiKey Price Qty (none) -> 1 CT; DigiKey Specs (none) -> 1 kΩ ±1%, 0402; DigiKey Status (none) -> Active / family verified; DigiKey URL (none) -> https://www.digikey.fr/en/products/result?keywords=RC0402FR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; DigiKey Unit Price EUR (none) -> 0.09; Footprint Audit (none) -> OK; LCSC C11702 -> (none); LCSC Part C11702 -> (none); Library Audit (none) -> KiCad standard; MPN 0402WGF1001TCE -> RC0402FR-071KL; Manufacturer UNI-ROYAL(Uniroyal Elec) -> YAGEO; Package (none) -> 0402 (1005); Price Checked (none) -> 2026-09-25

Commit message: assign Matek-style solder pad footprints in ANALOG_SENS.kicad_sch
Parts:
- J1: footprint (none) -> H743_Custom:SolderPadArray_1x04_P2.54mm_1x1mm; DigiKey Status TBD: connector not physically selected -> PCB feature / no purchased component; Footprint Audit BLOCKING: no footprint assigned -> OK: 4 square SMD pads 1.00x1.00 mm, P2.54 mm, no holes, no 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; Library Audit Generic KiCad connector -> Project-local H743_Custom footprint; Package TBD -> Solder pad array 1x4, P2.54 mm, 1.00x1.00 mm SMD
Changed lines of the file:
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@@
 			)
 		)
-		(property "Footprint" ""
+		(property "Footprint" "H743_Custom:SolderPadArray_1x04_P2.54mm_1x1mm"
 			(at 107.95 45.72 0)
 			(hide yes)
@@
 			)
 		)
-		(property "DigiKey Status" "TBD: connector not physically selected"
+		(property "DigiKey Status" "PCB feature / no purchased component"
 			(at 109.22 39.37 90)
 			(hide yes)
@@
 			)
 		)
-		(property "Package" "TBD"
+		(property "Package" "Solder pad array 1x4, P2.54 mm, 1.00x1.00 mm SMD"
 			(at 109.22 39.37 90)
 			(hide yes)
@@
 			)
 		)
-		(property "Footprint Audit" "BLOCKING: no footprint assigned"
+		(property "Footprint Audit" "OK: 4 square SMD pads 1.00x1.00 mm, P2.54 mm, no holes, no paste"
 			(at 109.22 39.37 90)
 			(hide yes)
@@
 			)
 		)
-		(property "Library Audit" "Generic KiCad connector"
+		(property "Library Audit" "Project-local H743_Custom footprint"
 			(at 109.22 39.37 90)
 			(hide yes)
