File: ANALOG_SENS.kicad_sch (KiCad schematic)
At the start: 10 parts, among them J1 Conn_01x04

Commit message: update
Parts:
- renumbered C16 to C33, C17 to C34, C18 to C35, R8 to R14, R9 to R15, R10 to R16, R11 to R17, R12 to R18, R13 to R19
Changed lines of the file:
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@@
 		(dnp no)
 		(fields_autoplaced yes)
-		(property "Reference" "R11"
+		(property "Reference" "R17"
 			(at 102.87 74.9299 0)
 			(show_name no)
@@
 			(project "H743_Ardupilot"
 				(path "/6b768b36-fce6-4be0-9021-6d41bddc3a70/05a39706-93dd-4215-aab0-0781f7da02e1"
-					(reference "R11")
+					(reference "R17")
 					(unit 1)
 				)
@@
 		(dnp no)
 		(fields_autoplaced yes)
-		(property "Reference" "#PWR031"
+		(property "Reference" "#PWR060"
 			(at 123.19 87.63 0)
 			(hide yes)
@@
 			(project "H743_Ardupilot"
 				(path "/6b768b36-fce6-4be0-9021-6d41bddc3a70/05a39706-93dd-4215-aab0-0781f7da02e1"
-					(reference "#PWR031")
+					(reference "#PWR060")
 					(unit 1)
 				)
@@
 		(dnp no)
 		(fields_autoplaced yes)
-		(property "Reference" "R8"
+		(property "Reference" "R14"
 			(at 71.12 67.3099 0)
 			(show_name no)
@@
 			(project "H743_Ardupilot"
 				(path "/6b768b36-fce6-4be0-9021-6d41bddc3a70/05a39706-93dd-4215-aab0-0781f7da02e1"
-					(reference "R8")
+					(reference "R14")
 					(unit 1)
 				)
@@
 		(in_pos_files yes)
 		(dnp no)
-		(property "Reference" "C18"
+		(property "Reference" "C35"
 			(at 125.73 74.9362 0)
 			(show_name no)
@@
 			(project "H743_Ardupilot"
 				(path "/6b768b36-fce6-4be0-9021-6d41bddc3a70/05a39706-93dd-4215-aab0-0781f7da02e1"
-					(reference "C18")
+					(reference "C35")
 					(unit 1)
 				)
@@
 		(in_pos_files yes)
 		(dnp no)
-		(property "Reference" "#PWR029"
+		(property "Reference" "#PWR058"
 			(at 107.95 57.15 0)
 			(hide yes)
@@
 			(project "H743_Ardupilot"
 				(path "/6b768b36-fce6-4be0-9021-6d41bddc3a70/05a39706-93dd-4215-aab0-0781f7da02e1"
-					(reference "#PWR029")
+					(reference "#PWR058")
 					(unit 1)
 				)
@@
 		(dnp no)
 		(fields_autoplaced yes)
-		(property "Reference" "R10"
+		(property "Reference" "R16"
 			(at 102.87 67.3099 0)
 			(show_name no)
@@
 			(project "H743_Ardupilot"
 				(path "/6b768b36-fce6-4be0-9021-6d41bddc3a70/05a39706-93dd-4215-aab0-0781f7da02e1"
-					(reference "R10")
+					(reference "R16")
 					(unit 1)
 				)
@@
 		(in_pos_files yes)
 		(dnp no)
-		(property "Reference" "C17"
+		(property "Reference" "C34"
 			(at 93.98 74.9362 0)
 			(show_name no)
@@
 			(project "H743_Ardupilot"
 				(path "/6b768b36-fce6-4be0-9021-6d41bddc3a70/05a39706-93dd-4215-aab0-0781f7da02e1"
-					(reference "C17")
+					(reference "C34")
 					(unit 1)
 				)
@@
 		(in_pos_files yes)
 		(dnp no)
-		(property "Reference" "C16"
+		(property "Reference" "C33"
 			(at 62.23 74.9362 0)
 			(show_name no)
@@
 			(project "H743_Ardupilot"
 				(path "/6b768b36-fce6-4be0-9021-6d41bddc3a70/05a39706-93dd-4215-aab0-0781f7da02e1"
-					(reference "C16")
+					(reference "C33")
 					(unit 1)
 				)
@@
 		(in_pos_files yes)
 		(dnp no)
-		(property "Reference" "#PWR025"
+		(property "Reference" "#PWR054"
 			(at 68.58 67.31 0)
 			(hide yes)
@@
 			(project "H743_Ardupilot"
 				(path "/6b768b36-fce6-4be0-9021-6d41bddc3a70/05a39706-93dd-4215-aab0-0781f7da02e1"
-					(reference "#PWR025")
+					(reference "#PWR054")
 					(unit 1)
 				)
@@
 		(dnp no)
 		(fields_autoplaced yes)
-		(property "Reference" "#PWR032"
+		(property "Reference" "#PWR061"
 			(at 132.08 87.63 0)
 			(hide yes)
@@
 			(project "H743_Ardupilot"
 				(path "/6b768b36-fce6-4be0-9021-6d41bddc3a70/05a39706-93dd-4215-aab0-0781f7da02e1"
-					(reference "#PWR032")
+					(reference "#PWR061")
 					(unit 1)
 				)
@@
 		(dnp no)
 		(fields_autoplaced yes)
-		(property "Reference" "#PWR027"
+		(property "Reference" "#PWR056"
 			(at 91.44 87.63 0)
 			(hide yes)
@@
 			(project "H743_Ardupilot"
 				(path "/6b768b36-fce6-4be0-9021-6d41bddc3a70/05a39706-93dd-4215-aab0-0781f7da02e1"
-					(reference "#PWR027")
+					(reference "#PWR056")
 					(unit 1)
 				)
@@
 		(dnp no)
 		(fields_autoplaced yes)
-		(property "Reference" "R9"
+		(property "Reference" "R15"
 			(at 71.12 74.9299 0)
 			(show_name no)
@@
 			(project "H743_Ardupilot"
 				(path "/6b768b36-fce6-4be0-9021-6d41bddc3a70/05a39706-93dd-4215-aab0-0781f7da02e1"
-					(reference "R9")
+					(reference "R15")
 					(unit 1)
 				)
@@
 		(dnp no)
 		(fields_autoplaced yes)
-		(property "Reference" "R13"
+		(property "Reference" "R19"
 			(at 134.62 74.9299 0)
 			(show_name no)
@@
 			(project "H743_Ardupilot"
 				(path "/6b768b36-fce6-4be0-9021-6d41bddc3a70/05a39706-93dd-4215-aab0-0781f7da02e1"
-					(reference "R13")
+					(reference "R19")
 					(unit 1)
 				)
@@
 		(dnp no)
 		(fields_autoplaced yes)
-		(property "Reference" "#PWR028"
+		(property "Reference" "#PWR057"
 			(at 100.33 87.63 0)
 			(hide yes)
@@
 			(project "H743_Ardupilot"
 				(path "/6b768b36-fce6-4be0-9021-6d41bddc3a70/05a39706-93dd-4215-aab0-0781f7da02e1"
-					(reference "#PWR028")
+					(reference "#PWR057")
 					(unit 1)
 				)
@@
 		(dnp no)
 		(fields_autoplaced yes)
-		(property "Reference" "#PWR026"
+		(property "Reference" "#PWR055"
 			(at 68.58 87.63 0)
 			(hide yes)
@@
 			(project "H743_Ardupilot"
 				(path "/6b768b36-fce6-4be0-9021-6d41bddc3a70/05a39706-93dd-4215-aab0-0781f7da02e1"
-					(reference "#PWR026")
+					(reference "#PWR055")
 					(unit 1)
 				)
@@
 		(dnp no)
 		(fields_autoplaced yes)
-		(property "Reference" "#PWR024"
+		(property "Reference" "#PWR053"
 			(at 59.69 87.63 0)
 			(hide yes)
@@
 			(project "H743_Ardupilot"
 				(path "/6b768b36-fce6-4be0-9021-6d41bddc3a70/05a39706-93dd-4215-aab0-0781f7da02e1"
-					(reference "#PWR024")
+					(reference "#PWR053")
 					(unit 1)
 				)
@@
 		(dnp no)
 		(fields_autoplaced yes)
-		(property "Reference" "R12"
+		(property "Reference" "R18"
 			(at 134.62 67.3099 0)
 			(show_name no)
@@
 			(project "H743_Ardupilot"
 				(path "/6b768b36-fce6-4be0-9021-6d41bddc3a70/05a39706-93dd-4215-aab0-0781f7da02e1"
-					(reference "R12")
+					(reference "R18")
 					(unit 1)
 				)
@@
 		(in_pos_files yes)
 		(dnp no)
-		(property "Reference" "#PWR030"
+		(property "Reference" "#PWR059"
 			(at 110.49 57.15 0)
 			(hide yes)
@@
 			(project "H743_Ardupilot"
 				(path "/6b768b36-fce6-4be0-9021-6d41bddc3a70/05a39706-93dd-4215-aab0-0781f7da02e1"
-					(reference "#PWR030")
+					(reference "#PWR059")
 					(unit 1)
 				)
