File: ANALOG_SENS.kicad_sch (KiCad schematic)
At the start: 10 parts, among them J1 Analog

Commit message: Review component footprints, restore local libraries and reconcile PCB pads
Parts:
- C33, C34, C35: symbol Device:C_Small -> FC01_Project:ANALOG_SENS__C_Small; Footprint Audit OK -> See verification/COMPONENTS.csv and verification/REPORT.md; Library Audit KiCad standard -> See verification/COMPONENTS.csv and verification/REPORT.md
- J1: symbol Connector_Generic:Conn_01x04 -> FC01_Project:ANALOG_SENS__Conn_01x04; Footprint Audit OK: 4 square SMD pads 1.00x1.00 mm, P2.54 mm, no holes, no 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 -> See verification/COMPONENTS.csv and verification/REPORT.md; Library Audit Project-local H743_Custom footprint -> See verification/COMPONENTS.csv and verification/REPORT.md
- R14, R15, R16, R17, R18, R19: symbol Device:R_Small -> FC01_Project:ANALOG_SENS__R_Small; Footprint Audit OK -> See verification/COMPONENTS.csv and verification/REPORT.md; Library Audit KiCad standard -> See verification/COMPONENTS.csv and verification/REPORT.md
Changed lines of the file:
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@@
 	)
 	(symbol
-		(lib_id "Device:R_Small")
+		(lib_id "FC01_Project:ANALOG_SENS__R_Small")
 		(at 100.33 76.2 0)
 		(unit 1)
@@
 			)
 		)
-		(property "Footprint Audit" "OK"
+		(property "Footprint Audit" "See verification/COMPONENTS.csv and verification/REPORT.md"
 			(at 102.87 74.9299 0)
 			(hide yes)
@@
 			)
 		)
-		(property "Library Audit" "KiCad standard"
+		(property "Library Audit" "See verification/COMPONENTS.csv and verification/REPORT.md"
 			(at 102.87 74.9299 0)
 			(hide yes)
@@
 	)
 	(symbol
-		(lib_id "power:GND")
+		(lib_id "FC01_Project:ANALOG_SENS__GND")
 		(at 123.19 81.28 0)
 		(unit 1)
@@
 	)
 	(symbol
-		(lib_id "Device:R_Small")
+		(lib_id "FC01_Project:ANALOG_SENS__R_Small")
 		(at 68.58 68.58 0)
 		(unit 1)
@@
 			)
 		)
-		(property "Footprint Audit" "OK"
+		(property "Footprint Audit" "See verification/COMPONENTS.csv and verification/REPORT.md"
 			(at 71.12 67.3099 0)
 			(hide yes)
@@
 			)
 		)
-		(property "Library Audit" "KiCad standard"
+		(property "Library Audit" "See verification/COMPONENTS.csv and verification/REPORT.md"
 			(at 71.12 67.3099 0)
 			(hide yes)
@@
 	)
 	(symbol
-		(lib_id "Device:C_Small")
+		(lib_id "FC01_Project:ANALOG_SENS__C_Small")
 		(at 123.19 76.2 0)
 		(unit 1)
@@
 			)
 		)
-		(property "Footprint Audit" "OK"
+		(property "Footprint Audit" "See verification/COMPONENTS.csv and verification/REPORT.md"
 			(at 125.73 74.9362 0)
 			(hide yes)
@@
 			)
 		)
-		(property "Library Audit" "KiCad standard"
+		(property "Library Audit" "See verification/COMPONENTS.csv and verification/REPORT.md"
 			(at 125.73 74.9362 0)
 			(hide yes)
@@
 	)
 	(symbol
-		(lib_id "power:GND")
+		(lib_id "FC01_Project:ANALOG_SENS__GND")
 		(at 107.95 53.34 0)
 		(unit 1)
@@
 	)
 	(symbol
-		(lib_id "Device:R_Small")
+		(lib_id "FC01_Project:ANALOG_SENS__R_Small")
 		(at 100.33 68.58 0)
 		(unit 1)
@@
 			)
 		)
-		(property "Footprint Audit" "OK"
+		(property "Footprint Audit" "See verification/COMPONENTS.csv and verification/REPORT.md"
 			(at 102.87 67.3099 0)
 			(hide yes)
@@
 			)
 		)
-		(property "Library Audit" "KiCad standard"
+		(property "Library Audit" "See verification/COMPONENTS.csv and verification/REPORT.md"
 			(at 102.87 67.3099 0)
 			(hide yes)
@@
 	)
 	(symbol
-		(lib_id "Device:C_Small")
+		(lib_id "FC01_Project:ANALOG_SENS__C_Small")
 		(at 91.44 76.2 0)
 		(unit 1)
@@
 			)
 		)
-		(property "Footprint Audit" "OK"
+		(property "Footprint Audit" "See verification/COMPONENTS.csv and verification/REPORT.md"
 			(at 93.98 74.9362 0)
 			(hide yes)
@@
 			)
 		)
-		(property "Library Audit" "KiCad standard"
+		(property "Library Audit" "See verification/COMPONENTS.csv and verification/REPORT.md"
 			(at 93.98 74.9362 0)
 			(hide yes)
@@
 	)
 	(symbol
-		(lib_id "Device:C_Small")
+		(lib_id "FC01_Project:ANALOG_SENS__C_Small")
 		(at 59.69 76.2 0)
 		(unit 1)
@@
 			)
 		)
-		(property "Footprint Audit" "OK"
+		(property "Footprint Audit" "See verification/COMPONENTS.csv and verification/REPORT.md"
 			(at 62.23 74.9362 0)
 			(hide yes)
@@
 			)
 		)
-		(property "Library Audit" "KiCad standard"
+		(property "Library Audit" "See verification/COMPONENTS.csv and verification/REPORT.md"
 			(at 62.23 74.9362 0)
 			(hide yes)
@@
 	)
 	(symbol
-		(lib_id "power:VAA")
+		(lib_id "FC01_Project:ANALOG_SENS__VAA")
 		(at 68.58 63.5 0)
 		(unit 1)
@@
 	)
 	(symbol
-		(lib_id "power:GND")
+		(lib_id "FC01_Project:ANALOG_SENS__GND")
 		(at 132.08 81.28 0)
 		(unit 1)
@@
 	)
 	(symbol
-		(lib_id "power:GND")
+		(lib_id "FC01_Project:ANALOG_SENS__GND")
 		(at 91.44 81.28 0)
 		(unit 1)
@@
 	)
 	(symbol
-		(lib_id "Device:R_Small")
+		(lib_id "FC01_Project:ANALOG_SENS__R_Small")
 		(at 68.58 76.2 0)
 		(unit 1)
@@
 			)
 		)
-		(property "Footprint Audit" "OK"
+		(property "Footprint Audit" "See verification/COMPONENTS.csv and verification/REPORT.md"
 			(at 71.12 74.9299 0)
 			(hide yes)
@@
 			)
 		)
-		(property "Library Audit" "KiCad standard"
+		(property "Library Audit" "See verification/COMPONENTS.csv and verification/REPORT.md"
 			(at 71.12 74.9299 0)
 			(hide yes)
@@
 	)
 	(symbol
-		(lib_id "Device:R_Small")
+		(lib_id "FC01_Project:ANALOG_SENS__R_Small")
 		(at 132.08 76.2 0)
 		(unit 1)
@@
 			)
 		)
-		(property "Footprint Audit" "OK"
+		(property "Footprint Audit" "See verification/COMPONENTS.csv and verification/REPORT.md"
 			(at 134.62 74.9299 0)
 			(hide yes)
@@
 			)
 		)
-		(property "Library Audit" "KiCad standard"
+		(property "Library Audit" "See verification/COMPONENTS.csv and verification/REPORT.md"
 			(at 134.62 74.9299 0)
 			(hide yes)
@@
 	)
 	(symbol
-		(lib_id "power:GND")
+		(lib_id "FC01_Project:ANALOG_SENS__GND")
 		(at 100.33 81.28 0)
 		(unit 1)
@@
 	)
 	(symbol
-		(lib_id "power:GND")
+		(lib_id "FC01_Project:ANALOG_SENS__GND")
 		(at 68.58 81.28 0)
 		(unit 1)
@@
 	)
 	(symbol
-		(lib_id "power:GND")
+		(lib_id "FC01_Project:ANALOG_SENS__GND")
 		(at 59.69 81.28 0)
 		(unit 1)
@@
 	)
 	(symbol
-		(lib_id "Device:R_Small")
+		(lib_id "FC01_Project:ANALOG_SENS__R_Small")
 		(at 132.08 68.58 0)
 		(unit 1)
@@
 			)
 		)
-		(property "Footprint Audit" "OK"
+		(property "Footprint Audit" "See verification/COMPONENTS.csv and verification/REPORT.md"
 			(at 134.62 67.3099 0)
 			(hide yes)
@@
 			)
 		)
-		(property "Library Audit" "KiCad standard"
+		(property "Library Audit" "See verification/COMPONENTS.csv and verification/REPORT.md"
 			(at 134.62 67.3099 0)
 			(hide yes)
@@
 	)
 	(symbol
-		(lib_id "power:GND")
+		(lib_id "FC01_Project:ANALOG_SENS__GND")
 		(at 110.49 53.34 0)
 		(unit 1)
@@
 	)
 	(symbol
-		(lib_id "Connector_Generic:Conn_01x04")
+		(lib_id "FC01_Project:ANALOG_SENS__Conn_01x04")
 		(at 107.95 45.72 90)
 		(unit 1)
@@
 			)
 		)
-		(property "Footprint Audit" "OK: 4 square SMD pads 1.00x1.00 mm, P2.54 mm, no holes, no paste"
+		(property "Footprint Audit" "See verification/COMPONENTS.csv and verification/REPORT.md"
 			(at 109.22 39.37 90)
 			(hide yes)
@@
 			)
 		)
-		(property "Library Audit" "Project-local H743_Custom footprint"
+		(property "Library Audit" "See verification/COMPONENTS.csv and verification/REPORT.md"
 			(at 109.22 39.37 90)
 			(hide yes)
