File: ANALOG_SENS.kicad_sch (KiCad schematic)
At the start: 10 parts, among them J1 Conn_01x04

Commit message: update pcb
Parts:
- J1: value Conn_01x04 -> Analog
Changed lines of the file:
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@@
 			)
 		)
-		(property "Value" "Conn_01x04"
+		(property "Value" "Analog"
 			(at 109.22 41.91 90)
 			(show_name no)

Commit message: ok
Connections:
- net ADC_VBAT1: no longer C35.1, R18.2, R19.1
- net ADC_VBAT2: now also C35.1, R18.2, R19.1
Changed lines of the file:
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@@
 		)
 	)
-	(label "ADC_VBAT1"
+	(label "ADC_VBAT2"
 		(at 110.49 72.39 0)
 		(effects
