File: MICRO_SD.kicad_sch (KiCad schematic)
At the start: 9 parts, among them J1 TF-028-H265

Commit message: update name
Other:
- note removed: "MICRO SD"
- company: Pierluigi Colangeli, PhD -> (none)
- title: LEVIA H7 -> (none)

Commit message: upsadte SPI4 set to Baro
Other:
- title: (none) -> H743_ARDUPILOT
Changed lines of the file:
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@@
 	(generator "eeschema")
 	(generator_version "10.0")
-	(paper "A5")
+	(paper "A3")
 	(title_block
+		(title "H743_ARDUPILOT")
 		(date "2026-09-24")
 	)

Commit message: re annotate componant globaly
Parts:
- renumbered C53 to C40, C54 to C41, J1 to J10, R36 to R35, R37 to R36, R38 to R37, R39 to R38, R40 to R39, R41 to R40
Changed lines of the file:
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@@
 		(in_pos_files yes)
 		(dnp no)
-		(property "Reference" "R40"
+		(property "Reference" "R39"
 			(at 151.13 62.23 90)
 			(show_name no)
@@
 			(project "H743_Ardupilot"
 				(path "/6b768b36-fce6-4be0-9021-6d41bddc3a70/f6fdd950-a71d-4aac-93a8-c5aad57c018b"
-					(reference "R40")
+					(reference "R39")
 					(unit 1)
 				)
@@
 		(in_pos_files yes)
 		(dnp no)
-		(property "Reference" "R39"
+		(property "Reference" "R38"
 			(at 151.13 59.69 90)
 			(show_name no)
@@
 			(project "H743_Ardupilot"
 				(path "/6b768b36-fce6-4be0-9021-6d41bddc3a70/f6fdd950-a71d-4aac-93a8-c5aad57c018b"
-					(reference "R39")
+					(reference "R38")
 					(unit 1)
 				)
@@
 		(in_pos_files yes)
 		(dnp no)
-		(property "Reference" "R36"
+		(property "Reference" "R35"
 			(at 151.13 52.07 90)
 			(show_name no)
@@
 			(project "H743_Ardupilot"
 				(path "/6b768b36-fce6-4be0-9021-6d41bddc3a70/f6fdd950-a71d-4aac-93a8-c5aad57c018b"
-					(reference "R36")
+					(reference "R35")
 					(unit 1)
 				)
@@
 		(dnp no)
 		(fields_autoplaced yes)
-		(property "Reference" "#PWR0116"
+		(property "Reference" "#PWR091"
 			(at 53.34 73.66 0)
 			(hide yes)
@@
 			(project "H743_Ardupilot"
 				(path "/6b768b36-fce6-4be0-9021-6d41bddc3a70/f6fdd950-a71d-4aac-93a8-c5aad57c018b"
-					(reference "#PWR0116")
+					(reference "#PWR091")
 					(unit 1)
 				)
@@
 		(in_pos_files yes)
 		(dnp no)
-		(property "Reference" "R38"
+		(property "Reference" "R37"
 			(at 151.13 57.15 90)
 			(show_name no)
@@
 			(project "H743_Ardupilot"
 				(path "/6b768b36-fce6-4be0-9021-6d41bddc3a70/f6fdd950-a71d-4aac-93a8-c5aad57c018b"
-					(reference "R38")
+					(reference "R37")
 					(unit 1)
 				)
@@
 		(in_pos_files yes)
 		(dnp no)
-		(property "Reference" "R37"
+		(property "Reference" "R36"
 			(at 151.13 54.61 90)
 			(show_name no)
@@
 			(project "H743_Ardupilot"
 				(path "/6b768b36-fce6-4be0-9021-6d41bddc3a70/f6fdd950-a71d-4aac-93a8-c5aad57c018b"
-					(reference "R37")
+					(reference "R36")
 					(unit 1)
 				)
@@
 		(in_pos_files yes)
 		(dnp no)
-		(property "Reference" "C54"
+		(property "Reference" "C41"
 			(at 60.96 59.69 0)
 			(show_name no)
@@
 			(project "H743_Ardupilot"
 				(path "/6b768b36-fce6-4be0-9021-6d41bddc3a70/f6fdd950-a71d-4aac-93a8-c5aad57c018b"
-					(reference "C54")
+					(reference "C41")
 					(unit 1)
 				)
@@
 		(in_pos_files yes)
 		(dnp no)
-		(property "Reference" "J1"
+		(property "Reference" "J10"
 			(at 105.41 39.37 0)
 			(show_name no)
@@
 			(project "H743_Ardupilot"
 				(path "/6b768b36-fce6-4be0-9021-6d41bddc3a70/f6fdd950-a71d-4aac-93a8-c5aad57c018b"
-					(reference "J1")
+					(reference "J10")
 					(unit 1)
 				)
@@
 		(in_pos_files yes)
 		(dnp no)
-		(property "Reference" "C53"
+		(property "Reference" "C40"
 			(at 54.61 59.69 0)
 			(show_name no)
@@
 			(project "H743_Ardupilot"
 				(path "/6b768b36-fce6-4be0-9021-6d41bddc3a70/f6fdd950-a71d-4aac-93a8-c5aad57c018b"
-					(reference "C53")
+					(reference "C40")
 					(unit 1)
 				)
@@
 		(in_pos_files yes)
 		(dnp no)
-		(property "Reference" "R41"
+		(property "Reference" "R40"
 			(at 151.13 64.77 90)
 			(show_name no)
@@
 			(project "H743_Ardupilot"
 				(path "/6b768b36-fce6-4be0-9021-6d41bddc3a70/f6fdd950-a71d-4aac-93a8-c5aad57c018b"
-					(reference "R41")
+					(reference "R40")
 					(unit 1)
 				)
@@
 		(dnp no)
 		(fields_autoplaced yes)
-		(property "Reference" "#PWR0115"
+		(property "Reference" "#PWR090"
 			(at 53.34 60.96 0)
 			(hide yes)
@@
 			(project "H743_Ardupilot"
 				(path "/6b768b36-fce6-4be0-9021-6d41bddc3a70/f6fdd950-a71d-4aac-93a8-c5aad57c018b"
-					(reference "#PWR0115")
+					(reference "#PWR090")
 					(unit 1)
 				)
@@
 		(dnp no)
 		(fields_autoplaced yes)
-		(property "Reference" "#PWR0117"
+		(property "Reference" "#PWR092"
 			(at 83.82 88.9 0)
 			(hide yes)
@@
 			(project "H743_Ardupilot"
 				(path "/6b768b36-fce6-4be0-9021-6d41bddc3a70/f6fdd950-a71d-4aac-93a8-c5aad57c018b"
-					(reference "#PWR0117")
+					(reference "#PWR092")
 					(unit 1)
 				)

Commit message: audit DigiKey metadata: MICRO_SD.kicad_sch
Parts:
- C40: DigiKey Part Number (none) -> 1276-1445-1-ND; DigiKey Price Qty (none) -> 1 CT; DigiKey Specs (none) -> 1 µF ±10%, 25 V, X5R, 0402; DigiKey Status (none) -> Active; DigiKey URL (none) -> https://www.digikey.fr/en/products/result?keywords=CL05A105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; DigiKey Unit Price EUR (none) -> 0.16; Footprint Audit (none) -> OK; LCSC C52923 -> (none); LCSC Part C52923 -> (none); Library Audit (none) -> KiCad standard; Package (none) -> 0402 (1005); Price Checked (none) -> 2026-09-25
- C41: DigiKey Part Number (none) -> 1276-1001-1-ND; DigiKey Price Qty (none) -> 1 CT; DigiKey Specs (none) -> 100 nF ±10%, 16 V, X7R, 0402; DigiKey Status (none) -> Active; DigiKey URL (none) -> https://www.digikey.fr/fr/products/detail/samsung-electro-m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; DigiKey Unit Price EUR (none) -> 0.09; Footprint Audit (none) -> OK; LCSC C1525 -> (none); LCSC Part C1525 -> (none); Library Audit (none) -> KiCad standard; MPN GRM022R60J104KE15D -> CL05B104KO5NNNC; Manufacturer Murata Electronics -> Samsung Electro-Mechanics; Package (none) -> 0402 (1005); Price Checked (none) -> 2026-09-25
- J10: DigiKey Specs (none) -> MicroSD push-pull socket, SMD, body height 2.65 mm, -20°C t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; DigiKey Status (none) -> No exact DigiKey listing found; supplier/LCSC part retained; Footprint Audit (none) -> CHECK EasyEDA footprint vs HANBO drawing before release; Library Audit (none) -> EasyEDA external; Manufacturer HANBO(汉博) -> HANBO; Package (none) -> MicroSD socket SMD H=2.65 mm; Price Checked (none) -> 2026-09-25
- R35, R36, R37, R38, R39, R40: DigiKey Price Qty (none) -> 1 CT; DigiKey Specs (none) -> 10K ±1%, 0402 (1005), thick film; DigiKey Status (none) -> Active / DigiKey family verified; DigiKey URL (none) -> https://www.digikey.fr/en/products/result?keywords=RC0402FR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; DigiKey Unit Price EUR (none) -> 0.09; Footprint Audit (none) -> OK; LCSC C25744 -> (none); LCSC Part C25744 -> (none); Library Audit (none) -> KiCad standard; MPN 0402WGF1002TCE -> RC0402FR-0710KL; Manufacturer UNI-ROYAL(Uniroyal Elec) -> YAGEO; Package (none) -> 0402 (1005 Metric); Price Checked (none) -> 2026-09-25

Commit message: update
Parts:
- renumbered C40 to C57, C41 to C58, J10 to J11, R35 to R41, R36 to R42, R37 to R43, R38 to R44, R39 to R45, R40 to R46
Changed lines of the file:
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@@
 		(in_pos_files yes)
 		(dnp no)
-		(property "Reference" "R39"
+		(property "Reference" "R45"
 			(at 151.13 62.23 90)
 			(show_name no)
@@
 			(project "H743_Ardupilot"
 				(path "/6b768b36-fce6-4be0-9021-6d41bddc3a70/f6fdd950-a71d-4aac-93a8-c5aad57c018b"
-					(reference "R39")
+					(reference "R45")
 					(unit 1)
 				)
@@
 		(in_pos_files yes)
 		(dnp no)
-		(property "Reference" "R38"
+		(property "Reference" "R44"
 			(at 151.13 59.69 90)
 			(show_name no)
@@
 			(project "H743_Ardupilot"
 				(path "/6b768b36-fce6-4be0-9021-6d41bddc3a70/f6fdd950-a71d-4aac-93a8-c5aad57c018b"
-					(reference "R38")
+					(reference "R44")
 					(unit 1)
 				)
@@
 		(in_pos_files yes)
 		(dnp no)
-		(property "Reference" "R35"
+		(property "Reference" "R41"
 			(at 151.13 52.07 90)
 			(show_name no)
@@
 			(project "H743_Ardupilot"
 				(path "/6b768b36-fce6-4be0-9021-6d41bddc3a70/f6fdd950-a71d-4aac-93a8-c5aad57c018b"
-					(reference "R35")
+					(reference "R41")
 					(unit 1)
 				)
@@
 		(dnp no)
 		(fields_autoplaced yes)
-		(property "Reference" "#PWR091"
+		(property "Reference" "#PWR0120"
 			(at 53.34 73.66 0)
 			(hide yes)
@@
 			(project "H743_Ardupilot"
 				(path "/6b768b36-fce6-4be0-9021-6d41bddc3a70/f6fdd950-a71d-4aac-93a8-c5aad57c018b"
-					(reference "#PWR091")
+					(reference "#PWR0120")
 					(unit 1)
 				)
@@
 		(in_pos_files yes)
 		(dnp no)
-		(property "Reference" "R37"
+		(property "Reference" "R43"
 			(at 151.13 57.15 90)
 			(show_name no)
@@
 			(project "H743_Ardupilot"
 				(path "/6b768b36-fce6-4be0-9021-6d41bddc3a70/f6fdd950-a71d-4aac-93a8-c5aad57c018b"
-					(reference "R37")
+					(reference "R43")
 					(unit 1)
 				)
@@
 		(in_pos_files yes)
 		(dnp no)
-		(property "Reference" "R36"
+		(property "Reference" "R42"
 			(at 151.13 54.61 90)
 			(show_name no)
@@
 			(project "H743_Ardupilot"
 				(path "/6b768b36-fce6-4be0-9021-6d41bddc3a70/f6fdd950-a71d-4aac-93a8-c5aad57c018b"
-					(reference "R36")
+					(reference "R42")
 					(unit 1)
 				)
@@
 		(in_pos_files yes)
 		(dnp no)
-		(property "Reference" "C41"
+		(property "Reference" "C58"
 			(at 60.96 59.69 0)
 			(show_name no)
@@
 			(project "H743_Ardupilot"
 				(path "/6b768b36-fce6-4be0-9021-6d41bddc3a70/f6fdd950-a71d-4aac-93a8-c5aad57c018b"
-					(reference "C41")
+					(reference "C58")
 					(unit 1)
 				)
@@
 		(in_pos_files yes)
 		(dnp no)
-		(property "Reference" "J10"
+		(property "Reference" "J11"
 			(at 105.41 39.37 0)
 			(show_name no)
@@
 			(project "H743_Ardupilot"
 				(path "/6b768b36-fce6-4be0-9021-6d41bddc3a70/f6fdd950-a71d-4aac-93a8-c5aad57c018b"
-					(reference "J10")
+					(reference "J11")
 					(unit 1)
 				)
@@
 		(in_pos_files yes)
 		(dnp no)
-		(property "Reference" "C40"
+		(property "Reference" "C57"
 			(at 54.61 59.69 0)
 			(show_name no)
@@
 			(project "H743_Ardupilot"
 				(path "/6b768b36-fce6-4be0-9021-6d41bddc3a70/f6fdd950-a71d-4aac-93a8-c5aad57c018b"
-					(reference "C40")
+					(reference "C57")
 					(unit 1)
 				)
@@
 		(in_pos_files yes)
 		(dnp no)
-		(property "Reference" "R40"
+		(property "Reference" "R46"
 			(at 151.13 64.77 90)
 			(show_name no)
@@
 			(project "H743_Ardupilot"
 				(path "/6b768b36-fce6-4be0-9021-6d41bddc3a70/f6fdd950-a71d-4aac-93a8-c5aad57c018b"
-					(reference "R40")
+					(reference "R46")
 					(unit 1)
 				)
@@
 		(dnp no)
 		(fields_autoplaced yes)
-		(property "Reference" "#PWR090"
+		(property "Reference" "#PWR0119"
 			(at 53.34 60.96 0)
 			(hide yes)
@@
 			(project "H743_Ardupilot"
 				(path "/6b768b36-fce6-4be0-9021-6d41bddc3a70/f6fdd950-a71d-4aac-93a8-c5aad57c018b"
-					(reference "#PWR090")
+					(reference "#PWR0119")
 					(unit 1)
 				)
@@
 		(dnp no)
 		(fields_autoplaced yes)
-		(property "Reference" "#PWR092"
+		(property "Reference" "#PWR0121"
 			(at 83.82 88.9 0)
 			(hide yes)
@@
 			(project "H743_Ardupilot"
 				(path "/6b768b36-fce6-4be0-9021-6d41bddc3a70/f6fdd950-a71d-4aac-93a8-c5aad57c018b"
-					(reference "#PWR092")
+					(reference "#PWR0121")
 					(unit 1)
 				)

Commit message: Adopt active Amphenol 10067099-200LF microSD connector
Parts:
- J11: value TF-028-H265 -> 10067099-200LF; DigiKey Status No exact DigiKey listing found; supplier/LCSC part retained -> Active; DigiKey 609-5773-1-ND (CT), 609-5773-2-ND (TR), 609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; Footprint Audit CHECK EasyEDA footprint vs HANBO drawing before release -> BLOCKING: replace/verify current legacy footprint against e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; MPN TF-028-H265 -> 10067099-200LF; Manufacturer HANBO -> Amphenol ICC (FCI); Package MicroSD socket SMD H=2.65 mm -> microSD, SMD right-angle top-mount, 10 positions (8+2), H=2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
Changed lines of the file:
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@@
 			)
 		)
-		(property "Value" "TF-028-H265"
+		(property "Value" "10067099-200LF"
 			(at 100.33 41.91 0)
 			(show_name no)
@@
 			)
 		)
-		(property "Datasheet" "https://item.szlcsc.com/6065985.html"
+		(property "Datasheet" "https://www.amphenol-cs.com/product/10067099200lf.html"
 			(at 109.22 58.42 0)
 			(hide yes)
@@
 			)
 		)
-		(property "Manufacturer" "HANBO"
+		(property "Manufacturer" "Amphenol ICC (FCI)"
 			(at 109.22 85.09 0)
 			(hide yes)
@@
 			)
 		)
-		(property "MPN" "TF-028-H265"
+		(property "MPN" "10067099-200LF"
 			(at 109.22 87.63 0)
 			(hide yes)
@@
 			)
 		)
-		(property "DigiKey Status" "No exact DigiKey listing found; supplier/LCSC part retained"
+		(property "DigiKey Status" "Active; DigiKey 609-5773-1-ND (CT), 609-5773-2-ND (TR), 609-5773-6-ND (Digi-Reel)"
 			(at 105.41 39.37 0)
 			(hide yes)
@@
 			)
 		)
-		(property "Package" "MicroSD socket SMD H=2.65 mm"
+		(property "Package" "microSD, SMD right-angle top-mount, 10 positions (8+2), H=2.65 mm"
 			(at 105.41 39.37 0)
 			(hide yes)
@@
 			)
 		)
-		(property "Footprint Audit" "CHECK EasyEDA footprint vs HANBO drawing before release"
+		(property "Footprint Audit" "BLOCKING: replace/verify current legacy footprint against exact Amphenol 10067099-200LF land pattern before PCB release"
 			(at 105.41 39.37 0)
 			(hide yes)

Commit message: Use project-local Amphenol 10067099-200LF footprint and metadata
Parts:
- J11: footprint EasyEDA:TF-SMD_TF-021B-H265 -> H743_Custom:Amphenol_10067099-200LF; DigiKey Price Qty (none) -> 1 CT; DigiKey Specs MicroSD push-pull socket, SMD, body height 2.65 mm, -20°C t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 -> 10 (8+2) positions; microSD; push-in/pull-out; right-angle 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; DigiKey URL (none) -> https://www.digikey.fr/fr/products/detail/amphenol-icc-fci/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; DigiKey Unit Price EUR (none) -> 0.78; Footprint Audit BLOCKING: replace/verify current legacy footprint against e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 -> OK: project-local footprint derived from Amphenol drawing 1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; LCSC C5310496 -> C5408015; LCSC Part C5310496 -> C5408015; Library Audit EasyEDA external -> H743_Custom project-local; Amphenol drawing Rev H
- R45: Price Checked 2026-09-25 -> 2026-09-26
Changed lines of the file:
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@@
 			)
 		)
-		(property "Price Checked" "2026-09-25"
+		(property "Price Checked" "2026-09-26"
 			(at 151.13 62.23 90)
 			(hide yes)
@@
 			)
 		)
-		(property "Footprint" "EasyEDA:TF-SMD_TF-021B-H265"
+		(property "Footprint" "H743_Custom:Amphenol_10067099-200LF"
 			(at 138.43 50.8 0)
 			(hide yes)
@@
 			)
 		)
-		(property "LCSC Part" "C5310496"
+		(property "LCSC Part" "C5408015"
 			(at 109.22 90.17 0)
 			(hide yes)
@@
 			)
 		)
-		(property "LCSC" "C5310496"
+		(property "LCSC" "C5408015"
 			(at 109.22 58.42 0)
 			(hide yes)
@@
 			)
 		)
-		(property "DigiKey URL" ""
+		(property "DigiKey URL" "https://www.digikey.fr/fr/products/detail/amphenol-icc-fci/10067099-200LF/4238739"
 			(at 105.41 39.37 0)
 			(hide yes)
@@
 			)
 		)
-		(property "DigiKey Specs" "MicroSD push-pull socket, SMD, body height 2.65 mm, -20°C to +85°C"
+		(property "DigiKey Specs" "10 (8+2) positions; microSD; push-in/pull-out; right-angle SMD; H=2.65 mm; Au contacts; 1.10 mm pitch"
 			(at 105.41 39.37 0)
 			(hide yes)
@@
 			)
 		)
-		(property "DigiKey Unit Price EUR" ""
+		(property "DigiKey Unit Price EUR" "0.78"
 			(at 105.41 39.37 0)
 			(hide yes)
@@
 			)
 		)
-		(property "DigiKey Price Qty" ""
+		(property "DigiKey Price Qty" "1 CT"
 			(at 105.41 39.37 0)
 			(hide yes)
@@
 			)
 		)
-		(property "Footprint Audit" "BLOCKING: replace/verify current legacy footprint against exact Amphenol 10067099-200LF land pattern before PCB release"
+		(property "Footprint Audit" "OK: project-local footprint derived from Amphenol drawing 10067099 Rev H; verify final PCB orientation against STEP before fabrication"
 			(at 105.41 39.37 0)
 			(hide yes)
@@
 			)
 		)
-		(property "Library Audit" "EasyEDA external"
+		(property "Library Audit" "H743_Custom project-local; Amphenol drawing Rev H"
 			(at 105.41 39.37 0)
 			(hide yes)
