File: MICRO_SD.kicad_sch (KiCad schematic)
At the start: 9 parts, among them J11 10067099-200LF

Commit message: Mark microSD footprint for final dimensional cross-check
Parts:
- J11: Footprint Audit OK: project-local footprint derived from Amphenol drawing 1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 -> CHECK FINAL: project-local footprint derived from Amphenol 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
Changed lines of the file:
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@@
 			)
 		)
-		(property "Footprint Audit" "OK: project-local footprint derived from Amphenol drawing 10067099 Rev H; verify final PCB orientation against STEP before fabrication"
+		(property "Footprint Audit" "CHECK FINAL: project-local footprint derived from Amphenol drawing 10067099 Rev H; pad geometry/orientation must be dimensionally cross-checked against drawing + STEP before PCB fabrication"
 			(at 105.41 39.37 0)
 			(hide yes)

Commit message: Validate 10067099-200LF land pattern dimensions
Parts:
- J11: Footprint Audit CHECK FINAL: project-local footprint derived from Amphenol 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 -> OK DIMENSIONAL: footprint cross-checked against Amphenol dr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
Changed lines of the file:
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@@
 			)
 		)
-		(property "Footprint Audit" "CHECK FINAL: project-local footprint derived from Amphenol drawing 10067099 Rev H; pad geometry/orientation must be dimensionally cross-checked against drawing + STEP before PCB fabrication"
+		(property "Footprint Audit" "OK DIMENSIONAL: footprint cross-checked against Amphenol drawing 10067099 Rev H and official STEP; verify only final board-side orientation/3D placement before fabrication"
 			(at 105.41 39.37 0)
 			(hide yes)

Commit message: Mark 10067099-200LF footprint invalid pending redraw
Parts:
- J11: Footprint Audit OK DIMENSIONAL: footprint cross-checked against Amphenol dr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 -> BLOCKING - DO NOT USE: custom footprint contains dimensiona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
Changed lines of the file:
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@@
 			)
 		)
-		(property "Footprint Audit" "OK DIMENSIONAL: footprint cross-checked against Amphenol drawing 10067099 Rev H and official STEP; verify only final board-side orientation/3D placement before fabrication"
+		(property "Footprint Audit" "BLOCKING - DO NOT USE: custom footprint contains dimensional interpretation errors versus Amphenol drawing 10067099 Rev H; must be rebuilt from recommended PCB layout"
 			(at 105.41 39.37 0)
 			(hide yes)

Commit message: Switch microSD to rebuilt Amphenol RevH footprint
Parts:
- J11: footprint H743_Custom:Amphenol_10067099-200LF -> H743_Custom:Amphenol_10067099-200LF_RevH; Footprint Audit BLOCKING - DO NOT USE: custom footprint contains dimensiona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 -> CHECK FINAL: new RevH footprint rebuilt from manufacturer r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
Changed lines of the file:
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@@
 			)
 		)
-		(property "Footprint" "H743_Custom:Amphenol_10067099-200LF"
+		(property "Footprint" "H743_Custom:Amphenol_10067099-200LF_RevH"
 			(at 138.43 50.8 0)
 			(hide yes)
@@
 			)
 		)
-		(property "Footprint Audit" "BLOCKING - DO NOT USE: custom footprint contains dimensional interpretation errors versus Amphenol drawing 10067099 Rev H; must be rebuilt from recommended PCB layout"
+		(property "Footprint Audit" "CHECK FINAL: new RevH footprint rebuilt from manufacturer recommended PCB layout; verify orientation and pad mapping in PCB editor before fabrication"
 			(at 105.41 39.37 0)
 			(hide yes)

Commit message: Update microSD footprint audit after RevH correction
Parts:
- J11: Footprint Audit CHECK FINAL: new RevH footprint rebuilt from manufacturer r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 -> LAND PATTERN VERIFIED: pad geometry checked against Ampheno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
Changed lines of the file:
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@@
 			)
 		)
-		(property "Footprint Audit" "CHECK FINAL: new RevH footprint rebuilt from manufacturer recommended PCB layout; verify orientation and pad mapping in PCB editor before fabrication"
+		(property "Footprint Audit" "LAND PATTERN VERIFIED: pad geometry checked against Amphenol 10067099 Rev H recommended PCB layout; only final board orientation remains to verify"
 			(at 105.41 39.37 0)
 			(hide yes)

Commit message: update cmp number
Parts:
- renumbered J11 to J12
Changed lines of the file:
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@@
 		(dnp no)
 		(fields_autoplaced yes)
-		(property "Reference" "#PWR0120"
+		(property "Reference" "#PWR0122"
 			(at 53.34 73.66 0)
 			(hide yes)
@@
 			(project "H743_Ardupilot"
 				(path "/6b768b36-fce6-4be0-9021-6d41bddc3a70/f6fdd950-a71d-4aac-93a8-c5aad57c018b"
-					(reference "#PWR0120")
+					(reference "#PWR0122")
 					(unit 1)
 				)
@@
 		(in_pos_files yes)
 		(dnp no)
-		(property "Reference" "J11"
+		(property "Reference" "J12"
 			(at 105.41 39.37 0)
 			(show_name no)
@@
 			(project "H743_Ardupilot"
 				(path "/6b768b36-fce6-4be0-9021-6d41bddc3a70/f6fdd950-a71d-4aac-93a8-c5aad57c018b"
-					(reference "J11")
+					(reference "J12")
 					(unit 1)
 				)
@@
 		(dnp no)
 		(fields_autoplaced yes)
-		(property "Reference" "#PWR0119"
+		(property "Reference" "#PWR0121"
 			(at 53.34 60.96 0)
 			(hide yes)
@@
 			(project "H743_Ardupilot"
 				(path "/6b768b36-fce6-4be0-9021-6d41bddc3a70/f6fdd950-a71d-4aac-93a8-c5aad57c018b"
-					(reference "#PWR0119")
+					(reference "#PWR0121")
 					(unit 1)
 				)
@@
 		(dnp no)
 		(fields_autoplaced yes)
-		(property "Reference" "#PWR0121"
+		(property "Reference" "#PWR0123"
 			(at 83.82 88.9 0)
 			(hide yes)
@@
 			(project "H743_Ardupilot"
 				(path "/6b768b36-fce6-4be0-9021-6d41bddc3a70/f6fdd950-a71d-4aac-93a8-c5aad57c018b"
-					(reference "#PWR0121")
+					(reference "#PWR0123")
 					(unit 1)
 				)

Commit message: Review component footprints, restore local libraries and reconcile PCB pads
Parts:
- C57, C58: symbol Device:C_Small -> FC01_Project:MICRO_SD__C_Small; Footprint Audit OK -> See verification/COMPONENTS.csv and verification/REPORT.md; Library Audit KiCad standard -> See verification/COMPONENTS.csv and verification/REPORT.md
- J12: symbol EasyEDA:Micro_SD_Card -> FC01_Project:MICRO_SD__Micro_SD_Card; Footprint Audit LAND PATTERN VERIFIED: pad geometry checked against Ampheno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 -> See verification/COMPONENTS.csv and verification/REPORT.md; Library Audit H743_Custom project-local; Amphenol drawing Rev H -> See verification/COMPONENTS.csv and verification/REPORT.md
- R41, R42, R43, R44, R45, R46: symbol Device:R_Small -> FC01_Project:MICRO_SD__R_Small; Footprint Audit OK -> See verification/COMPONENTS.csv and verification/REPORT.md; Library Audit KiCad standard -> See verification/COMPONENTS.csv and verification/REPORT.md
Changed lines of the file:
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@@
 	)
 	(symbol
-		(lib_id "Device:R_Small")
+		(lib_id "FC01_Project:MICRO_SD__R_Small")
 		(at 154.94 63.5 90)
 		(unit 1)
@@
 			)
 		)
-		(property "Footprint Audit" "OK"
+		(property "Footprint Audit" "See verification/COMPONENTS.csv and verification/REPORT.md"
 			(at 151.13 62.23 90)
 			(hide yes)
@@
 			)
 		)
-		(property "Library Audit" "KiCad standard"
+		(property "Library Audit" "See verification/COMPONENTS.csv and verification/REPORT.md"
 			(at 151.13 62.23 90)
 			(hide yes)
@@
 	)
 	(symbol
-		(lib_id "Device:R_Small")
+		(lib_id "FC01_Project:MICRO_SD__R_Small")
 		(at 154.94 60.96 90)
 		(unit 1)
@@
 			)
 		)
-		(property "Footprint Audit" "OK"
+		(property "Footprint Audit" "See verification/COMPONENTS.csv and verification/REPORT.md"
 			(at 151.13 59.69 90)
 			(hide yes)
@@
 			)
 		)
-		(property "Library Audit" "KiCad standard"
+		(property "Library Audit" "See verification/COMPONENTS.csv and verification/REPORT.md"
 			(at 151.13 59.69 90)
 			(hide yes)
@@
 	)
 	(symbol
-		(lib_id "Device:R_Small")
+		(lib_id "FC01_Project:MICRO_SD__R_Small")
 		(at 154.94 53.34 90)
 		(unit 1)
@@
 			)
 		)
-		(property "Footprint Audit" "OK"
+		(property "Footprint Audit" "See verification/COMPONENTS.csv and verification/REPORT.md"
 			(at 151.13 52.07 90)
 			(hide yes)
@@
 			)
 		)
-		(property "Library Audit" "KiCad standard"
+		(property "Library Audit" "See verification/COMPONENTS.csv and verification/REPORT.md"
 			(at 151.13 52.07 90)
 			(hide yes)
@@
 	)
 	(symbol
-		(lib_id "power:GND")
+		(lib_id "FC01_Project:MICRO_SD__GND")
 		(at 53.34 67.31 0)
 		(unit 1)
@@
 	)
 	(symbol
-		(lib_id "Device:R_Small")
+		(lib_id "FC01_Project:MICRO_SD__R_Small")
 		(at 154.94 58.42 90)
 		(unit 1)
@@
 			)
 		)
-		(property "Footprint Audit" "OK"
+		(property "Footprint Audit" "See verification/COMPONENTS.csv and verification/REPORT.md"
 			(at 151.13 57.15 90)
 			(hide yes)
@@
 			)
 		)
-		(property "Library Audit" "KiCad standard"
+		(property "Library Audit" "See verification/COMPONENTS.csv and verification/REPORT.md"
 			(at 151.13 57.15 90)
 			(hide yes)
@@
 	)
 	(symbol
-		(lib_id "Device:R_Small")
+		(lib_id "FC01_Project:MICRO_SD__R_Small")
 		(at 154.94 55.88 90)
 		(unit 1)
@@
 			)
 		)
-		(property "Footprint Audit" "OK"
+		(property "Footprint Audit" "See verification/COMPONENTS.csv and verification/REPORT.md"
 			(at 151.13 54.61 90)
 			(hide yes)
@@
 			)
 		)
-		(property "Library Audit" "KiCad standard"
+		(property "Library Audit" "See verification/COMPONENTS.csv and verification/REPORT.md"
 			(at 151.13 54.61 90)
 			(hide yes)
@@
 	)
 	(symbol
-		(lib_id "Device:C_Small")
+		(lib_id "FC01_Project:MICRO_SD__C_Small")
 		(at 59.69 62.23 0)
 		(unit 1)
@@
 			)
 		)
-		(property "Footprint Audit" "OK"
+		(property "Footprint Audit" "See verification/COMPONENTS.csv and verification/REPORT.md"
 			(at 60.96 59.69 0)
 			(hide yes)
@@
 			)
 		)
-		(property "Library Audit" "KiCad standard"
+		(property "Library Audit" "See verification/COMPONENTS.csv and verification/REPORT.md"
 			(at 60.96 59.69 0)
 			(hide yes)
@@
 	)
 	(symbol
-		(lib_id "EasyEDA:Micro_SD_Card")
+		(lib_id "FC01_Project:MICRO_SD__Micro_SD_Card")
 		(at 109.22 58.42 0)
 		(unit 1)
@@
 			)
 		)
-		(property "Datasheet" "https://www.amphenol-cs.com/product/10067099200lf.html"
+		(property "Datasheet" "https://cdn.amphenol-cs.com/media/wysiwyg/files/drawing/10067099.pdf"
 			(at 109.22 58.42 0)
 			(hide yes)
@@
 			)
 		)
-		(property "Footprint Audit" "LAND PATTERN VERIFIED: pad geometry checked against Amphenol 10067099 Rev H recommended PCB layout; only final board orientation remains to verify"
+		(property "Footprint Audit" "See verification/COMPONENTS.csv and verification/REPORT.md"
 			(at 105.41 39.37 0)
 			(hide yes)
@@
 			)
 		)
-		(property "Library Audit" "H743_Custom project-local; Amphenol drawing Rev H"
+		(property "Library Audit" "See verification/COMPONENTS.csv and verification/REPORT.md"
 			(at 105.41 39.37 0)
 			(hide yes)
@@
 	)
 	(symbol
-		(lib_id "Device:C_Small")
+		(lib_id "FC01_Project:MICRO_SD__C_Small")
 		(at 53.34 62.23 0)
 		(unit 1)
@@
 			)
 		)
-		(property "Footprint Audit" "OK"
+		(property "Footprint Audit" "See verification/COMPONENTS.csv and verification/REPORT.md"
 			(at 54.61 59.69 0)
 			(hide yes)
@@
 			)
 		)
-		(property "Library Audit" "KiCad standard"
+		(property "Library Audit" "See verification/COMPONENTS.csv and verification/REPORT.md"
 			(at 54.61 59.69 0)
 			(hide yes)
@@
 	)
 	(symbol
-		(lib_id "Device:R_Small")
+		(lib_id "FC01_Project:MICRO_SD__R_Small")
 		(at 154.94 66.04 90)
 		(unit 1)
@@
 			)
 		)
-		(property "Footprint Audit" "OK"
+		(property "Footprint Audit" "See verification/COMPONENTS.csv and verification/REPORT.md"
 			(at 151.13 64.77 90)
 			(hide yes)
@@
 			)
 		)
-		(property "Library Audit" "KiCad standard"
+		(property "Library Audit" "See verification/COMPONENTS.csv and verification/REPORT.md"
 			(at 151.13 64.77 90)
 			(hide yes)
@@
 	)
 	(symbol
-		(lib_id "power:+3V3")
+		(lib_id "FC01_Project:MICRO_SD__+3V3")
 		(at 53.34 57.15 0)
 		(unit 1)
@@
 	)
 	(symbol
-		(lib_id "power:GND")
+		(lib_id "FC01_Project:MICRO_SD__GND")
 		(at 83.82 82.55 0)
 		(unit 1)
