File: MCU.kicad_sch (KiCad schematic)
At the start: 29 parts, among them U2 STM32H743VIT6, Y1 8MHz

Commit message: revert tx / rx
Connections:
- net UART3.RX: now also U2.56 (PD9); no longer U2.55 (PD8)
- net UART3.TX: now also U2.55 (PD8); no longer U2.56 (PD9)
- net UART8.RX: no longer U2.98 (PE1)
- new net UART8.TX: U2.98 (PE1)
Changed lines of the file:
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@@
 		)
 	)
-	(label "IMU3_A_CS"
-		(at 44.45 119.38 180)
+	(label "UART8.TX"
+		(at 133.35 83.82 0)
 		(effects
 			(font
 				(size 1.27 1.27)
 			)
-			(justify right bottom)
+			(justify left bottom)
 		)
 	)
-	(label "UART8.RX"
-		(at 135.89 83.82 0)
+	(label "IMU3_A_CS"
+		(at 44.45 119.38 180)
 		(effects
 			(font
 				(size 1.27 1.27)
 			)
-			(justify left bottom)
+			(justify right bottom)
 		)
 	)
@@
 		)
 	)
+	(label "UART3.RX"
+		(at 139.7 147.32 180)
+		(effects
+			(font
+				(size 1.27 1.27)
+			)
+			(justify right bottom)
+		)
+	)
 	(label "SPI1.CS"
 		(at 278.13 71.12 180)
@@
 		)
 	)
+	(label "UART8.RX"
+		(at 133.35 81.28 0)
+		(effects
+			(font
+				(size 1.27 1.27)
+			)
+			(justify left bottom)
+		)
+	)
 	(label "SPI2.CS"
 		(at 44.45 133.35 180)
@@
 		)
 	)
+	(label "UART3.TX"
+		(at 139.7 144.78 180)
+		(effects
+			(font
+				(size 1.27 1.27)
+			)
+			(justify right bottom)
+		)
+	)
 	(label "SWDIO"
 		(at 207.01 91.44 180)
@@
 		)
 	)
-	(label "UART3.TX"
-		(at 140.97 147.32 180)
-		(effects
-			(font
-				(size 1.27 1.27)
-			)
-			(justify right bottom)
-		)
-	)
 	(label "SPI4.CS"
 		(at 45.72 105.41 180)
@@
 		)
 	)
-	(label "UART3.RX"
-		(at 140.97 144.78 180)
-		(effects
-			(font
-				(size 1.27 1.27)
-			)
-			(justify right bottom)
-		)
-	)
-	(label "UART8.TX"
-		(at 135.89 81.28 0)
-		(effects
-			(font
-				(size 1.27 1.27)
-			)
-			(justify left bottom)
-		)
-	)
 	(label "SPI1.SCLK"
 		(at 46.99 64.77 180)
@@
 		)
 	)
-	(embedded_fonts no)
 )

Commit message: update
Changed lines of the file:
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@@
 		)
 	)
+	(wire
+		(pts
+			(xy 130.81 175.26) (xy 130.81 177.8)
+		)
+		(stroke
+			(width 0)
+			(type default)
+		)
+	)
 	(bus
 		(pts
@@
 	(symbol
 		(lib_id "power:VDD")
-		(at 130.81 177.8 0)
+		(at 130.81 175.26 0)
 		(unit 1)
 		(body_style 1)
@@
 		(fields_autoplaced yes)
 		(property "Reference" "#PWR017"
-			(at 130.81 181.61 0)
+			(at 130.81 179.07 0)
 			(hide yes)
 			(show_name no)
@@
 		)
 		(property "Value" "VCAP"
-			(at 130.81 172.72 0)
+			(at 130.81 170.18 0)
 			(show_name no)
 			(do_not_autoplace no)
@@
 		)
 		(property "Footprint" ""
-			(at 130.81 177.8 0)
+			(at 130.81 175.26 0)
 			(hide yes)
 			(show_name no)
@@
 		)
 		(property "Datasheet" ""
-			(at 130.81 177.8 0)
+			(at 130.81 175.26 0)
 			(hide yes)
 			(show_name no)
@@
 		)
 		(property "Description" "Power symbol creates a global label with name \"VDD\""
-			(at 130.81 177.8 0)
+			(at 130.81 175.26 0)
 			(hide yes)
 			(show_name no)

Commit message: Align D1 Everlight M01 metadata with verified manufacturer/DigiKey status
Parts:
- C1, C10, C11, C12, C13, C14, C15, C2, C3, C4, C5, C6, C7, C8, C9, FB1, JP1, R3, R4, R5, R6, R7, TP1, TP2, TP3, TP4, U2, Y1: Price Checked 2026-09-25 -> 2026-09-26
- D1: value LED_RGB_EP -> 19-337/R6GHBHC-M01/2T; DigiKey Specs RGB LED, 6-pin SMD 1.6x1.6 mm class -> Exact M01 not listed on DigiKey; manufacturer specs: indepe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; DigiKey Status No exact DigiKey listing confirmed; LCSC source retained -> Exact M01 not listed on DigiKey; no DigiKey PN or price ass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; Footprint Audit CHECK supplier drawing before release -> CHECK: 6-SMD 1.6x1.6 mm class matches; verify pad geometry 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; Package 6-SMD RGB LED 1.6x1.6 mm -> 6-SMD, 1.6x1.6x0.35 mm; Price Checked 2026-09-25 -> 2026-09-26
Changed lines of the file:
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@@
 			)
 		)
-		(property "Price Checked" "2026-09-25"
+		(property "Price Checked" "2026-09-26"
 			(at 138.43 179.07 0)
 			(hide yes)
@@
 			)
 		)
-		(property "Price Checked" "2026-09-25"
+		(property "Price Checked" "2026-09-26"
 			(at 100.33 66.0399 0)
 			(hide yes)
@@
 			)
 		)
-		(property "Price Checked" "2026-09-25"
+		(property "Price Checked" "2026-09-26"
 			(at 123.19 25.4 0)
 			(hide yes)
@@
 			)
 		)
-		(property "Price Checked" "2026-09-25"
+		(property "Price Checked" "2026-09-26"
 			(at 247.396 56.134 90)
 			(hide yes)
@@
 			)
 		)
-		(property "Price Checked" "2026-09-25"
+		(property "Price Checked" "2026-09-26"
 			(at 236.22 48.26 90)
 			(hide yes)
@@
 			)
 		)
-		(property "Price Checked" "2026-09-25"
+		(property "Price Checked" "2026-09-26"
 			(at 69.85 147.32 90)
 			(hide yes)
@@
 			)
 		)
-		(property "Price Checked" "2026-09-25"
+		(property "Price Checked" "2026-09-26"
 			(at 134.62 25.4 0)
 			(hide yes)
@@
 			)
 		)
-		(property "Price Checked" "2026-09-25"
+		(property "Price Checked" "2026-09-26"
 			(at 116.84 25.4 0)
 			(hide yes)
@@
 			)
 		)
-		(property "Price Checked" "2026-09-25"
+		(property "Price Checked" "2026-09-26"
 			(at 133.604 53.34 0)
 			(hide yes)
@@
 			)
 		)
-		(property "Price Checked" "2026-09-25"
+		(property "Price Checked" "2026-09-26"
 			(at 132.08 179.07 0)
 			(hide yes)
@@
 			)
 		)
-		(property "Price Checked" "2026-09-25"
+		(property "Price Checked" "2026-09-26"
 			(at 190.5 43.18 0)
 			(hide yes)
@@
 			)
 		)
-		(property "Price Checked" "2026-09-25"
+		(property "Price Checked" "2026-09-26"
 			(at 147.32 25.4 0)
 			(hide yes)
@@
 			)
 		)
-		(property "Price Checked" "2026-09-25"
+		(property "Price Checked" "2026-09-26"
 			(at 118.11 72.39 90)
 			(hide yes)
@@
 			)
 		)
-		(property "Value" "LED_RGB_EP"
+		(property "Value" "19-337/R6GHBHC-M01/2T"
 			(at 63.5 157.48 0)
 			(hide yes)
@@
 			)
 		)
-		(property "Datasheet" "https://lcsc.com/product-detail/Light-Emitting-Diodes-LED_Everlight-Elec-19-337-R6GHBHC-M01-2T_C131204.html"
+		(property "Datasheet" "https://www.everlight-led.cn/zh/datasheet-download/item/19-337-r6ghbhc-m01-2t-2?tmpl=component&type=raw"
 			(at 63.5 149.86 0)
 			(hide yes)
@@
 			)
 		)
-		(property "Description" "RGB LED, 6 pin package with exposed pad"
+		(property "Description" "RGB LED, independent dies, 6-SMD, 1.6x1.6x0.35 mm, 120deg, 624/525/470 nm typ."
 			(at 63.5 148.59 0)
 			(hide yes)
@@
 			)
 		)
-		(property "DigiKey Specs" "RGB LED, 6-pin SMD 1.6x1.6 mm class"
+		(property "DigiKey Specs" "Exact M01 not listed on DigiKey; manufacturer specs: independent RGB, 6-SMD, 1.6x1.6x0.35 mm, 120deg, 624/525/470 nm typ., IF test 5.1/3.5/2.45 mA"
 			(at 63.5 138.43 0)
 			(hide yes)
@@
 			)
 		)
-		(property "Price Checked" "2026-09-25"
+		(property "Price Checked" "2026-09-26"
 			(at 63.5 138.43 0)
 			(hide yes)
@@
 			)
 		)
-		(property "DigiKey Status" "No exact DigiKey listing confirmed; LCSC source retained"
+		(property "DigiKey Status" "Exact M01 not listed on DigiKey; no DigiKey PN or price assigned"
 			(at 63.5 138.43 0)
 			(hide yes)
@@
 			)
 		)
-		(property "Package" "6-SMD RGB LED 1.6x1.6 mm"
+		(property "Package" "6-SMD, 1.6x1.6x0.35 mm"
 			(at 63.5 138.43 0)
 			(hide yes)
@@
 			)
 		)
-		(property "Footprint Audit" "CHECK supplier drawing before release"
+		(property "Footprint Audit" "CHECK: 6-SMD 1.6x1.6 mm class matches; verify pad geometry and pin numbering against Everlight M01 drawing before PCB release"
 			(at 63.5 138.43 0)
 			(hide yes)
@@
 			)
 		)
-		(property "Price Checked" "2026-09-25"
+		(property "Price Checked" "2026-09-26"
 			(at 110.49 25.4062 0)
 			(hide yes)
@@
 			)
 		)
-		(property "Price Checked" "2026-09-25"
+		(property "Price Checked" "2026-09-26"
 			(at 104.14 25.4 0)
 			(hide yes)
@@
 			)
 		)
-		(property "Price Checked" "2026-09-25"
+		(property "Price Checked" "2026-09-26"
 			(at 196.85 43.18 0)
 			(hide yes)
@@
 			)
 		)
-		(property "Price Checked" "2026-09-25"
+		(property "Price Checked" "2026-09-26"
 			(at 110.49 71.12 0)
 			(hide yes)
@@
 			)
 		)
-		(property "Price Checked" "2026-09-25"
+		(property "Price Checked" "2026-09-26"
 			(at 69.85 152.4 90)
 			(hide yes)
@@
 			)
 		)
-		(property "Price Checked" "2026-09-25"
+		(property "Price Checked" "2026-09-26"
 			(at 128.27 25.4 0)
 			(hide yes)
@@
 			)
 		)
-		(property "Price Checked" "2026-09-25"
+		(property "Price Checked" "2026-09-26"
 			(at 247.904 53.594 90)
 			(hide yes)
@@
 			)
 		)
-		(property "Price Checked" "2026-09-25"
+		(property "Price Checked" "2026-09-26"
 			(at 153.67 25.4 0)
 			(hide yes)
@@
 			)
 		)
-		(property "Price Checked" "2026-09-25"
+		(property "Price Checked" "2026-09-26"
 			(at 140.97 25.4 0)
 			(hide yes)
@@
 			)
 		)
-		(property "Price Checked" "2026-09-25"
+		(property "Price Checked" "2026-09-26"
 			(at 173.5933 191.77 0)
 			(hide yes)
@@
 			)
 		)
-		(property "Price Checked" "2026-09-25"
+		(property "Price Checked" "2026-09-26"
 			(at 90.17 59.69 90)
 			(hide yes)
@@
 			)
 		)
-		(property "Price Checked" "2026-09-25"
+		(property "Price Checked" "2026-09-26"
 			(at 247.396 58.674 90)
 			(hide yes)
@@
 			)
 		)
-		(property "Price Checked" "2026-09-25"
+		(property "Price Checked" "2026-09-26"
 			(at 194.31 30.48 90)
 			(hide yes)
@@
 			)
 		)
-		(property "Price Checked" "2026-09-25"
+		(property "Price Checked" "2026-09-26"
 			(at 69.85 142.24 90)
 			(hide yes)
@@
 			)
 		)
-		(property "Price Checked" "2026-09-25"
+		(property "Price Checked" "2026-09-26"
 			(at 248.158 50.8 90)
 			(hide yes)

Commit message: Fix D1-only audit date update
Parts:
- C1, C10, C11, C12, C13, C14, C15, C2, C3, C4, C5, C6, C7, C8, C9, FB1, JP1, R3, R4, R5, R6, R7, TP1, TP2, TP3, TP4, U2, Y1: Price Checked 2026-09-26 -> 2026-09-25
Changed lines of the file:
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@@
 			)
 		)
-		(property "Price Checked" "2026-09-26"
+		(property "Price Checked" "2026-09-25"
 			(at 138.43 179.07 0)
 			(hide yes)
@@
 			)
 		)
-		(property "Price Checked" "2026-09-26"
+		(property "Price Checked" "2026-09-25"
 			(at 100.33 66.0399 0)
 			(hide yes)
@@
 			)
 		)
-		(property "Price Checked" "2026-09-26"
+		(property "Price Checked" "2026-09-25"
 			(at 123.19 25.4 0)
 			(hide yes)
@@
 			)
 		)
-		(property "Price Checked" "2026-09-26"
+		(property "Price Checked" "2026-09-25"
 			(at 247.396 56.134 90)
 			(hide yes)
@@
 			)
 		)
-		(property "Price Checked" "2026-09-26"
+		(property "Price Checked" "2026-09-25"
 			(at 236.22 48.26 90)
 			(hide yes)
@@
 			)
 		)
-		(property "Price Checked" "2026-09-26"
+		(property "Price Checked" "2026-09-25"
 			(at 69.85 147.32 90)
 			(hide yes)
@@
 			)
 		)
-		(property "Price Checked" "2026-09-26"
+		(property "Price Checked" "2026-09-25"
 			(at 134.62 25.4 0)
 			(hide yes)
@@
 			)
 		)
-		(property "Price Checked" "2026-09-26"
+		(property "Price Checked" "2026-09-25"
 			(at 116.84 25.4 0)
 			(hide yes)
@@
 			)
 		)
-		(property "Price Checked" "2026-09-26"
+		(property "Price Checked" "2026-09-25"
 			(at 133.604 53.34 0)
 			(hide yes)
@@
 			)
 		)
-		(property "Price Checked" "2026-09-26"
+		(property "Price Checked" "2026-09-25"
 			(at 132.08 179.07 0)
 			(hide yes)
@@
 			)
 		)
-		(property "Price Checked" "2026-09-26"
+		(property "Price Checked" "2026-09-25"
 			(at 190.5 43.18 0)
 			(hide yes)
@@
 			)
 		)
-		(property "Price Checked" "2026-09-26"
+		(property "Price Checked" "2026-09-25"
 			(at 147.32 25.4 0)
 			(hide yes)
@@
 			)
 		)
-		(property "Price Checked" "2026-09-26"
+		(property "Price Checked" "2026-09-25"
 			(at 118.11 72.39 90)
 			(hide yes)
@@
 			)
 		)
-		(property "Price Checked" "2026-09-26"
+		(property "Price Checked" "2026-09-25"
 			(at 110.49 25.4062 0)
 			(hide yes)
@@
 			)
 		)
-		(property "Price Checked" "2026-09-26"
+		(property "Price Checked" "2026-09-25"
 			(at 104.14 25.4 0)
 			(hide yes)
@@
 			)
 		)
-		(property "Price Checked" "2026-09-26"
+		(property "Price Checked" "2026-09-25"
 			(at 196.85 43.18 0)
 			(hide yes)
@@
 			)
 		)
-		(property "Price Checked" "2026-09-26"
+		(property "Price Checked" "2026-09-25"
 			(at 110.49 71.12 0)
 			(hide yes)
@@
 			)
 		)
-		(property "Price Checked" "2026-09-26"
+		(property "Price Checked" "2026-09-25"
 			(at 69.85 152.4 90)
 			(hide yes)
@@
 			)
 		)
-		(property "Price Checked" "2026-09-26"
+		(property "Price Checked" "2026-09-25"
 			(at 128.27 25.4 0)
 			(hide yes)
@@
 			)
 		)
-		(property "Price Checked" "2026-09-26"
+		(property "Price Checked" "2026-09-25"
 			(at 247.904 53.594 90)
 			(hide yes)
@@
 			)
 		)
-		(property "Price Checked" "2026-09-26"
+		(property "Price Checked" "2026-09-25"
 			(at 153.67 25.4 0)
 			(hide yes)
@@
 			)
 		)
-		(property "Price Checked" "2026-09-26"
+		(property "Price Checked" "2026-09-25"
 			(at 140.97 25.4 0)
 			(hide yes)
@@
 			)
 		)
-		(property "Price Checked" "2026-09-26"
+		(property "Price Checked" "2026-09-25"
 			(at 173.5933 191.77 0)
 			(hide yes)
@@
 			)
 		)
-		(property "Price Checked" "2026-09-26"
+		(property "Price Checked" "2026-09-25"
 			(at 90.17 59.69 90)
 			(hide yes)
@@
 			)
 		)
-		(property "Price Checked" "2026-09-26"
+		(property "Price Checked" "2026-09-25"
 			(at 247.396 58.674 90)
 			(hide yes)
@@
 			)
 		)
-		(property "Price Checked" "2026-09-26"
+		(property "Price Checked" "2026-09-25"
 			(at 194.31 30.48 90)
 			(hide yes)
@@
 			)
 		)
-		(property "Price Checked" "2026-09-26"
+		(property "Price Checked" "2026-09-25"
 			(at 69.85 142.24 90)
 			(hide yes)
@@
 			)
 		)
-		(property "Price Checked" "2026-09-26"
+		(property "Price Checked" "2026-09-25"
 			(at 248.158 50.8 90)
 			(hide yes)

Commit message: update pad
Parts:
- JP1: footprint _pico:SolderJumper_Mini -> Jumper:SolderJumper-2_P1.3mm_Open_RoundedPad1.0x1.5mm
- TP1, TP2, TP3, TP4: footprint (none) -> TestPoint:TestPoint_Pad_1.0x1.0mm
Changed lines of the file:
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@@
 			)
 		)
-		(property "Footprint" ""
+		(property "Footprint" "TestPoint:TestPoint_Pad_1.0x1.0mm"
 			(at 248.92 62.23 0)
 			(hide yes)
@@
 			)
 		)
-		(property "Footprint" ""
+		(property "Footprint" "TestPoint:TestPoint_Pad_1.0x1.0mm"
 			(at 248.92 59.69 0)
 			(hide yes)
@@
 			)
 		)
-		(property "Footprint" "_pico:SolderJumper_Mini"
+		(property "Footprint" "Jumper:SolderJumper-2_P1.3mm_Open_RoundedPad1.0x1.5mm"
 			(at 90.17 63.5 0)
 			(hide yes)
@@
 			)
 		)
-		(property "Footprint" ""
+		(property "Footprint" "TestPoint:TestPoint_Pad_1.0x1.0mm"
 			(at 248.92 64.77 0)
 			(hide yes)
@@
 			)
 		)
-		(property "Footprint" ""
+		(property "Footprint" "TestPoint:TestPoint_Pad_1.0x1.0mm"
 			(at 248.92 57.15 0)
 			(hide yes)
