File: H743_Ardupilot.kicad_sch (KiCad schematic)
At the start: 8 parts, among them U1 USBLC6-2P6

Commit message: update
Changed lines of the file:
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@@
+		)
+	)
+	(wire
+		(pts
+			(xy 90.17 38.1) (xy 90.17 40.64)
+		)
+		(stroke
+			(width 0)
+			(type default)
 		)
 	)
@@
 	(symbol
 		(lib_id "power:VBUS")
-		(at 90.17 40.64 0)
+		(at 90.17 38.1 0)
 		(unit 1)
 		(body_style 1)
@@
 		(fields_autoplaced yes)
 		(property "Reference" "#PWR03"
-			(at 90.17 44.45 0)
+			(at 90.17 41.91 0)
 			(hide yes)
 			(show_name no)
@@
 		)
 		(property "Value" "VBUS"
-			(at 90.17 35.56 0)
+			(at 90.17 33.02 0)
 			(show_name no)
 			(do_not_autoplace no)
@@
 		)
 		(property "Footprint" ""
-			(at 90.17 40.64 0)
+			(at 90.17 38.1 0)
 			(hide yes)
 			(show_name no)
@@
 		)
 		(property "Datasheet" ""
-			(at 90.17 40.64 0)
+			(at 90.17 38.1 0)
 			(hide yes)
 			(show_name no)
@@
 		)
 		(property "Description" "Power symbol creates a global label with name \"VBUS\""
-			(at 90.17 40.64 0)
-			(hide yes)
-			(show_name no)
+			(at 90.17 38.1 0)
+			(hide yes)
+			(show_name no)

Commit message: update cmp number
Other:
- sheet BUZZER ports: added LED_STRIP; removed none
Changed lines of the file:
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@@
+		)
+	)
+	(wire
+		(pts
+			(xy 170.18 106.68) (xy 187.96 106.68)
+		)
+		(stroke
+			(width 0)
+			(type default)
 		)
 	)
@@
 		)
 		(pin "LED_STRIP" input
-			(at 120.65 71.12 180)
-			(effects
-				(font
-					(size 1.27 1.27)
-				)
-				(justify left)
+			(at 170.18 106.68 0)
+			(effects
+				(font
+					(size 1.27 1.27)
+				)
+				(justify right)
 			)
 		)
@@
 	(sheet
 		(at 187.96 100.33)
-		(size 22.86 7.62)
+		(size 22.86 8.89)
 		(exclude_from_sim no)
 		(in_bom yes)
@@
 		)
 		(property "Sheetfile" "BUZZER.kicad_sch"
-			(at 187.96 108.5346 0)
+			(at 187.96 109.8046 0)
 			(hide yes)
 			(show_name no)
@@
 			(effects
 				(font
+					(size 1.27 1.27)
+				)
+				(justify left)
+			)
+		)
+		(pin "LED_STRIP" input
+			(at 187.96 106.68 180)
+			(effects
+				(font

Commit message: update pad
Parts:
- H1, H2, H3, H4: footprint _pico:MountingHole_3.2mm_M3_ISO14580_Pad_TopBottom -> MountingHole:MountingHole_3.2mm_M3_ISO7380_Pad
Changed lines of the file:
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@@
 			)
 		)
-		(property "Footprint" "_pico:MountingHole_3.2mm_M3_ISO14580_Pad_TopBottom"
+		(property "Footprint" "MountingHole:MountingHole_3.2mm_M3_ISO7380_Pad"
 			(at 137.16 161.29 0)
 			(hide yes)
@@
 			)
 		)
-		(property "Footprint" "_pico:MountingHole_3.2mm_M3_ISO14580_Pad_TopBottom"
+		(property "Footprint" "MountingHole:MountingHole_3.2mm_M3_ISO7380_Pad"
 			(at 129.54 161.29 0)
 			(hide yes)
@@
 			)
 		)
-		(property "Footprint" "_pico:MountingHole_3.2mm_M3_ISO14580_Pad_TopBottom"
+		(property "Footprint" "MountingHole:MountingHole_3.2mm_M3_ISO7380_Pad"
 			(at 144.78 161.29 0)
 			(hide yes)
@@
 			)
 		)
-		(property "Footprint" "_pico:MountingHole_3.2mm_M3_ISO14580_Pad_TopBottom"
+		(property "Footprint" "MountingHole:MountingHole_3.2mm_M3_ISO7380_Pad"
 			(at 152.4 161.29 0)
 			(hide yes)

Commit message: update package
Parts:
- U1: value USBLC6-2P6 -> Power_Protection:USBLC6-2P6; footprint EasyEDA:SOT-666-6_L1.6-W1.2-P0.50-LS1.6-BL -> Package_TO_SOT_SMD:SOT-666; LCSC C2682291 -> (none); LCSC Part C2682291 -> (none); MPN TPUSBLC6-2P6 -> (none); Manufacturer TECH PUBLIC -> (none); mouser (none) -> 511-USBLC6-2P6
- USB1: value HC-TYPE-C-16P-01M -> USB_C_Receptacle_USB2.0_16P; footprint EasyEDA:USB-C-SMD_HCTL_HC-TYPE-C-16P-01M -> Connector_USB:USB_C_Receptacle_JAE_DX07S016JA1R1500
Changed lines of the file:
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@@
 			)
 		)
-		(property "Value" "HC-TYPE-C-16P-01M"
+		(property "Value" "USB_C_Receptacle_USB2.0_16P"
 			(at 53.34 35.56 0)
 			(hide yes)
@@
 			)
 		)
-		(property "Footprint" "EasyEDA:USB-C-SMD_HCTL_HC-TYPE-C-16P-01M"
+		(property "Footprint" "Connector_USB:USB_C_Receptacle_JAE_DX07S016JA1R1500"
 			(at 53.34 86.36 0)
 			(hide yes)
@@
 			)
 		)
-		(property "Datasheet" ""
+		(property "Datasheet" "https://www.mouser.com/catalog/specsheets/JAE%20Electronics_01282020_DX07.pdf"
 			(at 53.34 55.88 0)
 			(hide yes)
@@
 			)
 		)
-		(property "Value" "USBLC6-2P6"
+		(property "Value" "Power_Protection:USBLC6-2P6"
 			(at 91.8211 50.8 0)
 			(hide yes)
@@
 			)
 		)
-		(property "Footprint" "EasyEDA:SOT-666-6_L1.6-W1.2-P0.50-LS1.6-BL"
+		(property "Footprint" "Package_TO_SOT_SMD:SOT-666"
 			(at 91.186 62.611 0)
 			(hide yes)
@@
 			)
 		)
-		(property "Datasheet" "https://www.st.com/resource/en/datasheet/usblc6-2.pdf"
+		(property "Datasheet" "https://www.st.com/resource/en/datasheet/cd00050750.pdf"
 			(at 91.186 64.516 0)
 			(hide yes)
@@
 			)
 		)
-		(property "LCSC Part" "C2682291"
-			(at 90.17 55.88 0)
-			(hide yes)
-			(show_name no)
-			(do_not_autoplace no)
-			(effects
-				(font
-					(size 1.27 1.27)
-				)
-			)
-		)
-		(property "LCSC" "C2682291"
-			(at 90.17 55.88 0)
-			(hide yes)
-			(show_name no)
-			(do_not_autoplace no)
-			(effects
-				(font
-					(size 1.27 1.27)
-				)
-			)
-		)
-		(property "MPN" "TPUSBLC6-2P6"
-			(at 90.17 55.88 0)
-			(hide yes)
-			(show_name no)
-			(do_not_autoplace no)
-			(effects
-				(font
-					(size 1.27 1.27)
-				)
-			)
-		)
-		(property "Manufacturer" "TECH PUBLIC"
-			(at 90.17 55.88 0)
-			(hide yes)
+		(property "mouser" "511-USBLC6-2P6"
+			(at 90.17 55.88 0)
+			(hide yes)
+			(show_name no)
+			(do_not_autoplace no)
+			(effects
+				(font
+					(size 1.27 1.27)
+				)
+			)
+		)
+		(property "LCSC" ""
+			(at 90.17 55.88 0)
+			(hide yes)
+			(show_name no)
+			(do_not_autoplace no)
+			(effects
+				(font
+					(size 1.27 1.27)
+				)
+			)
+		)
+		(property "MPN" ""
+			(at 90.17 55.88 0)
+			(hide yes)
+			(show_name no)
+			(do_not_autoplace no)
+			(effects
+				(font
+					(size 1.27 1.27)
+				)
+			)
+		)
+		(property "Manufacturer" ""
+			(at 90.17 55.88 0)
+			(hide yes)

Commit message: Use local JAE USB-C footprint and add USB1 sourcing metadata
Parts:
- USB1: footprint Connector_USB:USB_C_Receptacle_JAE_DX07S016JA1R1500 -> H743_Custom:JAE_DX07S016JA1R1500_16P; DigiKey URL (none) -> https://www.digikey.com/en/products/detail/jae-electronics/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; Footprint Audit (none) -> OK: JAE DX07S016JA1R1500 mechanical geometry; A/B signal pa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; Footprint Source (none) -> KiCad JAE DX07S016JA1R1500 footprint geometry; copied to H7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; JAE Product URL (none) -> https://www.jae.com/en/connectors/series/detail/product/id=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; LCSC C2894899 -> (none); Library Audit (none) -> Project-local H743_Custom footprint; no EasyEDA footprint d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; MPN HC-TYPE-C-16P-01M -> DX07S016JA1R1500; Manufacturer HCTL -> JAE Electronics; Mouser URL (none) -> https://www.mouser.com/ProductDetail/JAE-Electronics/DX07S0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; Package (none) -> USB Type-C receptacle, 16 contacts, right-angle SMT; RS Part Number (none) -> 201-7049
Changed lines of the file:
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@@
 			)
 		)
-		(property "Footprint" "Connector_USB:USB_C_Receptacle_JAE_DX07S016JA1R1500"
+		(property "Footprint" "H743_Custom:JAE_DX07S016JA1R1500_16P"
 			(at 53.34 86.36 0)
 			(hide yes)
@@
 			)
 		)
-		(property "Datasheet" "https://www.mouser.com/catalog/specsheets/JAE%20Electronics_01282020_DX07.pdf"
+		(property "Datasheet" "https://www.jae.com/en/connectors/series/detail/product/id=91780"
 			(at 53.34 55.88 0)
 			(hide yes)
@@
 			)
 		)
-		(property "LCSC" "C2894899"
+		(property "Package" "USB Type-C receptacle, 16 contacts, right-angle SMT"
 			(at 53.34 55.88 0)
 			(hide yes)
@@
 			)
 		)
-		(property "MPN" "HC-TYPE-C-16P-01M"
+		(property "MPN" "DX07S016JA1R1500"
 			(at 53.34 55.88 0)
 			(hide yes)
@@
 			)
 		)
-		(property "Manufacturer" "HCTL"
+		(property "Manufacturer" "JAE Electronics"
 			(at 53.34 55.88 0)
 			(hide yes)
+			(show_name no)
+			(do_not_autoplace no)
+			(effects
+				(font
+					(size 1.27 1.27)
+				)
+			)
+		)
+		(property "JAE Product URL" "https://www.jae.com/en/connectors/series/detail/product/id=91780"
+			(at 53.34 55.88 0)
+			(hide yes)
+			(show_name no)
+			(do_not_autoplace no)
+			(effects
+				(font
+					(size 1.27 1.27)
+				)
+			)
+		)
+		(property "DigiKey URL" "https://www.digikey.com/en/products/detail/jae-electronics/DX07S016JA1R1500/5243883"
+			(at 53.34 55.88 0)
+			(hide yes)
+			(show_name no)
+			(do_not_autoplace no)
+			(effects
+				(font
+					(size 1.27 1.27)
+				)
+			)
+		)
+		(property "Mouser URL" "https://www.mouser.com/ProductDetail/JAE-Electronics/DX07S016JA1R1500"
+			(at 53.34 55.88 0)
+			(hide yes)
+			(show_name no)
+			(do_not_autoplace no)
+			(effects
+				(font
+					(size 1.27 1.27)
+				)
+			)
+		)
+		(property "RS Part Number" "201-7049"
+			(at 53.34 55.88 0)
+			(hide yes)
+			(show_name no)
+			(do_not_autoplace no)
+			(effects
+				(font
+					(size 1.27 1.27)
+				)
+			)
+		)
+		(property "Footprint Source" "KiCad JAE DX07S016JA1R1500 footprint geometry; copied to H743_Custom and shield hold-downs renumbered 25-28 to match the existing symbol"
+			(at 53.34 55.88 0)
+			(hide yes)
+			(show_name no)
+			(do_not_autoplace no)
+			(effects
+				(font
+					(size 1.27 1.27)
+				)
+			)
+		)
+		(property "Footprint Audit" "OK: JAE DX07S016JA1R1500 mechanical geometry; A/B signal pad numbers preserved; four shell pads mapped to symbol pins 25-28"
+			(at 53.34 55.88 0)
+			(hide yes)
+			(show_name no)
+			(do_not_autoplace no)
+			(effects
+				(font
+					(size 1.27 1.27)
+				)
+			)
+		)
+		(property "Library Audit" "Project-local H743_Custom footprint; no EasyEDA footprint dependency"
+			(at 53.34 55.88 0)
+			(hide yes)

Commit message: Clean USB1 metadata for JAE connector
Parts:
- USB1: LCSC Part C2894899 -> (none); Supplier Note (none) -> Industrial JAE connector; use DigiKey/Mouser/RS sourcing ra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
Changed lines of the file:
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@@
 			)
 		)
-		(property "Description" ""
+		(property "Description" "USB Type-C receptacle, USB 2.0, 16 positions, right-angle on-board SMT, JAE DX07S016JA1R1500"
 			(at 53.34 55.88 0)
 			(hide yes)
@@
 			)
 		)
-		(property "LCSC Part" "C2894899"
+		(property "Supplier Note" "Industrial JAE connector; use DigiKey/Mouser/RS sourcing rather than the previous HCTL/LCSC part"
 			(at 53.34 88.9 0)
 			(hide yes)

Commit message: Migrate USB1 symbol to project-local library
Parts:
- USB1: symbol EasyEDA:HC-TYPE-C-16P-01M -> H743_Ardupilot:USB_C_Receptacle_USB2.0_16P_JAE_DX07S016JA1R1500
Changed lines of the file:
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@@
 	)
 	(symbol
-		(lib_id "EasyEDA:HC-TYPE-C-16P-01M")
+		(lib_id "H743_Ardupilot:USB_C_Receptacle_USB2.0_16P_JAE_DX07S016JA1R1500")
 		(at 53.34 55.88 0)
 		(unit 1)
