File: MOTORS[1-4].kicad_sch (KiCad schematic)
At the start: 13 parts, among them U22 ZX-SH1.0-8PWT

Commit message: update name
Parts:
- removed TP10, TP3, TP4, TP5, TP6, TP7, TP8, TP9: (no value), EasyEDA:TestPoint_Pad_1.8x0.9mm, symbol Connector:TestPoint
- R42, R43, R44, R45: value 10R -> 200
Other:
- note removed: "MOTORS [1-4]"
- company: Pierluigi Colangeli, PhD -> (none)
- title: LEVIA H7 -> (none)
- moved on the sheet: R42, R43, R44, R45, U22

Commit message: upsadte SPI4 set to Baro
Other:
- title: (none) -> H743_ARDUPILOT
Changed lines of the file:
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@@
 	(generator "eeschema")
 	(generator_version "10.0")
-	(paper "A5")
+	(paper "A3")
 	(title_block
+		(title "H743_ARDUPILOT")
 		(date "2026-09-24")
 	)

Commit message: re annotate componant globaly
Parts:
- renumbered R42 to R41, R43 to R42, R44 to R43, R45 to R44, U22 to U11
Changed lines of the file:
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@@
 		(dnp no)
 		(fields_autoplaced yes)
-		(property "Reference" "#PWR0119"
+		(property "Reference" "#PWR094"
 			(at 123.19 90.17 0)
 			(hide yes)
@@
 			(project "H743_Ardupilot"
 				(path "/6b768b36-fce6-4be0-9021-6d41bddc3a70/647d5d7a-ea7f-42b5-bbeb-8045c387a5e2"
-					(reference "#PWR0119")
+					(reference "#PWR094")
 					(unit 1)
 				)
@@
 		(in_pos_files yes)
 		(dnp no)
-		(property "Reference" "R42"
+		(property "Reference" "R41"
 			(at 82.55 67.31 90)
 			(show_name no)
@@
 			(project "H743_Ardupilot"
 				(path "/6b768b36-fce6-4be0-9021-6d41bddc3a70/647d5d7a-ea7f-42b5-bbeb-8045c387a5e2"
-					(reference "R42")
+					(reference "R41")
 					(unit 1)
 				)
@@
 		(in_pos_files yes)
 		(dnp no)
-		(property "Reference" "R44"
+		(property "Reference" "R43"
 			(at 82.55 72.39 90)
 			(show_name no)
@@
 			(project "H743_Ardupilot"
 				(path "/6b768b36-fce6-4be0-9021-6d41bddc3a70/647d5d7a-ea7f-42b5-bbeb-8045c387a5e2"
-					(reference "R44")
+					(reference "R43")
 					(unit 1)
 				)
@@
 		(in_pos_files yes)
 		(dnp no)
-		(property "Reference" "R45"
+		(property "Reference" "R44"
 			(at 82.55 74.93 90)
 			(show_name no)
@@
 			(project "H743_Ardupilot"
 				(path "/6b768b36-fce6-4be0-9021-6d41bddc3a70/647d5d7a-ea7f-42b5-bbeb-8045c387a5e2"
-					(reference "R45")
+					(reference "R44")
 					(unit 1)
 				)
@@
 		(in_pos_files yes)
 		(dnp no)
-		(property "Reference" "#PWR0118"
+		(property "Reference" "#PWR093"
 			(at 123.19 59.69 0)
 			(hide yes)
@@
 			(project "H743_Ardupilot"
 				(path "/6b768b36-fce6-4be0-9021-6d41bddc3a70/647d5d7a-ea7f-42b5-bbeb-8045c387a5e2"
-					(reference "#PWR0118")
+					(reference "#PWR093")
 					(unit 1)
 				)
@@
 		(in_pos_files yes)
 		(dnp no)
-		(property "Reference" "R43"
+		(property "Reference" "R42"
 			(at 82.55 69.85 90)
 			(show_name no)
@@
 			(project "H743_Ardupilot"
 				(path "/6b768b36-fce6-4be0-9021-6d41bddc3a70/647d5d7a-ea7f-42b5-bbeb-8045c387a5e2"
-					(reference "R43")
+					(reference "R42")
 					(unit 1)
 				)
@@
 		(in_pos_files yes)
 		(dnp no)
-		(property "Reference" "U22"
+		(property "Reference" "U11"
 			(at 128.27 54.61 0)
 			(show_name no)
@@
 			(project "H743_Ardupilot"
 				(path "/6b768b36-fce6-4be0-9021-6d41bddc3a70/647d5d7a-ea7f-42b5-bbeb-8045c387a5e2"
-					(reference "U22")
+					(reference "U11")
 					(unit 1)
 				)

Commit message: audit DigiKey metadata: MOTORS[1-4].kicad_sch
Parts:
- R41, R42, R43, R44: DigiKey Specs (none) -> 200 ±1%, 0402 (1005), thick film; DigiKey Status (none) -> Active / DigiKey family verified; DigiKey URL (none) -> https://www.digikey.fr/en/products/result?keywords=RC0402FR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; Footprint Audit (none) -> OK; LCSC C25077 -> (none); LCSC Part C25077 -> (none); Library Audit (none) -> KiCad standard; MPN 0402WGF100JTCE -> RC0402FR-07200RL; Manufacturer UNI-ROYAL(Uniroyal Elec) -> YAGEO; Package (none) -> 0402 (1005 Metric); Price Checked (none) -> 2026-09-25
- U11: DigiKey Specs (none) -> SH 1.0 mm, 8-pin right-angle SMD, 1 A, 50 V; DigiKey Status (none) -> No exact DigiKey listing; supplier/LCSC part retained; Footprint Audit (none) -> OK by package-family drawing; final overlay recommended; Library Audit (none) -> EasyEDA external; Manufacturer Megastar(兆星) -> Megastar; Package (none) -> SH1.0 8P right-angle SMD; Price Checked (none) -> 2026-09-25

Commit message: update
Parts:
- renumbered R41 to R47, R42 to R48, R43 to R49, R44 to R50, U11 to U14
Changed lines of the file:
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@@
 		(dnp no)
 		(fields_autoplaced yes)
-		(property "Reference" "#PWR094"
+		(property "Reference" "#PWR0123"
 			(at 123.19 90.17 0)
 			(hide yes)
@@
 			(project "H743_Ardupilot"
 				(path "/6b768b36-fce6-4be0-9021-6d41bddc3a70/647d5d7a-ea7f-42b5-bbeb-8045c387a5e2"
-					(reference "#PWR094")
+					(reference "#PWR0123")
 					(unit 1)
 				)
@@
 		(in_pos_files yes)
 		(dnp no)
-		(property "Reference" "R41"
+		(property "Reference" "R47"
 			(at 82.55 67.31 90)
 			(show_name no)
@@
 			(project "H743_Ardupilot"
 				(path "/6b768b36-fce6-4be0-9021-6d41bddc3a70/647d5d7a-ea7f-42b5-bbeb-8045c387a5e2"
-					(reference "R41")
+					(reference "R47")
 					(unit 1)
 				)
@@
 		(in_pos_files yes)
 		(dnp no)
-		(property "Reference" "R43"
+		(property "Reference" "R49"
 			(at 82.55 72.39 90)
 			(show_name no)
@@
 			(project "H743_Ardupilot"
 				(path "/6b768b36-fce6-4be0-9021-6d41bddc3a70/647d5d7a-ea7f-42b5-bbeb-8045c387a5e2"
-					(reference "R43")
+					(reference "R49")
 					(unit 1)
 				)
@@
 		(in_pos_files yes)
 		(dnp no)
-		(property "Reference" "R44"
+		(property "Reference" "R50"
 			(at 82.55 74.93 90)
 			(show_name no)
@@
 			(project "H743_Ardupilot"
 				(path "/6b768b36-fce6-4be0-9021-6d41bddc3a70/647d5d7a-ea7f-42b5-bbeb-8045c387a5e2"
-					(reference "R44")
+					(reference "R50")
 					(unit 1)
 				)
@@
 		(in_pos_files yes)
 		(dnp no)
-		(property "Reference" "#PWR093"
+		(property "Reference" "#PWR0122"
 			(at 123.19 59.69 0)
 			(hide yes)
@@
 			(project "H743_Ardupilot"
 				(path "/6b768b36-fce6-4be0-9021-6d41bddc3a70/647d5d7a-ea7f-42b5-bbeb-8045c387a5e2"
-					(reference "#PWR093")
+					(reference "#PWR0122")
 					(unit 1)
 				)
@@
 		(in_pos_files yes)
 		(dnp no)
-		(property "Reference" "R42"
+		(property "Reference" "R48"
 			(at 82.55 69.85 90)
 			(show_name no)
@@
 			(project "H743_Ardupilot"
 				(path "/6b768b36-fce6-4be0-9021-6d41bddc3a70/647d5d7a-ea7f-42b5-bbeb-8045c387a5e2"
-					(reference "R42")
+					(reference "R48")
 					(unit 1)
 				)
@@
 		(in_pos_files yes)
 		(dnp no)
-		(property "Reference" "U11"
+		(property "Reference" "U14"
 			(at 128.27 54.61 0)
 			(show_name no)
@@
 			(project "H743_Ardupilot"
 				(path "/6b768b36-fce6-4be0-9021-6d41bddc3a70/647d5d7a-ea7f-42b5-bbeb-8045c387a5e2"
-					(reference "U11")
+					(reference "U14")
 					(unit 1)
 				)

Commit message: ok
Parts:
- U14: footprint EasyEDA:CONN-SMD_8P-P1.00_MEGASTAR_ZX-SH1.0-8PWT -> Connector_JST:JST_SH_SM09B-SRSS-TB_1x09-1MP_P1.00mm_Horizontal
Changed lines of the file:
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@@
 			)
 		)
-		(property "Footprint" "EasyEDA:CONN-SMD_8P-P1.00_MEGASTAR_ZX-SH1.0-8PWT"
+		(property "Footprint" "Connector_JST:JST_SH_SM09B-SRSS-TB_1x09-1MP_P1.00mm_Horizontal"
 			(at 130.81 88.9 0)
 			(hide yes)
