File: MOTORS[1-4].kicad_sch (KiCad schematic)
At the start: 5 parts, among them U14 ZX-SH1.0-8PWT

Commit message: Migrate SM08B-SRSS-TB(LF)(SN) to verified JST symbol and footprint
Parts:
- U14: value ZX-SH1.0-8PWT -> SM08B-SRSS-TB(LF)(SN); symbol EasyEDA:ZX-SH1.0-8PWT -> H743_Ardupilot:JST_SH_SM08B_SRSS_TB_8P; MPN ZX-SH1.0-8PWT -> SM08B-SRSS-TB(LF)(SN); Manufacturer Megastar -> JST
Changed lines of the file:
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@@
 	)
 	(symbol
-		(lib_id "EasyEDA:ZX-SH1.0-8PWT")
+		(lib_id "H743_Ardupilot:JST_SH_SM08B_SRSS_TB_8P")
 		(at 130.81 67.31 0)
 		(unit 1)
@@
 			)
 		)
-		(property "Value" "ZX-SH1.0-8PWT"
+		(property "Value" "SM08B-SRSS-TB(LF)(SN)"
 			(at 137.16 68.5799 0)
 			(hide yes)
@@
 			)
 		)
-		(property "Datasheet" "https://xonstorage.z8.web.core.windows.net/pdf/megastar_zxsh108pwt_apr22_xonlink.pdf"
+		(property "Datasheet" "https://www.jst-mfg.com/product/pdf/eng/eSH.pdf"
 			(at 130.81 91.44 0)
 			(hide yes)
@@
 			)
 		)
-		(property "Manufacturer" "Megastar"
+		(property "Manufacturer" "JST"
 			(at 130.81 93.98 0)
 			(hide yes)
@@
 			)
 		)
-		(property "MPN" "ZX-SH1.0-8PWT"
+		(property "MPN" "SM08B-SRSS-TB(LF)(SN)"
 			(at 130.81 96.52 0)
 			(hide yes)

Commit message: Review component footprints, restore local libraries and reconcile PCB pads
Parts:
- R47, R48, R49, R50: symbol Device:R_Small -> FC01_Project:MOTORS1-4__R_Small; Footprint Audit OK -> See verification/COMPONENTS.csv and verification/REPORT.md; Library Audit KiCad standard -> See verification/COMPONENTS.csv and verification/REPORT.md
- U14: footprint Connector_JST:JST_SH_SM09B-SRSS-TB_1x09-1MP_P1.00mm_Horizontal -> H743_Custom:JST_SH_SM08B-SRSS-TB_1x08_P1.00mm_Horizontal_GNDtabs; symbol H743_Ardupilot:JST_SH_SM08B_SRSS_TB_8P -> FC01_Project:MOTORS1-4__JST_SH_SM08B_SRSS_TB_8P; Footprint Audit OK by package-family drawing; final overlay recommended -> See verification/COMPONENTS.csv and verification/REPORT.md; Library Audit EasyEDA external -> See verification/COMPONENTS.csv and verification/REPORT.md; Package SH1.0 8P right-angle SMD -> JST SH 8 contacts, P1.00 mm, side entry; mounting tabs pads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
Changed lines of the file:
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@@
 	)
 	(symbol
-		(lib_id "power:GND")
+		(lib_id "FC01_Project:MOTORS1-4__GND")
 		(at 123.19 83.82 0)
 		(unit 1)
@@
 	)
 	(symbol
-		(lib_id "Device:R_Small")
+		(lib_id "FC01_Project:MOTORS1-4__R_Small")
 		(at 87.63 68.58 90)
 		(unit 1)
@@
 			)
 		)
-		(property "Footprint Audit" "OK"
+		(property "Footprint Audit" "See verification/COMPONENTS.csv and verification/REPORT.md"
 			(at 82.55 67.31 90)
 			(hide yes)
@@
 			)
 		)
-		(property "Library Audit" "KiCad standard"
+		(property "Library Audit" "See verification/COMPONENTS.csv and verification/REPORT.md"
 			(at 82.55 67.31 90)
 			(hide yes)
@@
 	)
 	(symbol
-		(lib_id "Device:R_Small")
+		(lib_id "FC01_Project:MOTORS1-4__R_Small")
 		(at 87.63 73.66 90)
 		(unit 1)
@@
 			)
 		)
-		(property "Footprint Audit" "OK"
+		(property "Footprint Audit" "See verification/COMPONENTS.csv and verification/REPORT.md"
 			(at 82.55 72.39 90)
 			(hide yes)
@@
 			)
 		)
-		(property "Library Audit" "KiCad standard"
+		(property "Library Audit" "See verification/COMPONENTS.csv and verification/REPORT.md"
 			(at 82.55 72.39 90)
 			(hide yes)
@@
 	)
 	(symbol
-		(lib_id "Device:R_Small")
+		(lib_id "FC01_Project:MOTORS1-4__R_Small")
 		(at 87.63 76.2 90)
 		(unit 1)
@@
 			)
 		)
-		(property "Footprint Audit" "OK"
+		(property "Footprint Audit" "See verification/COMPONENTS.csv and verification/REPORT.md"
 			(at 82.55 74.93 90)
 			(hide yes)
@@
 			)
 		)
-		(property "Library Audit" "KiCad standard"
+		(property "Library Audit" "See verification/COMPONENTS.csv and verification/REPORT.md"
 			(at 82.55 74.93 90)
 			(hide yes)
@@
 	)
 	(symbol
-		(lib_id "power:VAA")
+		(lib_id "FC01_Project:MOTORS1-4__VAA")
 		(at 123.19 55.88 0)
 		(unit 1)
@@
 	)
 	(symbol
-		(lib_id "Device:R_Small")
+		(lib_id "FC01_Project:MOTORS1-4__R_Small")
 		(at 87.63 71.12 90)
 		(unit 1)
@@
 			)
 		)
-		(property "Footprint Audit" "OK"
+		(property "Footprint Audit" "See verification/COMPONENTS.csv and verification/REPORT.md"
 			(at 82.55 69.85 90)
 			(hide yes)
@@
 			)
 		)
-		(property "Library Audit" "KiCad standard"
+		(property "Library Audit" "See verification/COMPONENTS.csv and verification/REPORT.md"
 			(at 82.55 69.85 90)
 			(hide yes)
@@
 	)
 	(symbol
-		(lib_id "H743_Ardupilot:JST_SH_SM08B_SRSS_TB_8P")
+		(lib_id "FC01_Project:MOTORS1-4__JST_SH_SM08B_SRSS_TB_8P")
 		(at 130.81 67.31 0)
 		(unit 1)
@@
 			)
 		)
-		(property "Footprint" "Connector_JST:JST_SH_SM09B-SRSS-TB_1x09-1MP_P1.00mm_Horizontal"
+		(property "Footprint" "H743_Custom:JST_SH_SM08B-SRSS-TB_1x08_P1.00mm_Horizontal_GNDtabs"
 			(at 130.81 88.9 0)
 			(hide yes)
@@
 			)
 		)
-		(property "Package" "SH1.0 8P right-angle SMD"
+		(property "Package" "JST SH 8 contacts, P1.00 mm, side entry; mounting tabs pads 9/10"
 			(at 128.27 54.61 0)
 			(hide yes)
@@
 			)
 		)
-		(property "Footprint Audit" "OK by package-family drawing; final overlay recommended"
+		(property "Footprint Audit" "See verification/COMPONENTS.csv and verification/REPORT.md"
 			(at 128.27 54.61 0)
 			(hide yes)
@@
 			)
 		)
-		(property "Library Audit" "EasyEDA external"
+		(property "Library Audit" "See verification/COMPONENTS.csv and verification/REPORT.md"
 			(at 128.27 54.61 0)
 			(hide yes)
