File: MOTORS[1-4].kicad_sch (KiCad schematic)
At the start: 5 parts, among them U14 SM08B-SRSS-TB(LF)(SN)

Commit message: pos down
Parts:
- added R52: 200, Resistor_SMD:R_0402_1005Metric, symbol FC01_Project:UART_I2C__R_Small
Connections:
- net UART8.RX: now also R52.1; no longer U14.4
- new net Rx8: R52.2, U14.4
