File: H743_Ardupilot.kicad_pcb (KiCad board)
At the start: 2 copper layers, 36.5 x 36.5 mm, 141 parts, among them J1 Conn_01x04, J10 Conn_01x03, J11 Conn_01x03, J12 10067099-200LF, J2 Conn_01x04, J3 Conn_01x04, J4 Conn_01x06, J5 Conn_01x04, J6 Conn_01x04, J7 Conn_01x04, J8 Conn_01x04, J9 Conn_01x04, Q1 AO3400A, U10 LSM6DSV16X, U12 BMP581, U2 STM32H743VIT6, U8 ZX-SH1.0-4PWT, U9 BMI088

Commit message: update package
Parts:
- added USB1: USB_C_Receptacle_USB2.0_16P, Connector_USB:USB_C_Receptacle_JAE_DX07S016JA1R1500, F.Cu at (93.0, 88.6)
- moved J12 51.6 mm to (80.8, 103.2), turned to -90 degrees
- moved U8 50.3 mm to (87.8, 119.2)
- moved L1 45.5 mm to (156.7, 93.5)
- moved L2 45.5 mm to (156.7, 99.0)
- moved U2 35.7 mm to (131.5, 87.5)

Commit message: ok
Parts:
- added U1: Power_Protection:USBLC6-2P6, Package_TO_SOT_SMD:SOT-666, F.Cu at (82.5, 88.0)
- added U14: ZX-SH1.0-8PWT, Connector_JST:JST_SH_SM09B-SRSS-TB_1x09-1MP_P1.00mm_Horizontal, F.Cu at (77.7, 100.4)
- added U3: LMR43620R5RPER, H743_Custom:TI_RPE0009B_VQFN-HR-9_2x2mm, F.Cu at (86.5, 96.5)
- added U4: LMR604303SRAKRQ1, H743_Custom:TI_RAK0009A_WQFN-HR-9_2.5x2.0mm, F.Cu at (82.5, 107.0)
- added U5: AP7361C-33FGE-7, Package_DFN_QFN:DFN-8-1EP_3x3mm_P0.65mm_EP1.5x2.25mm, F.Cu at (126.5, 107.3)
- added U6: AP7361C-33FGE-7, Package_DFN_QFN:DFN-8-1EP_3x3mm_P0.65mm_EP1.5x2.25mm, F.Cu at (126.5, 111.8)
- USB1: footprint Connector_USB:USB_C_Receptacle_JAE_DX07S016JA1R1500 -> H743_Custom:JAE_DX07S016JA1R1500_16P
- moved C17 123.3 mm to (82.5, 97.5), turned to 180 degrees
- moved D2 122.9 mm to (83.5, 93.0), turned to 180 degrees
- moved C22 122.8 mm to (82.0, 109.5), turned to 180 degrees
- moved C21 122.5 mm to (84.0, 98.0), turned to 90 degrees
- moved R9 120.2 mm to (82.0, 104.0), turned to 90 degrees
- moved R11 119.9 mm to (82.0, 110.5), turned to 180 degrees
- moved C25 118.7 mm to (89.0, 97.5), turned to 180 degrees
- moved R10 117.3 mm to (84.5, 109.5)
- moved R8 117.1 mm to (84.5, 107.5), turned to 90 degrees
- moved C20 112.4 mm to (87.0, 99.0)
- moved C27 109.2 mm to (80.0, 115.0), turned to 180 degrees
- moved C26 109.0 mm to (80.0, 113.0), turned to 180 degrees
- moved D3 107.9 mm to (90.0, 100.5), turned to -90 degrees
- moved C16 107.0 mm to (83.0, 96.0), turned to 180 degrees
- moved D4 105.0 mm to (93.5, 96.0), turned to 90 degrees
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
Commit message: Sync USB1 DX07S016JA1R1500 footprint on PCB
Parts:
- USB1: value USB_C_Receptacle_USB2.0_16P -> DX07S016JA1R1500
Changed lines of the file:
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@@
 			)
 		)
-		(property "Value" "USB_C_Receptacle_USB2.0_16P"
+		(property "Value" "DX07S016JA1R1500"
 			(at 0 5 180)
 			(layer "F.Fab")
@@
 			)
 		)
-		(property "Datasheet" "https://www.jae.com/en/connectors/series/detail/product/id=91780"
+		(property "Datasheet" "https://mm.digikey.com/Volume0/opasdata/d220001/medias/docus/7162/670_DX07S016JA1R1500.pdf"
 			(at 0 0 180)
 			(unlocked yes)
@@
 			)
 		)
-		(property "Description" "USB Type-C receptacle, USB 2.0, 16 positions, right-angle on-board SMT, JAE DX07S016JA1R1500"
+		(property "Description" "JAE DX07S016JA1R1500; USB Type-C USB 2.0 receptacle; 16 positions (24 = 16+8 dummy per DigiKey); on-board/right-angle, 1-row SMT + shell through-hole; shell DIP 0.9 mm; 5 A max; 48 Vrms; -40..+85 C; 10000 mating cycles. Supplier PDF: https://mm.digikey.com/Volume0/opasdata/d220001/medias/docus/7162/670_DX07S016JA1R1500.pdf"
 			(at 0 0 180)
 			(unlocked yes)
@@
 			)
 		)
+		(property "DigiKey Part Number" "670-DX07S016JA1R1500TR-ND"
+			(at 0 0 180)
+			(unlocked yes)
+			(layer "F.Fab")
+			(hide yes)
+			(effects
+				(font
+					(size 1 1)
+					(thickness 0.15)
+				)
+			)
+		)
 		(property "Manufacturer" "JAE Electronics"
 			(at 0 0 180)
@@
 		)
 		(property "DigiKey URL" "https://www.digikey.com/en/products/detail/jae-electronics/DX07S016JA1R1500/5243883"
+			(at 0 0 180)
+			(unlocked yes)
+			(layer "F.Fab")
+			(hide yes)
+			(effects
+				(font
+					(size 1 1)
+					(thickness 0.15)
+				)
+			)
+		)
+		(property "DigiKey Unit Price EUR" "0.86782"
+			(at 0 0 180)
+			(unlocked yes)
+			(layer "F.Fab")
+			(hide yes)
+			(effects
+				(font
+					(size 1 1)
+					(thickness 0.15)
+				)
+			)
+		)
+		(property "DigiKey Price Qty" "1500 (Tape & Reel)"
+			(at 0 0 180)
+			(unlocked yes)
+			(layer "F.Fab")
+			(hide yes)
+			(effects
+				(font
+					(size 1 1)
+					(thickness 0.15)
+				)
+			)
+		)
+		(property "Price Checked" "2026-09-27"
+			(at 0 0 180)
+			(unlocked yes)
+			(layer "F.Fab")
+			(hide yes)
+			(effects
+				(font
+					(size 1 1)
+					(thickness 0.15)
+				)
+			)
+		)
+		(property "Supplier PDF" "https://mm.digikey.com/Volume0/opasdata/d220001/medias/docus/7162/670_DX07S016JA1R1500.pdf"
+			(at 0 0 180)
+			(unlocked yes)
+			(layer "F.Fab")
+			(hide yes)
+			(effects
+				(font
+					(size 1 1)
+					(thickness 0.15)
+				)
+			)
+		)
+		(property "JAE Drawing" "SJ121836 / SJ121837"
 			(at 0 0 180)
 			(unlocked yes)
@@
 			(unit
 				(name "A")
-				(pins "25" "26" "27" "28" "A1" "A12" "B1" "B12" "A4" "A9" "B4" "B9" "A5"
-					"B5" "A6" "B6" "A7" "B7" "A8" "B8"
-				)
+				(pins "SH1" "SH2" "SH3" "SH4" "SH5" "SH6" "A1/B12" "A12/B1" "A4/B9" "B4/A9" "A5" "B5" "A6" "B6" "A7" "B7" "A8" "B8")
 			)
 		)
@@
 		(pad "" np_thru_hole circle
 			(at -3 -1.95 180)
-			(size 0.6 0.6)
-			(drill 0.6)
+			(size 0.63 0.63)
+			(drill 0.63)
 			(layers "*.Cu" "*.Mask")
 		)
-		(pad "" smd roundrect
+		(pad "SH1" smd roundrect
 			(at -1.4 1.15 180)
 			(size 1 2)
 			(layers "F.Cu" "F.Mask" "F.Paste")
 			(roundrect_rratio 0.25)
-		)
-		(pad "" smd roundrect
+			(net "GND")
+			(pinfunction "SHIELD")
+			(pintype "passive"))
+		(pad "SH2" smd roundrect
 			(at 1.4 1.15 180)
 			(size 1 2)
 			(layers "F.Cu" "F.Mask" "F.Paste")
 			(roundrect_rratio 0.25)
-		)
-		(pad "" np_thru_hole oval
+			(net "GND")
+			(pinfunction "SHIELD")
+			(pintype "passive"))
+		(pad "" np_thru_hole circle
 			(at 3 -1.95 180)
-			(size 0.85 0.6)
-			(drill oval 0.85 0.6)
+			(size 0.63 0.63)
+			(drill 0.63)
 			(layers "*.Cu" "*.Mask")
 		)
-		(pad "25" thru_hole oval
+		(pad "SH3" thru_hole oval
 			(at -4.32 -2.675 180)
-			(size 1.3 2.3)
-			(drill oval 0.6 1.6)
+			(size 1.158 2.316)
+			(drill oval 0.65 1.65)
 			(property pad_prop_mechanical)
 			(layers "*.Cu" "*.Mask")
 			(remove_unused_layers no)
 			(net "GND")
-			(pinfunction "SHIELD_25")
-			(pintype "passive")
-		)
-		(pad "26" thru_hole oval
+			(pinfunction "SHIELD")
+			(pintype "passive")
+		)
+		(pad "SH5" thru_hole oval
 			(at -4.32 1.15 180)
-			(size 1.3 2.6)
-			(drill oval 0.6 1.9)
+			(size 1.2 2.4)
+			(drill oval 0.65 1.95)
 			(property pad_prop_mechanical)
 			(layers "*.Cu" "*.Mask")
 			(remove_unused_layers no)
 			(net "GND")
-			(pinfunction "SHIELD_26")
-			(pintype "passive")
-		)
-		(pad "27" thru_hole oval
+			(pinfunction "SHIELD")
+			(pintype "passive")
+		)
+		(pad "SH4" thru_hole oval
 			(at 4.32 -2.675 180)
-			(size 1.3 2.3)
-			(drill oval 0.6 1.6)
+			(size 1.158 2.316)
+			(drill oval 0.65 1.65)
 			(property pad_prop_mechanical)
 			(layers "*.Cu" "*.Mask")
 			(remove_unused_layers no)
 			(net "GND")
-			(pinfunction "SHIELD_27")
-			(pintype "passive")
-		)
-		(pad "28" thru_hole oval
+			(pinfunction "SHIELD")
+			(pintype "passive")
+		)
+		(pad "SH6" thru_hole oval
 			(at 4.32 1.15 180)
-			(size 1.3 2.6)
-			(drill oval 0.6 1.9)
+			(size 1.2 2.4)
+			(drill oval 0.65 1.95)
 			(property pad_prop_mechanical)
 			(layers "*.Cu" "*.Mask")
 			(remove_unused_layers no)
 			(net "GND")
-			(pinfunction "SHIELD_28")
-			(pintype "passive")
-		)
-		(pad "A1" smd roundrect
+			(pinfunction "SHIELD")
+			(pintype "passive")
+		)
+		(pad "A1/B12" smd roundrect
 			(at -3.1 -3.05 180)
 			(size 0.52 1)
@@
 			(roundrect_rratio 0.25)
 			(net "GND")
-			(pinfunction "GND_A1")
-			(pintype "passive")
-		)
-		(pad "A4" smd roundrect
+			(pinfunction "A1/B12")
+			(pintype "passive")
+		)
+		(pad "A4/B9" smd roundrect
 			(at -2.35 -3.05 180)
 			(size 0.52 1)
@@
 			(roundrect_rratio 0.25)
 			(net "VBUS")
-			(pinfunction "VBUS_A4")
+			(pinfunction "A4/B9")
 			(pintype "passive")
 		)
@@
 			(pintype "bidirectional+no_connect")
 		)
-		(pad "A9" smd roundrect
+		(pad "A12/B1" smd roundrect
+			(at 3.1 -3.05 180)
+			(size 0.52 1)
+			(layers "F.Cu" "F.Mask" "F.Paste")
+			(roundrect_rratio 0.25)
+			(net "GND")
+			(pinfunction "A12/B1")
+			(pintype "passive")
+		)
+		(pad "B4/A9" smd roundrect
 			(at 2.35 -3.05 180)
 			(size 0.52 1)
@@
 			(roundrect_rratio 0.25)
 			(net "VBUS")
-			(pinfunction "VBUS_A9")
-			(pintype "passive")
-		)
-		(pad "A12" smd roundrect
-			(at 3.1 -3.05 180)
-			(size 0.52 1)
-			(layers "F.Cu" "F.Mask" "F.Paste")
-			(roundrect_rratio 0.25)
-			(net "GND")
-			(pinfunction "GND_A12")
-			(pintype "passive")
-		)
-		(pad "B1" smd roundrect
-			(at 3.1 -3.05 180)
-			(size 0.52 1)
-			(layers "F.Cu" "F.Mask" "F.Paste")
-			(roundrect_rratio 0.25)
-			(net "GND")
-			(pinfunction "GND_B1")
-			(pintype "passive")
-		)
-		(pad "B4" smd roundrect
-			(at 2.35 -3.05 180)
-			(size 0.52 1)
-			(layers "F.Cu" "F.Mask" "F.Paste")
-			(roundrect_rratio 0.25)
-			(net "VBUS")
-			(pinfunction "VBUS_B4")
+			(pinfunction "B4/A9")
 			(pintype "passive")
 		)
@@
 			(pintype "bidirectional+no_connect")
 		)
-		(pad "B9" smd roundrect
-			(at -2.35 -3.05 180)
-			(size 0.52 1)
-			(layers "F.Cu" "F.Mask" "F.Paste")
-			(roundrect_rratio 0.25)
-			(net "VBUS")
-			(pinfunction "VBUS_B9")
-			(pintype "passive")
-		)
-		(pad "B12" smd roundrect
-			(at -3.1 -3.05 180)
-			(size 0.52 1)
-			(layers "F.Cu" "F.Mask" "F.Paste")
-			(roundrect_rratio 0.25)
-			(net "GND")
-			(pinfunction "GND_B12")
-			(pintype "passive")
-		)
 		(embedded_fonts no)

Commit message: Update USB1 ESD protection footprint and package
Parts:
- U1: value Power_Protection:USBLC6-2P6 -> USBLC6-2P6; footprint Package_TO_SOT_SMD:SOT-666 -> H743_Custom:ST_USBLC6-2P6_SOT-666
Changed lines of the file:
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@@
 		)
 	)
-	(footprint "Package_TO_SOT_SMD:SOT-666"
+	(footprint "H743_Custom:ST_USBLC6-2P6_SOT-666"
 		(layer "F.Cu")
 		(at 82.5 88 -90)
-		(descr "SOT666")
-		(tags "SOT-666")
+		(descr "STMicroelectronics USBLC6-2P6, SOT-666; land pattern from supplier CAD ZIP; package 1.6 x 1.6 x 0.55 mm")
+		(tags "ST USBLC6-2P6 SOT-666 USB ESD")
 		(property "Reference" "U1"
 			(at 0 -2 90)
@@
 			)
 		)
-		(property "Value" "Power_Protection:USBLC6-2P6"
+		(property "Value" "USBLC6-2P6"
 			(at 0 1.75 90)
 			(layer "F.Fab")
@@
 			)
 		)
-		(property "Datasheet" "https://www.st.com/resource/en/datasheet/cd00050750.pdf"
+		(property "Datasheet" "https://www.st.com/resource/en/datasheet/usblc6-2.pdf"
 			(at 0 0 270)
 			(unlocked yes)
@@
 			)
 		)
-		(property "Description" "Very low capacitance ESD protection diode, 2 data-line, SOT-666"
+		(property "Description" "STMicroelectronics USBLC6-2P6; ESD protection for USB1 D+/D- and VBUS; SOT-666 1.6 x 1.6 x 0.55 mm; supplier PDF https://www.st.com/resource/en/datasheet/usblc6-2.pdf"
 			(at 0 0 270)
 			(unlocked yes)
@@
 			)
 		)
-		(property "MPN" ""
-			(at 0 0 270)
-			(unlocked yes)
-			(layer "F.Fab")
-			(hide yes)
-			(effects
-				(font
-					(size 1 1)
-					(thickness 0.15)
-				)
-			)
-		)
-		(property "Manufacturer" ""
+		(property "MPN" "USBLC6-2P6"
+			(at 0 0 270)
+			(unlocked yes)
+			(layer "F.Fab")
+			(hide yes)
+			(effects
+				(font
+					(size 1 1)
+					(thickness 0.15)
+				)
+			)
+		)
+		(property "Manufacturer" "STMicroelectronics"
 			(at 0 0 270)
 			(unlocked yes)
@@
 		(duplicate_pad_numbers_are_jumpers no)
 		(fp_line
-			(start 0.65 0.99)
-			(end -0.65 0.99)
+			(start 0.65 0.855)
+			(end -0.65 0.855)
 			(stroke
 				(width 0.12)
@@
 		)
 		(fp_line
-			(start 0.65 -0.99)
-			(end -0.4 -0.99)
+			(start 0.65 -0.855)
+			(end -0.65 -0.855)
 			(stroke
 				(width 0.12)
@@
 		)
 		(pad "1" smd roundrect
-			(at -0.85 -0.5375 270)
-			(size 0.5 0.375)
+			(at -0.69 -0.5)
+			(size 0.75 0.35)
 			(layers "F.Cu" "F.Mask" "F.Paste")
 			(roundrect_rratio 0.25)
@@
 		)
 		(pad "2" smd roundrect
-			(at -0.925 0 270)
-			(size 0.65 0.3)
+			(at -0.69 0)
+			(size 0.75 0.35)
 			(layers "F.Cu" "F.Mask" "F.Paste")
 			(roundrect_rratio 0.25)
@@
 		)
 		(pad "3" smd roundrect
-			(at -0.85 0.5375 270)
-			(size 0.5 0.375)
+			(at -0.69 0.5)
+			(size 0.75 0.35)
 			(layers "F.Cu" "F.Mask" "F.Paste")
 			(roundrect_rratio 0.25)
@@
 		)
 		(pad "4" smd roundrect
-			(at 0.85 0.5375 270)
-			(size 0.5 0.375)
+			(at 0.69 0.5)
+			(size 0.75 0.35)
 			(layers "F.Cu" "F.Mask" "F.Paste")
 			(roundrect_rratio 0.25)
@@
 		)
 		(pad "5" smd roundrect
-			(at 0.925 0 270)
-			(size 0.65 0.3)
+			(at 0.69 0)
+			(size 0.75 0.35)
 			(layers "F.Cu" "F.Mask" "F.Paste")
 			(roundrect_rratio 0.25)
@@
 		)
 		(pad "6" smd roundrect
-			(at 0.85 -0.5375 270)
-			(size 0.5 0.375)
-			(layers "F.Cu" "F.Mask" "F.Paste")
-			(roundrect_rratio 0.25)
+			(at 0.69 -0.5)
+			(size 0.75 0.35)
+			(layers "F.Cu" "F.Mask" "F.Paste")
+			(roundrect_rratio 0.25)

Commit message: Fix CAN schematic symbol and update SMAJ30CA footprint
Parts:
- D2: footprint Diode_SMD:D_SMA -> H743_Custom:SMAJ30CA_SMA_LTF
Changed lines of the file:
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@@
 		)
 	)
-	(footprint "Diode_SMD:D_SMA"
+	(footprint "H743_Custom:SMAJ30CA_SMA_LTF"
 		(layer "F.Cu")
 		(at 83.5 93 180)
-		(descr "Diode SMA (DO-214AC)")
-		(tags "Diode SMA (DO-214AC)")
+		(descr "SMAJ30CA DO-214AC/SMA; nominal SMASeries_LTF land pattern from user-supplied CAD ZIP")
+		(tags "SMAJ30CA SMA DO-214AC SMASeries LTF TVS")
 		(property "Reference" "D2"
 			(at 0 -2.5 0)
@@
 			)
 		)
-		(property "Footprint Audit" "OK"
-			(at 0 0 180)
-			(unlocked yes)
-			(layer "F.Fab")
-			(hide yes)
-			(effects
-				(font
-					(size 1 1)
-					(thickness 0.15)
-				)
-			)
-		)
-		(property "Library Audit" "KiCad standard"
+		(property "Footprint Audit" "VERIFIED: supplied SMAJ30CA.zip nominal SMASeries_LTF land pattern; pads 1.651 x 2.1844 mm at +/-1.7018 mm"
+			(at 0 0 180)
+			(unlocked yes)
+			(layer "F.Fab")
+			(hide yes)
+			(effects
+				(font
+					(size 1 1)
+					(thickness 0.15)
+				)
+			)
+		)
+		(property "Library Audit" "Project-local H743_Custom footprint"
 			(at 0 0 180)
 			(unlocked yes)
@@
 		(duplicate_pad_numbers_are_jumpers no)
 		(fp_line
-			(start -3.51 1.65)
-			(end 2 1.65)
-			(stroke
-				(width 0.12)
-				(type solid)
-			)
-			(layer "F.SilkS")
-		)
-		(fp_line
-			(start -3.51 -1.65)
-			(end 2 -1.65)
-			(stroke
-				(width 0.12)
-				(type solid)
-			)
-			(layer "F.SilkS")
-		)
-		(fp_line
-			(start -3.51 -1.65)
-			(end -3.51 1.65)
-			(stroke
-				(width 0.12)
-				(type solid)
-			)
-			(layer "F.SilkS")
-		)
-		(fp_line
-			(start 3.5 1.75)
-			(end -3.5 1.75)
-			(stroke
-				(width 0.05)
-				(type solid)
-			)
-			(layer "F.CrtYd")
-		)
-		(fp_line
-			(start 3.5 -1.75)
-			(end 3.5 1.75)
-			(stroke
-				(width 0.05)
-				(type solid)
-			)
-			(layer "F.CrtYd")
-		)
-		(fp_line
-			(start -3.5 1.75)
-			(end -3.5 -1.75)
-			(stroke
-				(width 0.05)
-				(type solid)
-			)
-			(layer "F.CrtYd")
-		)
-		(fp_line
-			(start -3.5 -1.75)
-			(end 3.5 -1.75)
-			(stroke
-				(width 0.05)
-				(type solid)
-			)
-			(layer "F.CrtYd")
-		)
-		(fp_line
-			(start 2.3 1.5)
-			(end -2.3 1.5)
-			(stroke
-				(width 0.1)
-				(type solid)
-			)
-			(layer "F.Fab")
-		)
-		(fp_line
-			(start 2.3 -1.5)
-			(end 2.3 1.5)
-			(stroke
-				(width 0.1)
-				(type solid)
-			)
-			(layer "F.Fab")
-		)
-		(fp_line
-			(start 2.3 -1.5)
-			(end -2.3 -1.5)
-			(stroke
-				(width 0.1)
-				(type solid)
-			)
-			(layer "F.Fab")
-		)
-		(fp_line
-			(start 0.50118 0.75032)
-			(end 0.50118 -0.79908)
-			(stroke
-				(width 0.1)
-				(type solid)
-			)
-			(layer "F.Fab")
-		)
-		(fp_line
-			(start 0.50118 0.00102)
-			(end 1.4994 0.00102)
-			(stroke
-				(width 0.1)
-				(type solid)
-			)
-			(layer "F.Fab")
-		)
-		(fp_line
-			(start -0.64944 0.00102)
-			(end 0.50118 0.75032)
-			(stroke
-				(width 0.1)
-				(type solid)
-			)
-			(layer "F.Fab")
-		)
-		(fp_line
-			(start -0.64944 0.00102)
-			(end 0.50118 -0.79908)
-			(stroke
-				(width 0.1)
-				(type solid)
-			)
-			(layer "F.Fab")
-		)
-		(fp_line
-			(start -0.64944 0.00102)
-			(end -1.55114 0.00102)
-			(stroke
-				(width 0.1)
-				(type solid)
-			)
-			(layer "F.Fab")
-		)
-		(fp_line
-			(start -0.64944 -0.79908)
-			(end -0.64944 0.80112)
-			(stroke
-				(width 0.1)
-				(type solid)
-			)
-			(layer "F.Fab")
-		)
-		(fp_line
-			(start -2.3 1.5)
-			(end -2.3 -1.5)
-			(stroke
-				(width 0.1)
-				(type solid)
-			)
+			(start -3.048 1.0795)
+			(end -3.048 -1.0795)
+			(stroke (width 0.1524) (type solid))
+			(layer "F.CrtYd")
+		)
+		(fp_line
+			(start -3.048 -1.0795)
+			(end -2.8956 -1.0795)
+			(stroke (width 0.1524) (type solid))
+			(layer "F.CrtYd")
+		)
+		(fp_line
+			(start 2.8956 -1.0795)
+			(end 3.048 -1.0795)
+			(stroke (width 0.1524) (type solid))
+			(layer "F.CrtYd")
+		)
+		(fp_line
+			(start 3.048 -1.0795)
+			(end 3.048 1.0795)
+			(stroke (width 0.1524) (type solid))
+			(layer "F.CrtYd")
+		)
+		(fp_line
+			(start 3.048 1.0795)
+			(end 2.8956 1.0795)
+			(stroke (width 0.1524) (type solid))
+			(layer "F.CrtYd")
+		)
+		(fp_line
+			(start -2.8956 1.0795)
+			(end -3.048 1.0795)
+			(stroke (width 0.1524) (type solid))
+			(layer "F.CrtYd")
+		)
+		(fp_line
+			(start -2.8956 1.651)
+			(end -2.8956 1.0795)
+			(stroke (width 0.1524) (type solid))
+			(layer "F.CrtYd")
+		)
+		(fp_line
+			(start -2.8956 -1.0795)
+			(end -2.8956 -1.651)
+			(stroke (width 0.1524) (type solid))
+			(layer "F.CrtYd")
+		)
+		(fp_line
+			(start -2.8956 -1.651)
+			(end 2.8956 -1.651)
+			(stroke (width 0.1524) (type solid))
+			(layer "F.CrtYd")
+		)
+		(fp_line
+			(start 2.8956 -1.651)
+			(end 2.8956 -1.0795)
+			(stroke (width 0.1524) (type solid))
+			(layer "F.CrtYd")
+		)
+		(fp_line
+			(start 2.8956 1.0795)
+			(end 2.8956 1.651)
+			(stroke (width 0.1524) (type solid))
+			(layer "F.CrtYd")
+		)
+		(fp_line
+			(start 2.8956 1.651)
+			(end -2.8956 1.651)
+			(stroke (width 0.1524) (type solid))
+			(layer "F.CrtYd")
+		)
+		(fp_line
+			(start -2.7686 1.524)
+			(end 2.7686 1.524)
+			(stroke (width 0.1524) (type solid))
+			(layer "F.SilkS")
+		)
+		(fp_line
+			(start 2.7686 1.524)
+			(end 2.7686 1.15824)
+			(stroke (width 0.1524) (type solid))
+			(layer "F.SilkS")
+		)
+		(fp_line
+			(start 2.7686 -1.524)
+			(end -2.7686 -1.524)
+			(stroke (width 0.1524) (type solid))
+			(layer "F.SilkS")
+		)
+		(fp_line
+			(start -2.7686 -1.524)
+			(end -2.7686 -1.15824)
+			(stroke (width 0.1524) (type solid))
+			(layer "F.SilkS")
+		)
+		(fp_line
+			(start -2.7686 1.15824)
+			(end -2.7686 1.524)
+			(stroke (width 0.1524) (type solid))
+			(layer "F.SilkS")
+		)
+		(fp_line
+			(start 2.7686 -1.15824)
+			(end 2.7686 -1.524)
+			(stroke (width 0.1524) (type solid))
+			(layer "F.SilkS")
+		)
+		(fp_line
+			(start -2.6416 1.397)
+			(end 2.6416 1.397)
+			(stroke (width 0.0254) (type solid))
+			(layer "F.Fab")
+		)
+		(fp_line
+			(start 2.6416 1.397)
+			(end 2.6416 -1.397)
+			(stroke (width 0.0254) (type solid))
+			(layer "F.Fab")
+		)
+		(fp_line
+			(start 2.6416 -1.397)
+			(end -2.6416 -1.397)
+			(stroke (width 0.0254) (type solid))
+			(layer "F.Fab")
+		)
+		(fp_line
+			(start -2.6416 -1.397)
+			(end -2.6416 1.397)
+			(stroke (width 0.0254) (type solid))
 			(layer "F.Fab")
 		)
 		(fp_text user "${REFERENCE}"
-			(at 0 -2.5 0)
-			(layer "F.Fab")
-			(effects
-				(font
-					(size 1 1)
-					(thickness 0.15)
-				)
-			)
-		)
-		(pad "1" smd roundrect
-			(at -2 0 180)
-			(size 2.5 1.8)
-			(layers "F.Cu" "F.Mask" "F.Paste")
-			(roundrect_rratio 0.1388888889)
+			(at 0 0 180)
+			(layer "F.Fab")
+			(effects (font (size 1 1) (thickness 0.15)))
+		)
+		(pad "1" smd rect
+			(at -1.7018 0 270)
+			(size 1.651 2.1844)
+			(layers "F.Cu" "F.Paste" "F.Mask")
 			(net "GND")
 			(pinfunction "A1_1")
 			(pintype "passive")
 		)
-		(pad "2" smd roundrect
-			(at 2 0 180)
-			(size 2.5 1.8)
-			(layers "F.Cu" "F.Mask" "F.Paste")
-			(roundrect_rratio 0.1388888889)
+		(pad "2" smd rect
+			(at 1.7018 0 270)
+			(size 1.651 2.1844)
+			(layers "F.Cu" "F.Paste" "F.Mask")
 			(net "VBAT")
 			(pinfunction "A2_2")
 			(pintype "passive")
 		)
+		(model "${KICAD10_3DMODEL_DIR}/Diode_SMD.3dshapes/D_SMA.step"
+			(offset (xyz 0 0 0))
+			(scale (xyz 1 1 1))
+			(rotate (xyz 0 0 0))
+		)
 		(embedded_fonts no)

Commit message: Sync U1 PCB footprint name with source CAD
Parts:
- U1: footprint H743_Custom:ST_USBLC6-2P6_SOT-666 -> H743_Custom:SOT50P160X60-6N
Changed lines of the file:
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@@
 		)
 	)
-	(footprint "H743_Custom:ST_USBLC6-2P6_SOT-666"
+	(footprint "H743_Custom:SOT50P160X60-6N"
 		(layer "F.Cu")
 		(at 82.5 88 -90)

Commit message: Sync U1 and D2 dedicated footprint library names on PCB
Parts:
- D2: footprint H743_Custom:SMAJ30CA_SMA_LTF -> SMAJ30CA:SMASeries_LTF
- U1: footprint H743_Custom:SOT50P160X60-6N -> USBLC6_2P6:SOT50P160X60-6N
Changed lines of the file:
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@@
 		)
 	)
-	(footprint "H743_Custom:SMAJ30CA_SMA_LTF"
+	(footprint "SMAJ30CA:SMASeries_LTF"
 		(layer "F.Cu")
 		(at 83.5 93 180)
@@
 		)
 	)
-	(footprint "H743_Custom:SOT50P160X60-6N"
+	(footprint "USBLC6_2P6:SOT50P160X60-6N"
 		(layer "F.Cu")
 		(at 82.5 88 -90)

Commit message: update pcb
Parts:
- added D5: PESD2CAN, Package_TO_SOT_SMD:SOT-23, F.Cu at (120.5, 105.8)
- added J13: Can1_2, H743_Custom:SolderPadArray_1x04_P2.54mm_1x1mm, F.Cu at (75.5, 109.5)
- added J14: Can1_1, H743_Custom:SolderPadArray_1x04_P2.54mm_1x1mm, F.Cu at (77.5, 109.5)
- added U7: TJA1051TK/3,118, Package_SON:HVSON-8-1EP_3x3mm_P0.65mm_EP1.6x2.4mm, B.Cu at (86.4, 117.6)
- C16, C17, C20, C21, C23, C24, C25, D2, D3, D4, J12, L1, R1, R2, R47, R48, R49, R50, R9, U1, U3, USB1: moved to B.Cu
- J1: value Conn_01x04 -> Analog
- J10: value Conn_01x03 -> Led ext
- J11: value Conn_01x03 -> Buzzer
- J2: value Conn_01x04 -> Uart1
- J3: value Conn_01x04 -> Uart4
- J4: value Conn_01x06 -> Uart7
- J5: value Conn_01x04 -> Uart(
- J6: value Conn_01x04 -> Uart6
- J7: value Conn_01x04 -> Uart3
- J8: value Conn_01x04 -> I2C1
- J9: value Conn_01x04 -> I2C_2
- U14: value ZX-SH1.0-8PWT -> SM08B-SRSS-TB(LF)(SN); moved to B.Cu
- U8: value ZX-SH1.0-4PWT -> SM04B-GHS-TB(LF)(SN); footprint Connector_JST:JST_GH_SM05B-GHS-TB_1x05-1MP_P1.25mm_Horizontal -> H743_Custom:JST_GH_SM04B-GHS-TB_1x04_P1.25mm_Horizontal_GNDtabs; moved to B.Cu
- moved C19 129.1 mm to (76.5, 100.0), turned to 180 degrees
- moved C18 113.4 mm to (77.5, 94.5), turned to 180 degrees
- moved J8 103.0 mm to (89.0, 121.0)
- moved J1 102.5 mm to (100.0, 88.5)
- moved J9 93.9 mm to (99.0, 121.0)
- moved J2 81.2 mm to (98.5, 86.5)
- moved J3 81.0 mm to (98.5, 90.5)
- moved J4 72.6 mm to (108.0, 99.0), turned to 90 degrees
- moved J7 70.2 mm to (108.0, 111.0), turned to 90 degrees
- moved J11 69.5 mm to (93.5, 119.0)
- moved J5 68.9 mm to (110.0, 98.0), turned to 90 degrees
- moved J6 68.2 mm to (110.0, 107.5), turned to 90 degrees
- moved J10 61.3 mm to (101.0, 119.0)
- moved J12 50.1 mm to (98.5, 95.8), turned to 0 degrees
- moved U10 31.3 mm to (178.8, 131.8)
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