File: BUZZER.kicad_sch (KiCad schematic)
At the start: 4 parts, among them J10 Conn_01x03, Q1 AO3400A

Commit message: update cmp number
Parts:
- added J10: Conn_01x03, H743_Custom:SolderPadArray_1x03_P2.54mm_1x1mm, symbol Connector_Generic:Conn_01x03
- renumbered J10 to J11
Connections:
- net +5V_SYS: now also J10.2 (Pin_2)
- net GND: now also J10.1 (Pin_1)
- new net LED_STRIP: J10.3 (Pin_3)

Commit message: update pcb
Parts:
- J10: value Conn_01x03 -> Led ext
- J11: value Conn_01x03 -> Buzzer
Changed lines of the file:
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@@
 			)
 		)
-		(property "Value" "Conn_01x03"
+		(property "Value" "Buzzer"
 			(at 144.78 53.3399 0)
 			(show_name no)
@@
 			)
 		)
-		(property "Value" "Conn_01x03"
+		(property "Value" "Led ext"
 			(at 62.23 81.2799 0)
 			(show_name no)

Commit message: Review component footprints, restore local libraries and reconcile PCB pads
Parts:
- J10, J11: symbol Connector_Generic:Conn_01x03 -> FC01_Project:BUZZER__Conn_01x03
- Q1: symbol Transistor_FET:AO3400A -> FC01_Project:BUZZER__AO3400A; Footprint Audit OK -> See verification/COMPONENTS.csv and verification/REPORT.md; Library Audit KiCad standard -> See verification/COMPONENTS.csv and verification/REPORT.md
- R39, R40: symbol Device:R_Small -> FC01_Project:BUZZER__R_Small; Footprint Audit OK -> See verification/COMPONENTS.csv and verification/REPORT.md; Library Audit KiCad standard -> See verification/COMPONENTS.csv and verification/REPORT.md
Changed lines of the file:
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@@
 	)
 	(symbol
-		(lib_id "power:GND")
+		(lib_id "FC01_Project:BUZZER__GND")
 		(at 135.89 62.23 0)
 		(unit 1)
@@
 	)
 	(symbol
-		(lib_id "Device:R_Small")
+		(lib_id "FC01_Project:BUZZER__R_Small")
 		(at 93.98 66.04 0)
 		(mirror y)
@@
 			)
 		)
-		(property "Footprint Audit" "OK"
+		(property "Footprint Audit" "See verification/COMPONENTS.csv and verification/REPORT.md"
 			(at 97.155 64.135 0)
 			(hide yes)
@@
 			)
 		)
-		(property "Library Audit" "KiCad standard"
+		(property "Library Audit" "See verification/COMPONENTS.csv and verification/REPORT.md"
 			(at 97.155 64.135 0)
 			(hide yes)
@@
 	)
 	(symbol
-		(lib_id "Connector_Generic:Conn_01x03")
+		(lib_id "FC01_Project:BUZZER__Conn_01x03")
 		(at 142.24 52.07 0)
 		(unit 1)
@@
 	)
 	(symbol
-		(lib_id "power:+5V")
+		(lib_id "FC01_Project:BUZZER__+5V")
 		(at 50.8 74.93 0)
 		(unit 1)
@@
 	)
 	(symbol
-		(lib_id "power:GND")
+		(lib_id "FC01_Project:BUZZER__GND")
 		(at 104.14 71.12 0)
 		(unit 1)
@@
 	)
 	(symbol
-		(lib_id "Device:R_Small")
+		(lib_id "FC01_Project:BUZZER__R_Small")
 		(at 88.9 62.23 90)
 		(unit 1)
@@
 			)
 		)
-		(property "Footprint Audit" "OK"
+		(property "Footprint Audit" "See verification/COMPONENTS.csv and verification/REPORT.md"
 			(at 85.09 60.96 90)
 			(hide yes)
@@
 			)
 		)
-		(property "Library Audit" "KiCad standard"
+		(property "Library Audit" "See verification/COMPONENTS.csv and verification/REPORT.md"
 			(at 85.09 60.96 90)
 			(hide yes)
@@
 	)
 	(symbol
-		(lib_id "power:+5V")
+		(lib_id "FC01_Project:BUZZER__+5V")
 		(at 133.35 46.99 0)
 		(unit 1)
@@
 	)
 	(symbol
-		(lib_id "Transistor_FET:AO3400A")
+		(lib_id "FC01_Project:BUZZER__AO3400A")
 		(at 101.6 62.23 0)
 		(unit 1)
@@
 			)
 		)
-		(property "Footprint Audit" "OK"
+		(property "Footprint Audit" "See verification/COMPONENTS.csv and verification/REPORT.md"
 			(at 107.95 60.9599 0)
 			(hide yes)
@@
 			)
 		)
-		(property "Library Audit" "KiCad standard"
+		(property "Library Audit" "See verification/COMPONENTS.csv and verification/REPORT.md"
 			(at 107.95 60.9599 0)
 			(hide yes)
@@
 	)
 	(symbol
-		(lib_id "power:GND")
+		(lib_id "FC01_Project:BUZZER__GND")
 		(at 53.34 90.17 0)
 		(unit 1)
@@
 	)
 	(symbol
-		(lib_id "Connector_Generic:Conn_01x03")
+		(lib_id "FC01_Project:BUZZER__Conn_01x03")
 		(at 59.69 80.01 0)
 		(unit 1)
