File: UART_I2C.kicad_sch (KiCad schematic)
At the start: 26 parts, among them J2 Conn_01x04, J3 Conn_01x04, J4 Conn_01x06, J5 Conn_01x04, J6 Conn_01x04, J7 Conn_01x04

Commit message: update
Parts:
- renumbered C19 to C36, C20 to C37, C21 to C38, C22 to C39, C23 to C40, C24 to C41, R14 to R20, R15 to R21, R16 to R22, R17 to R23, R18 to R24, R19 to R25, R20 to R26, R21 to R27, R22 to R28, R23 to R29, R24 to R30, R25 to R31, R26 to R32, R27 to R33

Commit message: update pcb
Parts:
- J2: value Conn_01x04 -> Uart1
- J3: value Conn_01x04 -> Uart4
- J4: value Conn_01x06 -> Uart7
- J5: value Conn_01x04 -> Uart(
- J6: value Conn_01x04 -> Uart6
- J7: value Conn_01x04 -> Uart3
Changed lines of the file:
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@@
 			)
 		)
-		(property "Value" "Conn_01x04"
+		(property "Value" "Uart("
 			(at 137.16 27.9399 0)
 			(show_name no)
@@
 			)
 		)
-		(property "Value" "Conn_01x04"
+		(property "Value" "Uart6"
 			(at 157.48 57.1499 0)
 			(show_name no)
@@
 			)
 		)
-		(property "Value" "Conn_01x04"
+		(property "Value" "Uart4"
 			(at 90.17 58.4199 0)
 			(show_name no)
@@
 			)
 		)
-		(property "Value" "Conn_01x04"
+		(property "Value" "Uart3"
 			(at 184.15 27.9399 0)
 			(show_name no)
@@
 		(in_pos_files yes)
 		(dnp no)
-		(fields_autoplaced yes)
 		(property "Reference" "J2"
 			(at 90.17 25.3999 0)
@@
 			)
 		)
-		(property "Value" "Conn_01x04"
-			(at 90.17 27.9399 0)
+		(property "Value" "Uart1"
+			(at 90.678 31.75 90)
 			(show_name no)
 			(do_not_autoplace no)
@@
 			)
 		)
-		(property "Value" "Conn_01x06"
+		(property "Value" "Uart7"
 			(at 110.49 83.8199 0)
 			(show_name no)

Commit message: Review component footprints, restore local libraries and reconcile PCB pads
Parts:
- C36, C37, C38, C39, C40, C41: symbol Device:C_Small -> FC01_Project:UART_I2C__C_Small; Footprint Audit OK -> See verification/COMPONENTS.csv and verification/REPORT.md; Library Audit KiCad standard -> See verification/COMPONENTS.csv and verification/REPORT.md
- J2, J3, J5, J6, J7: symbol Connector_Generic:Conn_01x04 -> FC01_Project:UART_I2C__Conn_01x04; Footprint Audit OK: 4 square SMD pads 1.00x1.00 mm, P2.54 mm, no holes, no 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 -> See verification/COMPONENTS.csv and verification/REPORT.md; Library Audit Project-local H743_Custom footprint -> See verification/COMPONENTS.csv and verification/REPORT.md
- J4: symbol Connector_Generic:Conn_01x06 -> FC01_Project:UART_I2C__Conn_01x06; Footprint Audit OK: 6 square SMD pads 1.00x1.00 mm, P2.54 mm, no holes, no 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 -> See verification/COMPONENTS.csv and verification/REPORT.md; Library Audit Project-local H743_Custom footprint -> See verification/COMPONENTS.csv and verification/REPORT.md
- R20, R21, R22, R23, R24, R25, R26, R27, R28, R29, R30, R31, R32, R33: symbol Device:R_Small -> FC01_Project:UART_I2C__R_Small; Footprint Audit OK -> See verification/COMPONENTS.csv and verification/REPORT.md; Library Audit KiCad standard -> See verification/COMPONENTS.csv and verification/REPORT.md
