File: SENSORS.kicad_sch (KiCad schematic)
At the start: 25 parts, among them J8 I2C1, J9 I2C_2, U10 LSM6DSV16X, U11 ICM-45686, U12 BMP581, U13 DPS368XTSA1, U9 BMI088

Commit message: Define SPI2 bus members across MCU and sensors
Changed lines of the file:
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@@
 		)
 	)
-	(hierarchical_label "SPI2{SPI}"
+	(hierarchical_label "SPI2{CS MISO MOSI SCLK}"
 		(shape bidirectional)
 		(at 27.94 115.57 180)

Commit message: Define reusable aliases for hierarchical buses
Changed lines of the file:
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@@
 		)
 	)
-	(hierarchical_label "SPI3{SPI}"
+	(hierarchical_label "SPI3{SPI_NO_CS}"
 		(shape bidirectional)
 		(at 29.21 88.9 180)
@@
 		)
 	)
-	(hierarchical_label "SPI2{CS MISO MOSI SCLK}"
+	(hierarchical_label "SPI2{SPI}"
 		(shape bidirectional)
 		(at 27.94 115.57 180)

Commit message: Correct ERC pin models and power connectivity
Changed lines of the file:
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@@
-	(wire
-		(pts
-			(xy 154.94 48.26) (xy 153.67 48.26)
-		)
-		(stroke
-			(width 0)
-			(type default)
-		)
-	)
 	(wire
 		(pts
@@
 	(wire
 		(pts
-			(xy 154.94 50.8) (xy 153.67 50.8)
-		)
-		(stroke
-			(width 0)
-			(type default)
-		)
-	)
-	(wire
-		(pts
 			(xy 190.5 60.96) (xy 207.01 60.96)
 		)
@@
 	(wire
 		(pts
-			(xy 154.94 53.34) (xy 153.67 53.34)
-		)
-		(stroke
-			(width 0)
-			(type default)
-		)
-	)
-	(wire
-		(pts
 			(xy 256.54 107.95) (xy 256.54 113.03)
 		)
@@
 	(wire
 		(pts
-			(xy 154.94 45.72) (xy 153.67 45.72)
-		)
-		(stroke
-			(width 0)
-			(type default)
-		)
-	)
-	(wire
-		(pts
 			(xy 105.41 144.78) (xy 105.41 143.51)
 		)
@@
 		)
 		(stroke
-			(width 0)
-			(type default)
-		)
-	)
-	(wire
-		(pts
-			(xy 154.94 43.18) (xy 153.67 43.18)
-		)
-		(stroke

Commit message: Fix U12 BMP581 footprint to Bosch DS004-13 land pattern
Parts:
- U12: Footprint Audit Bosch BMP581 DS004-13 pp.46,68–69: pads haut/bas corrigés à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 -> Bosch BMP581 DS004-13 §8.2 / Fig.32: land pads 0.325 x 0.30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
Changed lines of the file:
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@@
 			)
 		)
-		(property "Footprint Audit" "Bosch BMP581 DS004-13 pp.46,68–69: pads haut/bas corrigés à 0.300 x 0.325 mm (extension 25 um autour de la terminaison). Ouverture masque sous corps 2.2 x 2.2; recommandation Bosch sans solder mask sous capteur. Contrôle fab/assemblage nécessaire."
+		(property "Footprint Audit" "Bosch BMP581 DS004-13 §8.2 / Fig.32: land pads 0.325 x 0.300 mm (6x + 4x, orientés selon le côté), pas 0.5 mm, span 1.525 mm; ouverture solder mask 2.2 x 2.2 mm; pas de vias ni pistes sous le capteur. Empreinte projet alignée sur le land pattern constructeur."
 			(at 226.06 92.71 0)
 			(hide yes)
